File: HW/projects/fennek_2017_18/BMS/Current_Sense/current_sense_v1_lem/current_sense.sch (KiCad schematic (older format))
At the start: 7 parts, among them IC1 HO_25-NP/SP33, P1 Input, P2 output, P3 signal

Commit message: Update github repo with designs for fennek 2018
Parts:
- C1, C2, C3: symbol C_Small -> current_sense-rescue:C_Small
- IC1: symbol HO_25-NP/SP33 -> tera_general:HO_25-NP_SP33
- P1, P2: symbol CONN_01X03 -> current_sense-rescue:CONN_01X03
- P3: symbol CONN_01X04 -> current_sense-rescue:CONN_01X04
Changed lines of the file:
@@
-EESchema Schematic File Version 2
-LIBS:power
-LIBS:device
-LIBS:transistors
-LIBS:conn
-LIBS:linear
-LIBS:regul
-LIBS:74xx
-LIBS:cmos4000
-LIBS:adc-dac
-LIBS:memory
-LIBS:xilinx
-LIBS:microcontrollers
-LIBS:dsp
-LIBS:microchip
-LIBS:analog_switches
-LIBS:motorola
-LIBS:texas
-LIBS:intel
-LIBS:audio
-LIBS:interface
-LIBS:digital-audio
-LIBS:philips
-LIBS:display
-LIBS:cypress
-LIBS:siliconi
-LIBS:opto
-LIBS:atmel
-LIBS:contrib
-LIBS:valves
-LIBS:ft232rl
-LIBS:relais
-LIBS:Supply
-LIBS:tera_connectors
-LIBS:tera_emc_prodection
-LIBS:tera_general
-LIBS:tera_logic
-LIBS:tera_processors
-LIBS:tera_sensoric
-LIBS:tera_switches
-LIBS:lem_v1-cache
-EELAYER 25 0
+EESchema Schematic File Version 4
+LIBS:current_sense-cache
+EELAYER 26 0
 EELAYER END
 $Descr A4 11693 8268
@@
 $EndDescr
 $Comp
-L HO_25-NP/SP33 IC1
+L tera_general:HO_25-NP_SP33 IC1
 U 1 1 59360AFD
 P 5100 2800
@@
 	4200 2200 4600 2200
 Wire Wire Line
-	4600 2200 4600 2700
+	4600 2200 4600 2500
 Wire Wire Line
 	4600 2500 4700 2500
@@
 	4700 2900 4600 2900
 Wire Wire Line
-	4600 2900 4600 3250
+	4600 2900 4600 3000
 Wire Wire Line
 	4600 3250 4200 3250
@@
 NoConn ~ 5500 2800
 $Comp
-L CONN_01X04 P3
+L current_sense-rescue:CONN_01X04 P3
 U 1 1 59360F1D
 P 8200 2850
@@
 $EndComp
 Wire Wire Line
-	5550 3000 5550 3400
+	5550 3000 5550 3100
 Wire Wire Line
 	5550 3000 5500 3000
 Wire Wire Line
-	5500 2600 6300 2600
+	5500 2600 5950 2600
 Wire Wire Line
 	5500 2900 6300 2900
 $Comp
-L PWR_FLAG #FLG01
+L power1:PWR_FLAG #FLG01
 U 1 1 5936111B
 P 7800 2550
@@
 	7800 2550 7800 2700
 $Comp
-L PWR_FLAG #FLG02
+L power1:PWR_FLAG #FLG02
 U 1 1 5936115D
 P 7800 3150
@@
 	7800 3150 7800 3000
 $Comp
-L CONN_01X03 P1
+L current_sense-rescue:CONN_01X03 P1
 U 1 1 593612EB
 P 4000 2300
@@
 $EndComp
 $Comp
-L CONN_01X03 P2
+L current_sense-rescue:CONN_01X03 P2
 U 1 1 5936143F
 P 4000 3150
@@
 	4200 2300 4300 2300
 Wire Wire Line
-	4300 2300 4300 3150
+	4300 2300 4300 2400
 Wire Wire Line
 	4300 2400 4200 2400
@@
 HV-
 $Comp
-L GND #PWR03
+L power1:GND #PWR03
 U 1 1 59361FC6
 P 5550 3400
@@
 $EndComp
 $Comp
-L VCC #PWR04
+L power1:VCC #PWR04
 U 1 1 59362089
 P 6300 2400
@@
 Standby
 $Comp
-L VCC #PWR05
+L power1:VCC #PWR05
 U 1 1 5937E95D
 P 7500 2550
@@
 	7500 2550 7500 2700
 Wire Wire Line
-	7500 2700 8000 2700
+	7500 2700 7800 2700
 Connection ~ 7800 2700
 Wire Wire Line
-	7500 3000 8000 3000
-$Comp
-L GND #PWR06
+	7500 3000 7800 3000
+$Comp
+L power1:GND #PWR06
 U 1 1 5937EA9C
 P 7500 3050
@@
 Connection ~ 7800 3000
 Wire Wire Line
-	6300 2500 5500 2500
-$Comp
-L C_Small C1
+	6300 2500 6150 2500
+$Comp
+L current_sense-rescue:C_Small C1
 U 1 1 5937EC82
 P 5750 3100
@@
 $EndComp
 $Comp
-L C_Small C2
+L current_sense-rescue:C_Small C2
 U 1 1 5937EF96
 P 5950 3100
@@
 $EndComp
 $Comp
-L C_Small C3
+L current_sense-rescue:C_Small C3
 U 1 1 5937EFBE
 P 6150 3100
@@
 	5750 3200 5750 3300
 Wire Wire Line
-	5550 3300 6150 3300
+	5550 3300 5750 3300
 Connection ~ 5550 3300
 Wire Wire Line
@@
 Wire Wire Line
 	5750 2700 5500 2700
+Wire Wire Line
+	4600 2500 4600 2600
+Wire Wire Line
+	4600 2600 4600 2700
+Wire Wire Line
+	4600 3000 4600 3100
+Wire Wire Line
+	4600 3100 4600 3250
+Wire Wire Line
+	4300 3050 4300 3150
+Wire Wire Line
+	4300 2400 4300 3050
+Wire Wire Line
+	7800 2700 8000 2700
+Wire Wire Line
+	7800 3000 8000 3000
+Wire Wire Line
+	5950 2600 6300 2600
+Wire Wire Line
+	6150 2500 5500 2500
+Wire Wire Line
+	5550 3300 5550 3400
+Wire Wire Line
+	5750 3300 5950 3300
+Wire Wire Line
+	5950 3300 6150 3300
+Wire Wire Line
+	5550 3100 5550 3300
 $EndSCHEMATC
