File: HW/projects/fennek_2017_18/BMS/master_fennek18/BMS_Master_V7 -- fennek18/BMS_Master_V7_kicad.kicad_pcb (KiCad board)
At the start: 4 copper layers, 77 x 58.5 mm, 128 parts, among them K1 ASSR-1218, K2 ASSR-1218, K3 ASSR-1218, P1 Buttons, P17 CAN_CON_2pol, P2 Host_slave, P3 ExtGPIO, P4 LEM, P5 LEM, P6 CONN_02X22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

Commit message: Update github repo with designs for fennek 2018
Parts:
- removed D20: 5V, tera_diodes:DO-216AA
- removed D21: 3V3, tera_diodes:DO-216AA
- removed R11, R19, R20, R21: 1k, tera_rlc:R_0603in
- removed R15, R16, R17: 100k, tera_rlc:R_0603in
- added C23: 4u7, tera_rlc:C_0805in, B.Cu at (136.8, 78.2)
- added C24: 4u7, tera_rlc:C_0805in, B.Cu at (108.4, 94.2)
- added C28: 4u7, tera_rlc:C_0805in, B.Cu at (134.2, 72.4)
- added C29: 4u7, tera_rlc:C_0805in, B.Cu at (101.5, 97.0)
- added G2: TSR_0.5-2450, traco_power:TSR_0.5, F.Cu at (134.2, 69.1)
- added G3: TSR_0.5-2433, traco_power:TSR_0.5, F.Cu at (100.4, 94.9)
- added L4: 3u3, tera_rlc:L_0805in, B.Cu at (136.8, 74.0)
- added L5: 3u3, tera_rlc:L_0805in, B.Cu at (104.2, 94.2)
- R12, R13, R14: value 1k -> 100R
- moved REF** 10.0 mm to (62.0, 56.0)
- moved R22 5.00 mm to (104.3, 91.4), turned to 90 degrees
- moved C1 4.99 mm to (131.6, 82.0), turned to 180 degrees
- moved C10 1.81 mm to (138.0, 66.2)
- moved R30 1.03 mm to (138.0, 63.0)
- moved L1 0.44 mm to (135.1, 82.0)
Connections:
- JP1 pad 2: /SPI_Controller/MISO_5V_1 -> /SPI_MISO_5V
- JP4 pad 2: /SPI_Controller/MOSI_5V_1 -> /SPI_MOSI_5V
- JP5 pad 2: /SPI_Controller/SCLK_5V_1 -> /SPI_CLK_5V
- R18 pad 1: /SPI_Controller/MISO_5V_1 -> /SPI_MISO_5V
- U5 pad 11: /SPI_Controller/SCLK_5V_1 -> /SPI_CLK_5V
- U5 pad 12: /SPI_Controller/MOSI_5V_1 -> /SPI_MOSI_5V
- U5 pad 13: /SPI_Controller/MISO_5V_1 -> /SPI_MISO_5V
- U5 pad 8: Net-(R11-Pad1) -> /SPI_CS
Routing:
- net /SPI_MISO_5V: track 54.4 -> 65.2 mm
- net /SPI_CS: track 24.5 -> 35.2 mm, vias 0 -> 1
- net /SPI_MOSI_5V: track 58.4 -> 67.7 mm
- net Net-(R11-Pad1): track 9.06 -> 0.00 mm, vias 1 -> 0
- net /SPI_Controller/MISO_5V_1: track 8.81 -> 0.00 mm
- net /SPI_CLK_5V: track 63.1 -> 70.3 mm
- net /SPI_Controller/MOSI_5V_1: track 6.94 -> 0.00 mm
- net /Interlock_On1: track 39.0 -> 33.2 mm
- net Net-(C28-Pad1): track 0.00 -> 5.51 mm
- net /SPI_Controller/SCLK_5V_1: track 5.35 -> 0.00 mm
- net Net-(K1-Pad1): track 6.95 -> 11.6 mm
- net /NFAULT: track 57.0 -> 52.6 mm, vias 2 -> 1
- net GND: track 61.3 -> 57.7 mm, vias 55 -> 56
- net /NALERT: track 60.4 -> 56.9 mm, vias 2 -> 1
- net /NCS_12V_Relay: track 32.1 -> 34.5 mm
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- added copper zone on B.Cu, net +12V
- added copper zone on B.Cu, net Net-(C29-Pad1)
- removed copper zone on B.Cu, net +5V
Other:
- board text added: "BMS Master Fennek (V7.0) TERA TU Graz ©Pöschl, Apr. 2018 Solderpad v0.51"
- board text added: "©Pöschl, 2018 Solderpad v0.51"
- board text removed: "BMS Master Fennek (V7.0) TERA TU Graz ©Pöschl, Jun.2017 Solderpad v0.51"
- board text removed: "©Pöschl, 2017 Solderpad v0.51"
