File: HW/projects/fennek_2017_18/BMS/measurement_and_balancing/bms_board_V6-1__12s_fennek2017/Daisychain.sch (KiCad schematic (older format))
At the start: 23 parts

Commit message: Update github repo with designs for fennek 2018
Parts:
- C35, C36, C37, C38, C39, C40, C52, C53, C54: symbol C_Small -> bms_board-rescue:C_Small
- R22, R23, R24, R25, R26, R27, R28, R29, R30, R31, R32, R33, R34, R35: symbol R_Small -> bms_board-rescue:R_Small
Changed lines of the file:
@@
-EESchema Schematic File Version 2
-LIBS:power
-LIBS:device
-LIBS:transistors
-LIBS:conn
-LIBS:linear
-LIBS:regul
-LIBS:74xx
-LIBS:cmos4000
-LIBS:adc-dac
-LIBS:memory
-LIBS:xilinx
-LIBS:microcontrollers
-LIBS:dsp
-LIBS:microchip
-LIBS:analog_switches
-LIBS:motorola
-LIBS:texas
-LIBS:intel
-LIBS:audio
-LIBS:interface
-LIBS:digital-audio
-LIBS:philips
-LIBS:display
-LIBS:cypress
-LIBS:siliconi
-LIBS:opto
-LIBS:atmel
-LIBS:contrib
-LIBS:valves
-LIBS:relais
-LIBS:Supply
-LIBS:tera_general
-LIBS:tera_logic
-LIBS:tera_processors
-LIBS:tera_switches
-LIBS:local_power
-LIBS:ft232rl
-LIBS:tera_connectors
-LIBS:tera_emc_prodection
+EESchema Schematic File Version 4
 LIBS:bms_board-cache
-EELAYER 25 0
+EELAYER 26 0
 EELAYER END
 $Descr A4 11693 8268
@@
 $EndDescr
 $Comp
-L R_Small R29
+L bms_board-rescue:R_Small R29
 U 1 1 5882CD79
 P 4150 4850
@@
 $EndComp
 $Comp
-L R_Small R26
+L bms_board-rescue:R_Small R26
 U 1 1 5882CD80
 P 4150 2450
@@
 $EndComp
 $Comp
-L R_Small R27
+L bms_board-rescue:R_Small R27
 U 1 1 5882CD87
 P 4150 2550
@@
 $EndComp
 $Comp
-L R_Small R28
+L bms_board-rescue:R_Small R28
 U 1 1 5882CD8E
 P 4150 2900
@@
 $EndComp
 $Comp
-L R_Small R22
+L bms_board-rescue:R_Small R22
 U 1 1 5882CD95
 P 3600 3100
@@
 $EndComp
 $Comp
-L R_Small R23
+L bms_board-rescue:R_Small R23
 U 1 1 5882CD9C
 P 3800 3100
@@
 $EndComp
 $Comp
-L R_Small R25
+L bms_board-rescue:R_Small R25
 U 1 1 5882CDA3
 P 4000 3100
@@
 $EndComp
 $Comp
-L R_Small R24
+L bms_board-rescue:R_Small R24
 U 1 1 5882CDAA
 P 3800 5100
@@
 $EndComp
 $Comp
-L C_Small C36
+L bms_board-rescue:C_Small C36
 U 1 1 5882CDB7
 P 3400 4400
@@
 $EndComp
 $Comp
-L C_Small C35
+L bms_board-rescue:C_Small C35
 U 1 1 5882CDBE
 P 3400 2350
@@
 $EndComp
 $Comp
-L R_Small R33
+L bms_board-rescue:R_Small R33
 U 1 1 5882CDD7
 P 5750 4750
@@
 $EndComp
 $Comp
-L R_Small R32
+L bms_board-rescue:R_Small R32
 U 1 1 5882CDDE
 P 5750 4650
@@
 $EndComp
 $Comp
-L R_Small R31
+L bms_board-rescue:R_Small R31
 U 1 1 5882CDE5
 P 5750 4550
@@
 $EndComp
 $Comp
-L R_Small R30
+L bms_board-rescue:R_Small R30
 U 1 1 5882CDEC
 P 5750 2800
@@
 $EndComp
 $Comp
-L C_Small C40
+L bms_board-rescue:C_Small C40
 U 1 1 5882CDF3
 P 6250 3050
@@
 $EndComp
 $Comp
-L C_Small C38
+L bms_board-rescue:C_Small C38
 U 1 1 5882CDFA
 P 6050 3050
@@
 $EndComp
 $Comp
-L C_Small C37
+L bms_board-rescue:C_Small C37
 U 1 1 5882CE01
 P 5850 3050
@@
 $EndComp
 $Comp
-L C_Small C39
+L bms_board-rescue:C_Small C39
 U 1 1 5882CE08
 P 6050 5100
@@
 $EndComp
 $Comp
-L R_Small R34
+L bms_board-rescue:R_Small R34
 U 1 1 5882CE0F
 P 6450 2300
@@
 $EndComp
 $Comp
-L R_Small R35
+L bms_board-rescue:R_Small R35
 U 1 1 5882CE16
 P 6550 4300
@@
 CONV_2
 $Comp
-L C_Small C53
+L bms_board-rescue:C_Small C53
 U 1 1 5866A39B
 P 4950 3000
@@
 $EndComp
 $Comp
-L C_Small C52
+L bms_board-rescue:C_Small C52
 U 1 1 5866BB1F
 P 4950 2300
@@
 VBatt-
 $Comp
-L C_Small C54
+L bms_board-rescue:C_Small C54
 U 1 1 5868D075
 P 4950 2650
