File: HW/projects/fennek_2017_18/BMS/measurement_and_balancing/bms_board_V6-1__12s_fennek2017/bms_board.sch (KiCad schematic (older format))
At the start: 11 parts, among them P1 Battery_Interface, P2 TS1, P3 TS2

Commit message: Update github repo with designs for fennek 2018
Parts:
- removed P1: Battery_Interface, tera_Connectors_JST:JST_XH_S13B-XH-A_13x2.50mm_Angled, symbol CONN_01X13
- added P1: CONN_01X07, tera_Connectors_JST:JST_EH_S07B-EH_07x2.50mm_Angled, symbol bms_board-rescue:CONN_01X07
- added P5: CONN_01X07, tera_Connectors_JST:JST_XH_S07B-XH-A_07x2.50mm_Angled, symbol bms_board-rescue:CONN_01X07
- C16, C17, C51: symbol C_Small -> bms_board-rescue:C_Small
- P2, P3: symbol CONN_01X02 -> bms_board-rescue:CONN_01X02
- R10, R11, R5, R8, R9: symbol R_Small -> bms_board-rescue:R_Small
Connections:
- wire segments 102 -> 131
- no-connect marks 12 -> 13
Other:
- moved on the sheet: C51
