File: HW/projects/fennek_2017_18/BMS/measurement_and_balancing/bms_board_V6__12s_fennek2017/BalancerOneCell.sch (KiCad schematic (older format))
At the start: 11 parts, among them Q1 BSS205N

Commit message: Update github repo with designs for fennek 2018
Parts:
- C1, C4: symbol C -> Device:C
- D1, D3: symbol ZENER -> Device:D_Zener
- D2: symbol LED -> Device:LED
- Q1: symbol BSS205N -> tera_general:BSS205N
- R1, R2, R3, R4: symbol R -> Device:R
Changed lines of the file:
@@
-EESchema Schematic File Version 2
-LIBS:power
-LIBS:device
-LIBS:transistors
-LIBS:conn
-LIBS:linear
-LIBS:regul
-LIBS:74xx
-LIBS:cmos4000
-LIBS:adc-dac
-LIBS:memory
-LIBS:xilinx
-LIBS:microcontrollers
-LIBS:dsp
-LIBS:microchip
-LIBS:analog_switches
-LIBS:motorola
-LIBS:texas
-LIBS:intel
-LIBS:audio
-LIBS:interface
-LIBS:digital-audio
-LIBS:philips
-LIBS:display
-LIBS:cypress
-LIBS:siliconi
-LIBS:opto
-LIBS:atmel
-LIBS:contrib
-LIBS:valves
-LIBS:relais
-LIBS:Supply
-LIBS:tera_general
-LIBS:tera_logic
-LIBS:tera_processors
-LIBS:tera_switches
-LIBS:local_power
-LIBS:ft232rl
-LIBS:tera_connectors
-LIBS:tera_emc_prodection
+EESchema Schematic File Version 4
 LIBS:bms_board-cache
-EELAYER 25 0
+EELAYER 26 0
 EELAYER END
 $Descr A4 11693 8268
@@
 Celln+
 $Comp
-L R R1
+L Device:R R1
 U 1 1 56F08038
 P 3800 3400
@@
 $EndComp
 $Comp
-L LED D2
+L Device:LED D2
 U 1 1 56F0808B
 P 3800 3850
@@
 $EndComp
 $Comp
-L ZENER D1
+L Device:D_Zener D1
 U 1 1 56F08187
 P 2850 3850
@@
 $EndComp
 $Comp
-L ZENER D3
+L Device:D_Zener D3
 U 1 1 56F08242
 P 4750 4500
@@
 $EndComp
 $Comp
-L BSS205N Q1
+L tera_general:BSS205N Q1
 U 1 1 56F08379
 P 3950 4500
@@
 $EndComp
 $Comp
-L R R3
+L Device:R R3
 U 1 1 56F084AC
 P 5150 4500
@@
 $EndComp
 $Comp
-L R R4
+L Device:R R4
 U 1 1 56F085A7
 P 5550 4250
@@
 VCn
 Wire Wire Line
-	3800 3550 3800 3650
+	3800 3550 3800 3700
 Wire Wire Line
 	4100 4100 4100 3550
 Wire Wire Line
-	3800 4100 4100 4100
-Wire Wire Line
-	3800 4100 3800 4050
+	3800 4100 3950 4100
+Wire Wire Line
+	3800 4100 3800 4000
 Wire Wire Line
 	3950 4100 3950 4300
 Connection ~ 3950 4100
 Wire Wire Line
-	2750 3200 5300 3200
+	2750 3200 2850 3200
 Wire Wire Line
 	3800 3200 3800 3250
@@
 Connection ~ 3800 3200
 Wire Wire Line
-	2700 4750 5150 4750
+	2700 4750 2850 4750
 Wire Wire Line
 	3950 4750 3950 4600
 Wire Wire Line
-	4750 4750 4750 4700
+	4750 4750 4750 4650
 Connection ~ 3950 4750
 Wire Wire Line
-	4750 4300 4750 4250
-Wire Wire Line
-	4150 4250 5400 4250
+	4750 4350 4750 4250
+Wire Wire Line
+	4150 4250 4750 4250
 Wire Wire Line
 	4150 4250 4150 4500
@@
 	5900 4250 5700 4250
 Connection ~ 5150 4250
-Wire Wire Line
-	2850 4050 2850 4750
 Connection ~ 2850 4750
-Wire Wire Line
-	2850 3650 2850 3200
 Connection ~ 2850 3200
 Connection ~ 4100 3200
 $Comp
-L C C1
+L Device:C C1
 U 1 1 56F0944E
 P 3200 3900
@@
 AR Path="/585C2532/5868CA28/56F0944E" Ref="C47"  Part="1"
 AR Path="/585C2532/5868CA2F/56F0944E" Ref="C49"  Part="1"
+AR Path="/56F0944E" Ref="C3"  Part="1"
 F 0 "C3" H 3315 3946 50  0000 L CNN
 F 1 "100n" H 3315 3855 50  0000 L CNN
@@
 Connection ~ 3200 4750
 $Comp
-L R R2
+L Device:R R2
 U 1 1 5862B789
 P 4100 3400
@@
 $EndComp
 $Comp
-L C C4
+L Device:C C4
 U 1 1 5862BE29
 P 5700 3450
@@
 AR Path="/585C2532/5868CA28/5862BE29" Ref="C48"  Part="1"
 AR Path="/585C2532/5868CA2F/5862BE29" Ref="C50"  Part="1"
+AR Path="/5862BE29" Ref="C4"  Part="1"
 F 0 "C4" H 5815 3496 50  0000 L CNN
 F 1 "100n 50V" H 5815 3405 50  0000 L CNN
@@
 $EndComp
 $Comp
-L R R4
+L Device:R R4
 U 1 1 5862BF0B
 P 5450 3200
@@
 $EndComp
 Wire Wire Line
-	5600 3200 5900 3200
+	5600 3200 5700 3200
 Wire Wire Line
 	5700 3300 5700 3200
@@
 Text Notes 5400 4900 0    60   ~ 0
 Balancing circuit
+Wire Wire Line
+	3950 4100 4100 4100
+Wire Wire Line
+	3800 3200 4100 3200
+Wire Wire Line
+	3950 4750 4750 4750
+Wire Wire Line
+	4750 4250 5150 4250
+Wire Wire Line
+	4750 4750 5150 4750
+Wire Wire Line
+	5150 4250 5400 4250
+Wire Wire Line
+	2850 4750 3200 4750
+Wire Wire Line
+	2850 3200 3200 3200
+Wire Wire Line
+	4100 3200 5300 3200
+Wire Wire Line
+	3200 3200 3800 3200
+Wire Wire Line
+	3200 4750 3950 4750
+Wire Wire Line
+	5700 3200 5900 3200
+Wire Wire Line
+	2850 3200 2850 3700
+Wire Wire Line
+	2850 4000 2850 4750
 $EndSCHEMATC
