File: HW/projects/fennek_2017_18/BMS/measurement_and_balancing/bms_board_V6__12s_fennek2017/Chip.sch (KiCad schematic (older format))
At the start: 11 parts, among them IC1 TI-bq76pl536, X1 Prog_Voltage

Commit message: Update github repo with designs for fennek 2018
Parts:
- C1, C11, C12, C14, C15, C2, C5, C7, C8: symbol C -> Device:C
- IC1: symbol TI-bq76pl536-multiunit -> bms_board-rescue:TI-bq76pl536-multiunit
- X1: symbol CONN_01X02 -> Connector_Generic:Conn_01x02
