File: HW/projects/fennek_2017_18/BMS/measurement_and_balancing/bms_board_V6__12s_fennek2017/Host_connect.sch (KiCad schematic (older format))
At the start: 5 parts, among them P4 Host_Interface, Q1 BSS205N, Q2 BSS205N

Commit message: Update github repo with designs for fennek 2018
Parts:
- P4: symbol CONN_01X10 -> Connector_Generic:Conn_01x10
- Q1, Q2: symbol BSS205N -> tera_general:BSS205N
- R36, R37: symbol R_Small -> Device:R_Small
Changed lines of the file:
@@
-EESchema Schematic File Version 2
-LIBS:power
-LIBS:device
-LIBS:transistors
-LIBS:conn
-LIBS:linear
-LIBS:regul
-LIBS:74xx
-LIBS:cmos4000
-LIBS:adc-dac
-LIBS:memory
-LIBS:xilinx
-LIBS:microcontrollers
-LIBS:dsp
-LIBS:microchip
-LIBS:analog_switches
-LIBS:motorola
-LIBS:texas
-LIBS:intel
-LIBS:audio
-LIBS:interface
-LIBS:digital-audio
-LIBS:philips
-LIBS:display
-LIBS:cypress
-LIBS:siliconi
-LIBS:opto
-LIBS:atmel
-LIBS:contrib
-LIBS:valves
-LIBS:relais
-LIBS:Supply
-LIBS:tera_general
-LIBS:tera_logic
-LIBS:tera_processors
-LIBS:tera_switches
-LIBS:local_power
-LIBS:ft232rl
-LIBS:tera_connectors
-LIBS:tera_emc_prodection
+EESchema Schematic File Version 4
 LIBS:bms_board-cache
-EELAYER 25 0
+EELAYER 26 0
 EELAYER END
 $Descr A4 11693 8268
@@
 $EndDescr
 $Comp
-L CONN_01X10 P4
+L Connector_Generic:Conn_01x10 P4
 U 1 1 5886A607
-P 3300 2300
-F 0 "P4" H 3377 2338 50  0000 L CNN
-F 1 "Host_Interface" H 3377 2247 50  0000 L CNN
-F 2 "tera_Connectors_Molex:Molex_PicoBlade_53398-1071_10x1.25mm_Straight" H 3300 2300 50  0001 C CNN
-F 3 "" H 3300 2300 50  0000 C CNN
-F 4 "03-0210" H 3300 2300 60  0001 C CNN "HPN"
-	1    3300 2300
+P 3300 2250
+F 0 "P4" H 3377 2288 50  0000 L CNN
+F 1 "Host_Interface" H 3377 2197 50  0000 L CNN
+F 2 "tera_Connectors_Molex:Molex_PicoBlade_53398-1071_10x1.25mm_Straight" H 3300 2250 50  0001 C CNN
+F 3 "" H 3300 2250 50  0000 C CNN
+F 4 "03-0210" H 3300 2250 60  0001 C CNN "HPN"
+	1    3300 2250
 	1    0    0    -1
 $EndComp
 $Comp
-L BSS205N Q1
+L tera_general:BSS205N Q1
 U 1 1 5886A60E
 P 2200 3000
@@
 $EndComp
 $Comp
-L BSS205N Q2
+L tera_general:BSS205N Q2
 U 1 1 5886A615
 P 2600 3000
@@
 $EndComp
 $Comp
-L R_Small R36
+L Device:R_Small R36
 U 1 1 5886A628
 P 2200 1650
@@
 $EndComp
 $Comp
-L R_Small R37
+L Device:R_Small R37
 U 1 1 5886A635
 P 2600 1650
@@
 	1700 2650 3100 2650
 Wire Wire Line
-	2200 3100 3100 3100
+	2200 3100 2600 3100
 Wire Wire Line
 	2600 3100 2600 3400
@@
 	2600 1350 2600 1550
 Wire Wire Line
-	2200 1750 2200 2800
+	2200 1750 2200 2050
 Wire Wire Line
-	2600 1750 2600 2800
+	2600 1750 2600 2250
 Wire Wire Line
 	2850 2150 3100 2150
@@
 5V
 Wire Wire Line
-	1950 1350 3050 1350
+	1950 1350 2200 1350
 Connection ~ 2600 1350
 Connection ~ 2200 1350
+Wire Wire Line
+	2600 3100 3100 3100
+Wire Wire Line
+	2200 2050 2200 2800
+Wire Wire Line
+	2600 2250 2600 2800
+Wire Wire Line
+	2600 1350 3050 1350
+Wire Wire Line
+	2200 1350 2600 1350
 $EndSCHEMATC
