File: HW/projects/fennek_2017_18/BMS/measurement_and_balancing/bms_board_V6__12s_fennek2017/bms_board.sch (KiCad schematic (older format))
At the start: 11 parts, among them P1 Battery_Interface, P2 TS1, P3 TS2

Commit message: Update github repo with designs for fennek 2018
Parts:
- C16, C17, C51: symbol C_Small -> Device:C_Small
- P1: symbol CONN_01X13 -> Connector_Generic:Conn_01x13
- P2, P3: symbol CONN_01X02 -> Connector_Generic:Conn_01x02
- R10, R11, R5, R8, R9: symbol R_Small -> Device:R_Small
Changed lines of the file:
@@
-EESchema Schematic File Version 2
-LIBS:power
-LIBS:device
-LIBS:transistors
-LIBS:conn
-LIBS:linear
-LIBS:regul
-LIBS:74xx
-LIBS:cmos4000
-LIBS:adc-dac
-LIBS:memory
-LIBS:xilinx
-LIBS:microcontrollers
-LIBS:dsp
-LIBS:microchip
-LIBS:analog_switches
-LIBS:motorola
-LIBS:texas
-LIBS:intel
-LIBS:audio
-LIBS:interface
-LIBS:digital-audio
-LIBS:philips
-LIBS:display
-LIBS:cypress
-LIBS:siliconi
-LIBS:opto
-LIBS:atmel
-LIBS:contrib
-LIBS:valves
-LIBS:relais
-LIBS:Supply
-LIBS:tera_general
-LIBS:tera_logic
-LIBS:tera_processors
-LIBS:tera_switches
-LIBS:local_power
-LIBS:ft232rl
-LIBS:tera_connectors
-LIBS:tera_emc_prodection
+EESchema Schematic File Version 4
 LIBS:bms_board-cache
-EELAYER 25 0
+EELAYER 26 0
 EELAYER END
 $Descr A4 11693 8268
@@
 $EndDescr
 $Comp
-L R_Small R5
+L Device:R_Small R5
 U 1 1 56ED75BD
 P 9100 4750
@@
 $EndSheet
 $Comp
-L +5V #PWR01
+L power:+5V #PWR01
 U 1 1 58667247
 P 3850 2100
@@
 $EndComp
 $Comp
-L GND #PWR02
+L power:GND #PWR02
 U 1 1 5879171A
 P 3900 4650
@@
 $EndSheet
 $Comp
-L +5V #PWR03
+L power:+5V #PWR03
 U 1 1 58876F92
 P 3250 3400
@@
 	3100 4400 4000 4400
 $Comp
-L GND #PWR04
+L power:GND #PWR04
 U 1 1 5887E1A7
 P 3350 4650
@@
 	5050 3050 5550 3050
 $Comp
-L GND #PWR05
+L power:GND #PWR05
 U 1 1 5888DC46
 P 5400 2100
@@
 	5400 2100 5550 2100
 $Comp
-L Vmiddle #PWR06
+L local_power:Vmiddle #PWR06
 U 1 1 58893F4C
 P 5350 1950
@@
 	6900 3050 7700 3050
 $Comp
-L Vmiddle #PWR07
+L local_power:Vmiddle #PWR07
 U 1 1 588A8C1E
 P 5300 3900
@@
 	5300 4000 5050 4000
 $Comp
-L Vmiddle #PWR08
+L local_power:Vmiddle #PWR08
 U 1 1 588AA79D
 P 7550 4700
@@
 	6850 4000 7700 4000
 $Comp
-L +BATT #PWR09
+L power:+BATT #PWR09
 U 1 1 588BC192
 P 9050 2200
@@
 $EndComp
 Wire Wire Line
-	9050 2200 9050 3050
+	9050 2200 9050 2300
 Wire Wire Line
 	9050 3050 8850 3050
@@
 Connection ~ 9050 2300
 $Comp
-L GND #PWR010
+L power:GND #PWR010
 U 1 1 588C4DFF
 P 3850 3150
@@
 $EndComp
 Wire Wire Line
-	3850 2300 3850 3150
+	3850 2300 3850 2400
 Wire Wire Line
 	3850 2300 4000 2300
@@
 Connection ~ 3850 3050
 $Comp
-L CONN_01X13 P1
+L Connector_Generic:Conn_01x13 P1
 U 1 1 588D77C9
 P 6250 5250
@@
 $EndComp
 $Comp
-L GND #PWR011
+L power:GND #PWR011
 U 1 1 588DB998
 P 5450 5150
@@
 $EndComp
 Wire Wire Line
-	5450 4950 5450 5150
+	5450 4950 5450 5000
 Wire Wire Line
 	5450 5000 5650 5000
 Wire Wire Line
-	5650 4600 5650 5050
-$Comp
-L +BATT #PWR012
+	5650 4600 5650 5000
+$Comp
+L power:+BATT #PWR012
 U 1 1 588DD065
 P 7150 5000
@@
 $EndComp
 Wire Wire Line
-	6850 4000 6850 5050
-Wire Wire Line
-	6850 5000 7150 5000
-$Comp
-L Vmiddle #PWR013
+	6850 4000 6850 5000
+Wire Wire Line
+	6850 5000 6950 5000
+$Comp
+L local_power:Vmiddle #PWR013
 U 1 1 588E152C
 P 6250 3900
@@
 $EndComp
 Wire Wire Line
-	6250 3900 6250 5050
+	6250 3900 6250 4000
 Connection ~ 5650 5000
 Wire Wire Line
@@
 5V_C2
 $Comp
-L PWR_FLAG #FLG014
+L power:PWR_FLAG #FLG014
 U 1 1 589514D9
 P 5450 4950
@@
 Connection ~ 5450 5000
 $Comp
-L PWR_FLAG #FLG015
+L power:PWR_FLAG #FLG015
 U 1 1 589547FF
 P 6950 5000
@@
 Connection ~ 6950 5000
 $Comp
-L PWR_FLAG #FLG016
+L power:PWR_FLAG #FLG016
 U 1 1 58965E29
 P 6250 4000
@@
 Connection ~ 6250 4000
 $Comp
-L CONN_01X02 P2
+L Connector_Generic:Conn_01x02 P2
 U 1 1 585A2812
-P 2850 5300
-F 0 "P2" H 3050 5250 50  0000 C CNN
-F 1 "TS1" H 3000 5150 50  0000 C CNN
-F 2 "tera_Connectors_Molex:Molex_PicoBlade_53261-0271_02x1.25mm_Angled" H 2850 5300 50  0001 C CNN
-F 3 "" H 2850 5300 50  0000 C CNN
-F 4 "03-0202" H 2850 5300 60  0001 C CNN "HPN"
-	1    2850 5300
+P 2850 5350
+F 0 "P2" H 3050 5300 50  0000 C CNN
+F 1 "TS1" H 3000 5200 50  0000 C CNN
+F 2 "tera_Connectors_Molex:Molex_PicoBlade_53261-0271_02x1.25mm_Angled" H 2850 5350 50  0001 C CNN
+F 3 "" H 2850 5350 50  0000 C CNN
+F 4 "03-0202" H 2850 5350 60  0001 C CNN "HPN"
+	1    2850 5350
 	-1   0    0    1
 $EndComp
 $Comp
-L C_Small C16
+L Device:C_Small C16
 U 1 1 585A2819
 P 3550 5250
@@
 $EndComp
 $Comp
-L R_Small R8
+L Device:R_Small R8
 U 1 1 585A2820
 P 3200 5350
@@
 $EndComp
 $Comp
-L R_Small R9
+L Device:R_Small R9
 U 1 1 585A2827
 P 3550 5450
@@
 $EndComp
 $Comp
-L CONN_01X02 P3
+L Connector_Generic:Conn_01x02 P3
 U 1 1 585A282E
-P 9950 5700
-F 0 "P3" H 10150 5650 50  0000 C CNN
-F 1 "TS2" H 10100 5550 50  0000 C CNN
-F 2 "tera_Connectors_Molex:Molex_PicoBlade_53261-0271_02x1.25mm_Angled" H 9950 5700 50  0001 C CNN
-F 3 "" H 9950 5700 50  0000 C CNN
-F 4 "03-0202" H 9950 5700 60  0001 C CNN "HPN"
-	1    9950 5700
+P 9950 5750
+F 0 "P3" H 10150 5700 50  0000 C CNN
+F 1 "TS2" H 10100 5600 50  0000 C CNN
+F 2 "tera_Connectors_Molex:Molex_PicoBlade_53261-0271_02x1.25mm_Angled" H 9950 5750 50  0001 C CNN
+F 3 "" H 9950 5750 50  0000 C CNN
+F 4 "03-0202" H 9950 5750 60  0001 C CNN "HPN"
+	1    9950 5750
 	1    0    0    1
 $EndComp
 $Comp
-L C_Small C17
+L Device:C_Small C17
 U 1 1 585A2835
 P 9250 5650
@@
 $EndComp
 $Comp
-L R_Small R11
+L Device:R_Small R11
 U 1 1 585A283C
 P 9600 5750
@@
 $EndComp
 $Comp
-L R_Small R10
+L Device:R_Small R10
 U 1 1 585A2843
 P 9250 5850
@@
 	3100 5250 3050 5250
 Wire Wire Line
-	3100 5100 3100 5250
+	3100 5100 3100 5150
 Wire Wire Line
 	3100 5150 3550 5150
@@
 Connection ~ 3550 5350
 Wire Wire Line
-	3300 5350 4000 5350
+	3300 5350 3550 5350
 Wire Wire Line
 	3550 5550 4000 5550
@@
 	9700 5650 9750 5650
 Wire Wire Line
-	9700 5450 9700 5650
+	9700 5450 9700 5550
 Wire Wire Line
 	9700 5550 9250 5550
@@
 Connection ~ 9250 5750
 Wire Wire Line
-	8850 5750 9500 5750
+	8850 5750 9250 5750
 Wire Wire Line
 	8850 5950 9250 5950
 $Comp
-L +5V #PWR017
+L power:+5V #PWR017
 U 1 1 585E9C2D
 P 3100 5100
@@
 5V_C2
 $Comp
-L C_Small C51
+L Device:C_Small C51
 U 1 1 58677B6B
 P 6000 5850
@@
 $EndComp
 $Comp
-L GND #PWR018
+L power:GND #PWR018
 U 1 1 5867DDC7
 P 5900 5850
@@
 $EndComp
 $Comp
-L Vmiddle #PWR019
+L local_power:Vmiddle #PWR019
 U 1 1 5868539B
 P 6100 5850
@@
 	0    1    1    0
 $EndComp
+Wire Wire Line
+	9050 2950 9050 3050
+Wire Wire Line
+	9050 2850 9050 2950
+Wire Wire Line
+	9050 2750 9050 2850
+Wire Wire Line
+	9050 2600 9050 2750
+Wire Wire Line
+	9050 2500 9050 2600
+Wire Wire Line
+	9050 2400 9050 2500
+Wire Wire Line
+	9050 2300 9050 2400
+Wire Wire Line
+	3850 2400 3850 2500
+Wire Wire Line
+	3850 2500 3850 2600
+Wire Wire Line
+	3850 2600 3850 2750
+Wire Wire Line
+	3850 2750 3850 2850
+Wire Wire Line
+	3850 2850 3850 2950
+Wire Wire Line
+	3850 2950 3850 3050
+Wire Wire Line
+	3850 3050 3850 3150
+Wire Wire Line
+	5650 5000 5650 5050
+Wire Wire Line
+	6850 5000 6850 5050
+Wire Wire Line
+	5450 5000 5450 5150
+Wire Wire Line
+	6950 5000 7150 5000
+Wire Wire Line
+	6250 4000 6250 5050
+Wire Wire Line
+	3100 5150 3100 5250
+Wire Wire Line
+	3550 5350 4000 5350
+Wire Wire Line
+	9700 5550 9700 5650
+Wire Wire Line
+	9250 5750 9500 5750
 $EndSCHEMATC
