File: HW/projects/fennek_2017_18/BMS/power_distribution/fennek_power_distribution_v1/fennek_power_distribution.kicad_pcb (KiCad board)
At the start: 4 copper layers, 115.5 x 65 mm, 95 parts, among them IC1 ACS722LLCTR-20AB-T, IC2 ACS722LLCTR-20AB-T, K1 SPDT-16A_12VDC-Coil, K2 SPDT-16A_12VDC-Coil, P1 HV_in, P10 Precharge_relays, P11 Main_relay, P12 Main_relay_coil, P13 SEM_telemetry_supply, P2 12V_relays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

Commit message: Update github repo with designs for fennek 2018
Parts:
- F2: value 2.5A 12VDC -> 3A 12VDC
- R1, R11: value 100R, 250mW -> 100R 250mW
- R12: value 10R, 500mW -> 10R 500mW
- R13, R14: value 22R, 2W -> 22R 2W
- R2: value 470R, 5W -> 470R 5W
- U1: value TEN_30-4812_single_output -> TEN_30-4812WIN_single_output
Changed lines of the file:
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@@
-(kicad_pcb (version 4) (host pcbnew no-vcs-found-product)
+(kicad_pcb (version 20171130) (host pcbnew 6.0.0-rc1-unknown-r13685-202b35bc)
   (general
-    (links 166)
-    (no_connects 0)
-    (area 66.924999 56.924999 182.575001 122.075001)
     (thickness 1.6)
     (drawings 38)
@@
     (zone_45_only no)
     (trace_min 0.2)
-    (segment_width 0.2)
-    (edge_width 0.15)
     (via_size 0.75)
     (via_drill 0.3)
@@
     (uvia_min_size 0.2)
     (uvia_min_drill 0.1)
+    (edge_width 0.15)
+    (segment_width 0.2)
     (pcb_text_width 0.3)
     (pcb_text_size 1.5 1.5)
@@
       (layerselection 0x010f0_ffffffff)
       (usegerberextensions false)
+      (usegerberattributes false)
+      (usegerberadvancedattributes false)
+      (creategerberjobfile false)
       (excludeedgelayer true)
       (linewidth 0.100000)
@@
       (hpglpennumber 1)
       (hpglpenspeed 20)
-      (hpglpendiameter 15)
+      (hpglpendiameter 15.000000)
       (psnegative false)
       (psa4output false)
@@
       (drillshape 0)
       (scaleselection 1)
-      (outputdirectory gerber/))
+      (outputdirectory "gerber/"))
   )
   (net 0 "")
@@
       (effects (font (size 1 1) (thickness 0.15)) (justify mirror))
     )
-    (fp_text value "22R, 2W" (at 0 -1 90) (layer B.Fab)
+    (fp_text value "22R 2W" (at 0 -1 90) (layer B.Fab)
       (effects (font (size 0.6 0.6) (thickness 0.1)) (justify mirror))
     )
@@
       (effects (font (size 1 1) (thickness 0.15)) (justify mirror))
     )
-    (fp_text value "22R, 2W" (at 0 -1 270) (layer B.Fab)
+    (fp_text value "22R 2W" (at 0 -1 270) (layer B.Fab)
       (effects (font (size 0.6 0.6) (thickness 0.1)) (justify mirror))
     )
@@
       (effects (font (size 0.75 0.75) (thickness 0.12)))
     )
-    (fp_text value "10R, 500mW" (at 0.25 1.75 270) (layer F.Fab)
+    (fp_text value "10R 500mW" (at 0.25 1.75 270) (layer F.Fab)
       (effects (font (size 0.6 0.6) (thickness 0.1)))
     )
@@
       (effects (font (size 0.75 0.75) (thickness 0.12)))
     )
-    (fp_text value "100R, 250mW" (at 0 1.75 180) (layer F.Fab)
+    (fp_text value "100R 250mW" (at 0 1.75 180) (layer F.Fab)
       (effects (font (size 0.75 0.75) (thickness 0.12)))
     )
@@
       (effects (font (size 0.75 0.75) (thickness 0.12)) (justify mirror))
     )
-    (fp_text value "100R, 250mW" (at 0 -1.75 180) (layer B.Fab)
+    (fp_text value "100R 250mW" (at 0 -1.75 180) (layer B.Fab)
       (effects (font (size 0.75 0.75) (thickness 0.12)) (justify mirror))
     )
@@
       (effects (font (size 1 1) (thickness 0.15)))
     )
-    (fp_text value "2.5A 12VDC" (at 4.75 3.5) (layer F.Fab)
+    (fp_text value "3A 12VDC" (at 4.75 3.5) (layer F.Fab)
       (effects (font (size 1 1) (thickness 0.15)))
     )
@@
       (effects (font (size 1 1) (thickness 0.15)))
     )
-    (fp_text value TEN_30-4812_single_output (at 8.62 22.86 180) (layer F.Fab)
+    (fp_text value TEN_30-4812WIN_single_output (at 8.62 22.86 180) (layer F.Fab)
       (effects (font (size 1 1) (thickness 0.15)))
     )
@@
       (effects (font (size 1 1) (thickness 0.15)))
     )
-    (fp_text value "470R, 5W" (at 0 1 180) (layer F.Fab)
+    (fp_text value "470R 5W" (at 0 1 180) (layer F.Fab)
       (effects (font (size 1 1) (thickness 0.15)))
     )
@@
     (attr smd)
     (fp_text reference svg2mod (at 0 -5.714667) (layer F.SilkS) hide
-      (effects (font (thickness 0.3048)))
+      (effects (font (size 1.524 1.524) (thickness 0.3048)))
     )
     (fp_text value G*** (at 0 5.714667) (layer F.SilkS) hide
-      (effects (font (thickness 0.3048)))
+      (effects (font (size 1.524 1.524) (thickness 0.3048)))
     )
     (fp_poly (pts (xy -0.000023 -2.666667) (xy -0.000023 -2.400911) (xy 0.040353 -2.400866) (xy 0.080672 -2.400733)
@@
     (attr smd)
     (fp_text reference svg2mod (at 0 7.048 180) (layer B.SilkS) hide
-      (effects (font (thickness 0.3048)) (justify mirror))
+      (effects (font (size 1.524 1.524) (thickness 0.3048)) (justify mirror))
     )
     (fp_text value G*** (at 0 -7.048 180) (layer B.SilkS) hide
-      (effects (font (thickness 0.3048)) (justify mirror))
+      (effects (font (size 1.524 1.524) (thickness 0.3048)) (justify mirror))
     )
     (fp_poly (pts (xy -0.000034 4) (xy -0.000034 3.601367) (xy 0.060529 3.6013) (xy 0.121008 3.6011)
@@
     (fp_line (start 1.95 2.45) (end 1.95 -2.45) (layer B.Fab) (width 0.05))
     (fp_line (start -1.95 2.45) (end 1.95 2.45) (layer B.Fab) (width 0.05))
-    (fp_text user %R (at -0.3 0.2 540) (layer B.Fab)
+    (fp_text user %R (at -0.3 0.2 180) (layer B.Fab)
       (effects (font (size 1 1) (thickness 0.15)) (justify mirror))
     )
