File: HW/projects/fennek_2017_18/BMS/power_distribution/fennek_power_distribution_v1/fennek_power_distribution.sch (KiCad schematic (older format))
At the start: 61 parts, among them IC1 ACS722LLCTR-20AB-T, IC2 ACS722LLCTR-20AB-T, K1 SPDT-16A_12VDC-Coil, K2 SPDT-16A_12VDC-Coil, P1 HV_in, P10 Precharge_relays, P11 Main_relay, P12 Main_relay_coil, P13 SEM_telemetry_supply, P2 12V_relays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

Commit message: Update github repo with designs for fennek 2018
Parts:
- C1, C2: symbol C_Small -> Device:C_Small
- C3: symbol CP_Small -> Device:CP_Small
- D1, D12, D4: symbol ZENERsmall -> fennek_power_distribution-rescue:ZENERsmall
- D10, D11, D13, D2, D3, D9: symbol D_Small -> Device:D_Small
- D5, D6, D7, D8: symbol Led_Small -> Device:LED_Small
- F1, F2, F3, F4, F5, F6, F7: symbol F_Small -> Device:Fuse_Small
- IC1, IC2: symbol ACS722LLCTR-20AB-T -> tera_sensoric:ACS722LLCTR-20AB-T
- JP1: symbol JUMPER3_NO -> tera_general:JUMPER3_NO
- K1, K2: symbol Finder-41.61.9.012.0010_SPDT-16A_12VDC-Coil -> relais:Finder-41.61.9.012.0010_SPDT-16A_12VDC-Coil
- P1, P3, P5: symbol CONN_01X03 -> Connector_Generic:Conn_01x03
- P10, P11, P2, P4, P7: symbol CONN_01X04 -> Connector_Generic:Conn_01x04
- P12, P13, P6, P8, P9: symbol CONN_01X02 -> Connector_Generic:Conn_01x02
- Q1, Q2, Q3, Q4: symbol IRLML2246TRPBF-1 -> tera_general:IRLML2246TRPBF-1
- R1, R10, R11, R12, R13, R14, R2, R3, R4, R5, R6, R7, R8, R9: symbol R_Small -> Device:R_Small
- U1: symbol TEN_30-xxxx_single_output -> Supply:TEN_30-xxxx_single_output
- U2: symbol THD_12-xxxx_single_output -> fennek_power_distribution-rescue:THD_12-xxxx_single_output
