File: HW/projects/fennek_2017_18/BMS/power_distribution/fennek_power_distribution_v2/HV_distribution.sch (KiCad schematic (older format))
At the start: 21 parts, among them IC1 ACS722LLCTR-20AB-T, IC2 ACS722LLCTR-20AB-T, K1 SPDT-16A_12VDC-Coil, K3 ASSR-1218, P1 HV_in, P12 Main_relay_coil, P4 HV_Emergency_Stop_Relay, P6 MCU_HV_supply

Commit message: Update github repo with designs for fennek 2018
Parts:
- removed K1: SPDT-16A_12VDC-Coil, tera_relais:Finder-41.61.9.012.0010_SPDT-16A_12VDC-Coil, symbol Finder-41.61.9.012.0010_SPDT-16A_12VDC-Coil
- added F2: 1A 63VDC, tera_general:Fuse_1206_3216Metric_Pad1.24x1.80mm_HandSolder, symbol Device:Fuse_Small
- added JP3: Jumper_NO_Small, tera_general:SOLDERJUMPER_2_3mm_HV, symbol Device:Jumper_NO_Small
- added K1: TE_OJ-SH-112DM, tera_relais:RELAIS-TE-OJ, symbol relais:TE_OJ-SH-112DM_MU
- added P7: Horn, tera_Connectors_JST:JST_XH_S02B-XH-A_02x2.50mm_Angled, symbol Connector_Generic:Conn_01x02
- C2, C4: symbol C_Small -> Device:C_Small
- C3: symbol CP_Small -> Device:CP_Small
- D1: symbol ZENERsmall -> Device:D_Zener_Small
- D11, D13: symbol D_Small -> Device:D_Small
- F1: symbol F_Small -> Device:Fuse_Small
- IC1, IC2: symbol ACS722LLCTR-20AB-T -> tera_sensoric:ACS722LLCTR-20AB-T
- K3: symbol ASSR-1218 -> relais:ASSR-1218
- P1: symbol CONN_01X03 -> Connector_Generic:Conn_01x03
- P12: symbol CONN_01X02 -> Connector_Generic:Conn_01x02; HPN 02-???? -> 02-1002
- P4: symbol CONN_01X04 -> Connector_Generic:Conn_01x04
- P6: symbol CONN_01X02 -> Connector_Generic:Conn_01x02
- R11: value 510R 250mW -> 180R; symbol R_Small -> Device:R_Small; HPN 13-510R -> 11-180R
- R12, R13, R14, R2: symbol R_Small -> Device:R_Small
- R17: symbol R -> Device:R
Connections:
- net +12VDC_switched: now also K1.A1
- net -VBatt: now also P7.1 (Pin_1)
- net HV+_after_main_relais: now also JP3.1, K1.11
- net VBatt_Switched: now also F2.1, JP3.2, K1.14
- net Main_Relay_A1: now reaches D13.1 (K), K3.4, P12.2 (Pin_2)
- net LowSideSwitch_MainRelay/CHANNEL1 renamed Main_Relay_A2
- net LowSideSwitch_PreCharge/CHANNEL1 renamed PreCharger_A2
- net PreCharger_A2: now also K1.A2
- new net V+_Horn: F2.2, P7.2 (Pin_2)
- no-connect marks 3 -> 1
Other:
- note added: "Coil info: 12VDC (Hold = 9VDC), 720 Ohm, 200mW"
- note added: "Holding voltage: 9V\n=> R11 max = 240R"
- note added: "Time constands:\nTurn on: 5tau=180ms\nTurn off: tau= 626ms (Relay coil in series!)"
- note removed: "Coil info: 12VDC, 0.36W => 400 Ohm, 30mA"
- note removed: "Holding voltage: 0.4 Un \n=> R11 max = 600 Ohm"
- note removed: "Time constands:\nTurn on: 5tau=180ms\nTurn off: tau= 360ms (Relay coil in series!)"
