File: HW/projects/fennek_2017_18/BMS/power_distribution/fennek_power_distribution_v2/fennek_power_distribution.kicad_pcb (KiCad board)
At the start: 4 copper layers, 134 x 58.5 mm, 144 parts, among them IC1 ACS722LLCTR-20AB-T, IC2 ACS722LLCTR-20AB-T, IC3 TLE8102SG, IC4 TLE8102SG, IC5 TLE8102SG, K1 SPDT-16A_12VDC-Coil, K2 SPDT-16A_12VDC-Coil, K3 ASSR-1218, K4 Panasonic_AQY414S, K5 Panasonic_AQY414S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

Commit message: Update github repo with designs for fennek 2018
Parts:
- removed K5: Panasonic_AQY414S, tera_general:SO-4
- removed R23: 1k, tera_rlc:R_0603in
- removed the REF** at (89.4, 98.5)
- removed the REF** at (87.8, 101.5)
- removed the REF** at (89.4, 101.5)
- removed the REF** at (87.8, 98.5)
- removed the REF** at (88.2, 94.2)
- removed the REF** at (89.3, 95.4)
- removed the REF** at (90.7, 91.8)
- removed the REF** at (91.8, 92.9)
- removed the REF** at (93.1, 89.3)
- removed the REF** at (94.2, 90.5)
- removed the REF** at (95.4, 87.0)
- removed the REF** at (96.5, 88.2)
- removed the REF** at (99.5, 85.2)
- removed the REF** at (96.9, 91.0)
- removed the REF** at (94.7, 93.2)
- removed the REF** at (91.7, 96.2)
- added F2: 1A 63VDC, tera_general:Fuse_1206_3216Metric_Pad1.24x1.80mm_HandSolder, F.Cu at (103.8, 71.2)
- added P7: Horn, tera_Connectors_JST:JST_XH_S02B-XH-A_02x2.50mm_Angled, F.Cu at (105.5, 66.0)
- added REF**: Via-0.4, local_footprints:Via-0.4, F.Cu at (152.8, 104.8)
- added REF**: Via-0.2, local_footprints:Via-0.2, F.Cu at (99.8, 91.5)
- added REF**: Via-0.2, local_footprints:Via-0.2, F.Cu at (98.5, 92.0)
- added REF**: Via-0.2, local_footprints:Via-0.2, F.Cu at (99.5, 93.0)
- added REF**: Via-0.2, local_footprints:Via-0.2, F.Cu at (96.0, 94.5)
- added REF**: Via-0.2, local_footprints:Via-0.2, F.Cu at (97.0, 95.5)
- added REF**: Via-0.2, local_footprints:Via-0.2, F.Cu at (93.5, 97.0)
- added REF**: Via-0.2, local_footprints:Via-0.2, F.Cu at (94.5, 98.0)
- added REF**: Via-0.2, local_footprints:Via-0.2, F.Cu at (92.0, 100.5)
- added REF**: Via-0.2, local_footprints:Via-0.2, F.Cu at (91.0, 99.5)
- added REF**: Via-0.2, local_footprints:Via-0.2, F.Cu at (88.5, 102.0)
- added REF**: Via-0.4, local_footprints:Via-0.4, F.Cu at (150.5, 104.8)
- added REF**: Via-0.2, local_footprints:Via-0.2, F.Cu at (87.8, 103.5)
- added REF**: Via-0.2, local_footprints:Via-0.2, F.Cu at (89.2, 103.2)
- added REF**: Via-0.4, local_footprints:Via-0.4, F.Cu at (99.8, 70.0)
- added REF**: Via-0.2, local_footprints:Via-0.2, F.Cu at (102.0, 87.0)
- added REF**: Via-0.2, local_footprints:Via-0.2, F.Cu at (102.0, 89.0)
- added REF**: Via-0.2, local_footprints:Via-0.2, F.Cu at (98.5, 86.8)
- added REF**: Via-0.2, local_footprints:Via-0.2, F.Cu at (99.8, 86.2)
- added REF**: Via-0.2, local_footprints:Via-0.2, F.Cu at (98.5, 89.0)
- added REF**: Via-0.2, local_footprints:Via-0.2, F.Cu at (99.8, 88.5)
- D5, R18, R19, R20, R21: moved to B.Cu
- F7: footprint tera_general:Fuse_Phoenix_SI-H-FKS_15 -> tera_general:Fuse_0805_2012Metric_Pad1.15x1.50mm_HandSolder
- JP3: footprint tera_general:SOLDERJUMPER_2_1mm -> tera_general:SOLDERJUMPER_2_3mm_HV
- K1, K2: value SPDT-16A_12VDC-Coil -> TE_OJ-SH-112DM; footprint tera_relais:Finder-41.61.9.012.0010_SPDT-16A_12VDC-Coil -> tera_relais:RELAIS-TE-OJ
- P13: footprint tera_Connectors_Phoenix:PhoenixContact_MC-GF_02x3.50mm_Angled_ThreadedFlange -> tera_Connectors_JST:JST_XH_S02B-XH-A_02x2.50mm_Angled; moved to F.Cu
- R1, R11: value 510R 250mW -> 180R
- R2: moved to F.Cu
- moved D20 32.0 mm to (104.6, 93.8), turned to 0 degrees
- moved R21 27.7 mm to (106.4, 91.5), turned to 180 degrees
- moved REF** 27.2 mm to (83.5, 71.5)
- moved JP3 25.5 mm to (107.9, 72.8), turned to 270 degrees
- moved D19 24.5 mm to (110.8, 93.7), turned to 180 degrees
- moved D22 24.3 mm to (102.2, 93.8)
- moved REF** 23.4 mm to (91.8, 76.0)
- moved R11 23.3 mm to (105.2, 91.3)
- moved D11 22.8 mm to (107.7, 88.3), turned to 180 degrees
- moved R20 22.5 mm to (110.5, 91.5)
- moved REF** 21.6 mm to (92.8, 74.5)
- moved K1 20.3 mm to (107.8, 82.0), turned to 90 degrees
- moved REF** 19.8 mm to (95.0, 77.5)
- moved R18 19.7 mm to (138.2, 59.4)
- moved R19 19.4 mm to (136.1, 60.5)
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Connections:
- net /High voltage/LowSideSwitch_MainRelay/CHANNEL1 renamed /High voltage/Main_Relay_A2
- net Net-(D13-Pad1) renamed /High voltage/Main_Relay_A1
- net Net-(JP2-Pad1) renamed /12VDC Bordnet/BN_on
- net Net-(K4-Pad4) renamed /12VDC Bordnet/BN_IL
- C3 pad 2: /High voltage/LowSideSwitch_PreCharge/CHANNEL1 -> /High voltage/PreCharger_A2
- D11 pad 2: /High voltage/LowSideSwitch_PreCharge/CHANNEL1 -> /High voltage/PreCharger_A2
- D21 pad 2: /High voltage/LowSideSwitch_PreCharge/CHANNEL1 -> /High voltage/PreCharger_A2
- JP3 pad 1: Net-(JP3-Pad1) -> /High voltage/HV+_after_main_relais
- JP3 pad 2: Net-(JP3-Pad2) -> /High voltage/VBatt_Switched
- K3 pad 2: /12VDC telemetry/IL_next- -> /Master Connector/IL_master-
- R11 pad 1: /High voltage/LowSideSwitch_PreCharge/CHANNEL1 -> /High voltage/PreCharger_A2
- R17 pad 1: /12VDC telemetry/IL_next- -> /Master Connector/IL_master-
- U2 pad 1: Net-(JP3-Pad1) -> Net-(U2-Pad1)
Routing:
- net Net-(D20-Pad1): track 44.5 -> 9.18 mm, vias 3 -> 1
- net Net-(JP3-Pad2): track 28.3 -> 0.00 mm
- net Net-(D19-Pad1): track 38.8 -> 10.5 mm
- net /Master Connector/+12VDC_BMS_Switched: track 10.9 -> 36.5 mm, vias 5 -> 3
- net /High voltage/LowSideSwitch_PreCharge/CHANNEL1: track 21.4 -> 0.00 mm, vias 1 -> 0
- net /High voltage/PreCharger_A2: track 0.00 -> 20.8 mm, vias 0 -> 1
- net /Master Connector/+12VDC_BMS: track 113.4 -> 93.1 mm, vias 1 -> 2
- net /12VDC telemetry/IL_next-: track 19.7 -> 0.00 mm, vias 1 -> 0
- net Net-(D15-Pad2): track 22.3 -> 4.25 mm, vias 1 -> 0
- net Net-(D16-Pad2): track 20.4 -> 5.51 mm, vias 1 -> 0
- net /Master Connector/IL_master-: track 28.7 -> 42.8 mm, vias 0 -> 1
- net Net-(D9-Pad2): track 13.2 -> 0.99 mm
- net Net-(D4-Pad2): track 11.9 -> 0.99 mm
- net /12VDC Bordnet/+12VDC: track 9.68 -> 0.00 mm
- net /12VDC telemetry/+12V_telemetry: track 0.00 -> 6.27 mm
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- added copper zone on In1.Cu, net /High voltage/+HV_in
- added copper zone on F.Cu, net /Master Connector/+12VDC_BMS
- removed copper zone on F.Cu, net /12VDC telemetry/+12V_telemetry
Other:
- board text added: "Horn (50V/1A)"
- board text added: "Shell Bord- computer (12V/1A)"
- board text removed: "Shell Bordcomputer"
