File: HW/projects/fennek_2017_18/BMS/power_distribution/fennek_power_distribution_v2/master_connector.sch (KiCad schematic (older format))
At the start: 4 parts, among them P3 CONN_02X22

Commit message: Update github repo with designs for fennek 2018
Parts:
- C7, C8, C9: symbol C_Small -> Device:C_Small
- P3: symbol CONN_02X22 -> Connector_Generic:Conn_02x22_Odd_Even
Changed lines of the file:
@@
-EESchema Schematic File Version 2
-LIBS:power
-LIBS:device
-LIBS:transistors
-LIBS:conn
-LIBS:linear
-LIBS:regul
-LIBS:74xx
-LIBS:cmos4000
-LIBS:adc-dac
-LIBS:memory
-LIBS:xilinx
-LIBS:microcontrollers
-LIBS:dsp
-LIBS:microchip
-LIBS:analog_switches
-LIBS:motorola
-LIBS:texas
-LIBS:intel
-LIBS:audio
-LIBS:interface
-LIBS:digital-audio
-LIBS:philips
-LIBS:display
-LIBS:cypress
-LIBS:siliconi
-LIBS:opto
-LIBS:atmel
-LIBS:contrib
-LIBS:valves
-LIBS:local_power
-LIBS:ft232rl
-LIBS:relais
-LIBS:Supply
-LIBS:tera_connectors
-LIBS:tera_emc_prodection
-LIBS:tera_general
-LIBS:tera_logic
-LIBS:tera_processors
-LIBS:tera_switches
-LIBS:tera_sensoric
+EESchema Schematic File Version 4
 LIBS:fennek_power_distribution-cache
-EELAYER 25 0
+EELAYER 26 0
 EELAYER END
 $Descr A4 11693 8268
@@
 $EndDescr
 Wire Wire Line
-	3600 2250 3750 2250
-Wire Wire Line
-	3650 2150 3650 2350
-$Comp
-L C_Small C7
+	3600 2250 3650 2250
+Wire Wire Line
+	3650 2150 3650 2250
+$Comp
+L Device:C_Small C7
 U 1 1 593789CD
 P 5900 2250
@@
 	5750 2250 5750 2150
 Wire Wire Line
-	4250 2250 5800 2250
+	4250 2250 5600 2250
 Connection ~ 5750 2250
 $Comp
-L C_Small C8
+L Device:C_Small C8
 U 1 1 593789DF
 P 5900 2950
@@
 $EndComp
 $Comp
-L PWR_FLAG #FLG012
+L power:PWR_FLAG #FLG012
 U 1 1 593789F0
 P 5600 2150
@@
 Connection ~ 5600 2250
 $Comp
-L PWR_FLAG #FLG013
+L power:PWR_FLAG #FLG013
 U 1 1 593789F8
 P 5600 2850
@@
 	4400 2350 4250 2350
 Wire Wire Line
-	3650 3850 3650 4250
+	3650 3850 3650 3950
 Wire Wire Line
 	3650 4250 3750 4250
@@
 Interlock_OK
 Wire Wire Line
-	3600 4050 3750 4050
+	3600 4050 3650 4050
 Wire Wire Line
 	3650 3150 3750 3150
@@
 SPI_MISO
 Wire Wire Line
-	3600 2750 3750 2750
+	3600 2750 3650 2750
 Wire Wire Line
 	3650 2850 3750 2850
@@
 	5600 2850 5600 2950
 Wire Wire Line
-	4250 2950 5800 2950
+	4250 2950 5600 2950
 Wire Wire Line
 	5750 2950 5750 2850
@@
 	4400 3850 4250 3850
 $Comp
-L CONN_02X22 P3
+L Connector_Generic:Conn_02x22_Odd_Even P3
 U 1 1 5937F738
-P 4000 3200
-F 0 "P3" H 4000 4465 50  0000 C CNN
-F 1 "CONN_02X22" H 4000 4374 50  0000 C CNN
-F 2 "tera_Connectors_other:ESW-122-12-L-D" H 4000 2300 50  0001 C CNN
-F 3 "" H 4000 2300 50  0000 C CNN
-	1    4000 3200
+P 3950 3250
+F 0 "P3" H 3950 4515 50  0000 C CNN
+F 1 "CONN_02X22" H 3950 4424 50  0000 C CNN
+F 2 "tera_Connectors_other:ESW-122-12-L-D" H 3950 2350 50  0001 C CNN
+F 3 "" H 3950 2350 50  0000 C CNN
+	1    3950 3250
 	1    0    0    1
 $EndComp
@@
 	3650 3250 3750 3250
 $Comp
-L C_Small C9
+L Device:C_Small C9
 U 1 1 5933A614
 P 5900 4050
@@
 	5750 3950 5750 4050
 Wire Wire Line
-	4250 4050 5800 4050
+	4250 4050 5750 4050
 Connection ~ 5750 4050
 Text HLabel 5750 3950 1    50   Output ~ 0
@@
 	3750 4150 3650 4150
 Wire Wire Line
-	3650 2550 3650 2850
+	3650 2550 3650 2650
 Wire Wire Line
 	3650 3650 3750 3650
 Wire Wire Line
-	3650 2950 3650 3250
+	3650 2950 3650 3050
 Text HLabel 3650 3650 0    60   Input ~ 0
 GND_BN
@@
 	3650 2950 3750 2950
 Connection ~ 3650 3050
+Wire Wire Line
+	5750 2250 5800 2250
+Wire Wire Line
+	5600 2250 5750 2250
+Wire Wire Line
+	3650 2250 3750 2250
+Wire Wire Line
+	3650 2250 3650 2350
+Wire Wire Line
+	3650 4150 3650 4250
+Wire Wire Line
+	3650 3150 3650 3250
+Wire Wire Line
+	3650 2750 3750 2750
+Wire Wire Line
+	3650 2750 3650 2850
+Wire Wire Line
+	3650 2650 3650 2750
+Wire Wire Line
+	5750 2950 5800 2950
+Wire Wire Line
+	5600 2950 5750 2950
+Wire Wire Line
+	5750 4050 5800 4050
+Wire Wire Line
+	3650 4050 3650 4150
+Wire Wire Line
+	3650 4050 3750 4050
+Wire Wire Line
+	3650 3950 3650 4050
+Wire Wire Line
+	3650 3100 3650 3150
+Wire Wire Line
+	3650 3050 3650 3100
 $EndSCHEMATC
