File: HW/projects/ibex/BMS_Ibex/HostInterfaceSplitter/HostInterfaceSplitter-V2.1/HostInterfaceSplitter-V2.kicad_pcb (KiCad board)
At the start: 4 copper layers, 57.5 x 45 mm, 54 parts, among them P1 SPI_IN, P10 Digital_In, P11 SPI_Out, P12 12V_Out, P13 Digital_In, P14 SPI_Out, P15 12V_Out, P2 12V, P3 Digital_Out, P4 Digital_In, P5 SPI_Out, P6 12V_Out, P7 Digital_In, P8 SPI_Out, P9 12V_Out, U1 SN74HC21D, U2 74HCT1G125GW-Q100, U3 NC7WZ16P6X, U4 74HCT1G125GW-Q100, U5 NC7WZ16P6X, U6 74HCT1G125GW-Q100, U7 NC7WZ16P6X, U8 74HCT1G125GW-Q100, U9 NC7WZ16P6X

Commit message: Sync ibex bms with tera local
Parts:
- removed D2: ~Alert, tera_diodes:LED_0805
- removed D3: ~Fault, tera_diodes:LED_0805
- removed R1, R2: 5k1, tera_rlc:C_0805in
- removed the REF*** at (151.8, 110.6)
- removed the svg2mod at (112.5, 113.8)
- added C10: 100n, tera_rlc:C_0603in, B.Cu at (143.8, 105.0)
- added C11: 100n, tera_rlc:C_0603in, B.Cu at (143.8, 107.2)
- added C12: 100n, tera_rlc:C_0603in, B.Cu at (140.5, 109.2)
- added C13: 100n, tera_rlc:C_0603in, B.Cu at (140.5, 103.0)
- added C14: 1n, tera_rlc:C_0603in, B.Cu at (118.2, 82.9)
- added C15: 1n, tera_rlc:C_0603in, B.Cu at (118.2, 87.5)
- added C16: 1n, tera_rlc:C_0603in, B.Cu at (118.2, 85.2)
- added C17: 100n, tera_rlc:C_0603in, B.Cu at (118.2, 89.8)
- added C18: 100n, tera_rlc:C_0603in, B.Cu at (124.8, 91.0)
- added C19: 1n, tera_rlc:C_0603in, B.Cu at (124.8, 86.3)
- added C20: 1n, tera_rlc:C_0603in, B.Cu at (124.8, 88.7)
- added C21: 1n, tera_rlc:C_0603in, B.Cu at (124.8, 84.0)
- added C22: 100n, tera_rlc:C_0603in, B.Cu at (128.5, 82.3)
- added C23: 100n, tera_rlc:C_0603in, B.Cu at (140.7, 85.4)
- added C24: 100n, tera_rlc:C_0603in, B.Cu at (146.6, 114.8)
- added C25: 100n, tera_rlc:C_0603in, B.Cu at (146.6, 117.0)
- added C26: 100n, tera_rlc:C_0603in, B.Cu at (143.2, 119.0)
- added C27: 100n, tera_rlc:C_0603in, B.Cu at (143.2, 112.8)
- added C28: 1n, tera_rlc:C_0603in, B.Cu at (111.3, 94.4)
- added C29: 1n, tera_rlc:C_0603in, B.Cu at (111.3, 99.0)
- added C30: 1n, tera_rlc:C_0603in, B.Cu at (111.3, 96.7)
- added C31: 100n, tera_rlc:C_0603in, B.Cu at (111.3, 101.3)
- added C32: 100n, tera_rlc:C_0603in, B.Cu at (117.9, 102.5)
- added C33: 1n, tera_rlc:C_0603in, B.Cu at (117.9, 97.8)
- added C34: 1n, tera_rlc:C_0603in, B.Cu at (117.9, 100.2)
- added C35: 1n, tera_rlc:C_0603in, B.Cu at (117.9, 95.5)
- added C36: 100n, tera_rlc:C_0603in, B.Cu at (121.6, 93.8)
- added C37: 100n, tera_rlc:C_0603in, B.Cu at (140.6, 95.4)
- added C38: 100n, tera_rlc:C_0603in, B.Cu at (137.1, 123.2)
- added C39: 100n, tera_rlc:C_0603in, B.Cu at (137.1, 125.5)
- added C40: 100n, tera_rlc:C_0603in, B.Cu at (133.8, 127.5)
- added C41: 100n, tera_rlc:C_0603in, B.Cu at (133.8, 121.2)
- added C42: 1n, tera_rlc:C_0603in, B.Cu at (118.3, 106.2)
- added C43: 1n, tera_rlc:C_0603in, B.Cu at (118.3, 110.8)
- added C44: 1n, tera_rlc:C_0603in, B.Cu at (118.3, 108.5)
- added C45: 100n, tera_rlc:C_0603in, B.Cu at (118.3, 113.2)
- added C46: 100n, tera_rlc:C_0603in, B.Cu at (125.0, 114.3)
- added C47: 1n, tera_rlc:C_0603in, B.Cu at (125.0, 109.7)
- added C48: 1n, tera_rlc:C_0603in, B.Cu at (125.0, 112.0)
- added C49: 1n, tera_rlc:C_0603in, B.Cu at (125.0, 107.4)
- added C50: 100n, tera_rlc:C_0603in, B.Cu at (128.7, 105.7)
- added C51: 100n, tera_rlc:C_0603in, B.Cu at (144.8, 95.5)
- added C52: 100n, tera_rlc:C_0603in, B.Cu at (148.2, 120.0)
- added C53: 100n, tera_rlc:C_0603in, B.Cu at (145.9, 120.0)
- added C54: 100n, tera_rlc:C_0603in, B.Cu at (142.9, 123.4)
- added C55: 100n, tera_rlc:C_0603in, B.Cu at (149.1, 123.4)
- added C56: 1n, tera_rlc:C_0603in, B.Cu at (111.2, 117.0)
- added C57: 1n, tera_rlc:C_0603in, B.Cu at (111.2, 121.6)
- added C58: 1n, tera_rlc:C_0603in, B.Cu at (111.2, 119.3)
- added C59: 100n, tera_rlc:C_0603in, B.Cu at (111.2, 123.9)
- added C60: 100n, tera_rlc:C_0603in, B.Cu at (117.9, 126.2)
- added C61: 1n, tera_rlc:C_0603in, B.Cu at (117.9, 121.6)
- added C62: 1n, tera_rlc:C_0603in, B.Cu at (117.9, 123.9)
- added C63: 1n, tera_rlc:C_0603in, B.Cu at (117.9, 119.3)
- added C64: 100n, tera_rlc:C_0603in, B.Cu at (121.6, 117.5)
- added C65: 100n, tera_rlc:C_0603in, B.Cu at (154.8, 95.3)
- added D10: 5V, tera_diodes:SD05_tvs_5v, B.Cu at (128.5, 86.2)
- added D11: 15V, tera_diodes:CDSOD323-T15S_tvs_15v, B.Cu at (138.7, 85.4)
- added D12: 5V, tera_diodes:SD05_tvs_5v, B.Cu at (137.7, 119.8)
- added D13: 5V, tera_diodes:SD05_tvs_5v, B.Cu at (137.6, 112.4)
- added D14: 5V, tera_diodes:SD05_tvs_5v, B.Cu at (121.6, 103.3)
- added D15: 5V, tera_diodes:SD05_tvs_5v, B.Cu at (121.6, 99.5)
- added D16: 5V, tera_diodes:SD05_tvs_5v, B.Cu at (121.6, 101.5)
- added D17: 5V, tera_diodes:SD05_tvs_5v, B.Cu at (121.6, 95.8)
- added D18: 5V, tera_diodes:SD05_tvs_5v, B.Cu at (121.6, 97.7)
- added D19: 15V, tera_diodes:CDSOD323-T15S_tvs_15v, B.Cu at (138.6, 95.4)
- added D20: 5V, tera_diodes:SD05_tvs_5v, B.Cu at (128.2, 128.2)
- added D21: 5V, tera_diodes:SD05_tvs_5v, B.Cu at (128.2, 120.2)
- added D22: 5V, tera_diodes:SD05_tvs_5v, B.Cu at (128.7, 115.2)
- added D23: 5V, tera_diodes:SD05_tvs_5v, B.Cu at (128.7, 111.4)
- added D24: 5V, tera_diodes:SD05_tvs_5v, B.Cu at (128.7, 113.3)
- added D25: 5V, tera_diodes:SD05_tvs_5v, B.Cu at (128.7, 107.6)
- added D26: 5V, tera_diodes:SD05_tvs_5v, B.Cu at (128.7, 109.5)
- added D27: 15V, tera_diodes:CDSOD323-T15S_tvs_15v, B.Cu at (144.8, 97.5)
- added D28: 5V, tera_diodes:SD05_tvs_5v, B.Cu at (141.3, 127.8)
- added D29: 5V, tera_diodes:SD05_tvs_5v, B.Cu at (150.2, 127.8)
- added D30: 5V, tera_diodes:SD05_tvs_5v, B.Cu at (121.6, 127.1)
- added D31: 5V, tera_diodes:SD05_tvs_5v, B.Cu at (121.6, 123.3)
- added D32: 5V, tera_diodes:SD05_tvs_5v, B.Cu at (121.6, 125.2)
- added D33: 5V, tera_diodes:SD05_tvs_5v, B.Cu at (121.6, 119.5)
- added D34: 5V, tera_diodes:SD05_tvs_5v, B.Cu at (121.6, 121.4)
- added D35: 15V, tera_diodes:CDSOD323-T15S_tvs_15v, B.Cu at (154.8, 97.2)
- added D4: 5V, tera_diodes:SD05_tvs_5v, B.Cu at (134.7, 109.8)
- added D5: 5V, tera_diodes:SD05_tvs_5v, B.Cu at (134.7, 102.3)
- added D6: 5V, tera_diodes:SD05_tvs_5v, B.Cu at (128.5, 91.8)
- added D7: 5V, tera_diodes:SD05_tvs_5v, B.Cu at (128.5, 88.0)
- added D8: 5V, tera_diodes:SD05_tvs_5v, B.Cu at (128.5, 90.0)
- added D9: 5V, tera_diodes:SD05_tvs_5v, B.Cu at (128.5, 84.2)
- added R11: 1k, tera_rlc:R_0603in, B.Cu at (140.5, 105.0)
- added R12: 1k, tera_rlc:R_0603in, B.Cu at (140.5, 107.2)
- added R13: 1k, tera_rlc:R_0603in, B.Cu at (121.5, 82.9)
- added R14: 1k, tera_rlc:R_0603in, B.Cu at (121.5, 87.5)
- added R15: 1k, tera_rlc:R_0603in, B.Cu at (121.5, 85.2)
- added R16: 1k, tera_rlc:R_0603in, B.Cu at (121.5, 89.8)
- added R17: 1k, tera_rlc:R_0603in, B.Cu at (143.2, 114.8)
- added R18: 1k, tera_rlc:R_0603in, B.Cu at (143.2, 117.0)
- added R19: 1k, tera_rlc:R_0603in, B.Cu at (114.5, 94.4)
- added R20: 1k, tera_rlc:R_0603in, B.Cu at (114.5, 99.0)
- added R21: 1k, tera_rlc:R_0603in, B.Cu at (114.5, 96.7)
- added R22: 1k, tera_rlc:R_0603in, B.Cu at (114.5, 101.3)
- added R23: 1k, tera_rlc:R_0603in, B.Cu at (133.8, 123.2)
- added R24: 1k, tera_rlc:R_0603in, B.Cu at (133.8, 125.5)
- added R25: 1k, tera_rlc:R_0603in, B.Cu at (121.6, 106.2)
- added R26: 1k, tera_rlc:R_0603in, B.Cu at (121.6, 110.8)
- added R27: 1k, tera_rlc:R_0603in, B.Cu at (121.6, 108.5)
- added R28: 1k, tera_rlc:R_0603in, B.Cu at (121.6, 113.2)
- added R29: 1k, tera_rlc:R_0603in, B.Cu at (147.1, 123.4)
- added R30: 1k, tera_rlc:R_0603in, B.Cu at (144.9, 123.4)
- added R31: 1k, tera_rlc:R_0603in, B.Cu at (114.5, 118.2)
- added R32: 1k, tera_rlc:R_0603in, B.Cu at (114.5, 122.8)
- added R33: 1k, tera_rlc:R_0603in, B.Cu at (114.5, 120.5)
- added R34: 1k, tera_rlc:R_0603in, B.Cu at (114.5, 125.0)
- C1: footprint tera_rlc:C_0805in -> tera_rlc:C_0603in; moved to B.Cu
- C2, C3, C4, C5, C6, C7, C8, C9, U1, U2, U3, U4, U5, U6, U7, U8, U9: moved to B.Cu
- R10, R3, R4, R5, R6, R7, R8, R9: footprint tera_rlc:R_0805in -> tera_rlc:R_0603in; moved to B.Cu
- moved svg2mod 47.8 mm to (108.0, 128.4)
- moved P3 42.1 mm to (156.1, 117.2)
- moved U1 40.9 mm to (153.8, 109.1), turned to 270 degrees
- moved C1 33.8 mm to (148.2, 110.9), turned to 90 degrees
- moved R6 32.3 mm to (140.8, 113.8), turned to 270 degrees
- moved R5 32.2 mm to (140.8, 118.0), turned to 90 degrees
- moved R3 31.0 mm to (137.8, 108.4), turned to 90 degrees
- moved R4 31.0 mm to (137.8, 104.0), turned to 270 degrees
- moved C6 28.9 mm to (110.0, 111.5), turned to 180 degrees
- moved R10 28.3 mm to (148.1, 125.9), turned to 180 degrees
- moved P7 27.8 mm to (138.2, 117.3)
- moved C8 27.3 mm to (111.2, 126.2), turned to 0 degrees
- moved P4 26.8 mm to (135.1, 107.3)
- moved U6 26.4 mm to (110.0, 114.2), turned to 90 degrees
- moved U9 25.6 mm to (105.8, 117.5)
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Connections:
- P10 pad 1: /~FAULT3 -> /Line3/~Fault_Ext
- P10 pad 2: /~ALERT3 -> /Line3/~Alert_Ext
- P11 pad 2: /Line3/CLK_S -> Net-(C49-Pad2)
- P11 pad 3: /Line3/MISO_S -> Net-(C48-Pad2)
- P11 pad 4: /Line3/MOSI_S -> Net-(C47-Pad2)
- P11 pad 5: /NCS3 -> Net-(C46-Pad2)
- P13 pad 1: /~FAULT4 -> /Line4/~Fault_Ext
- P13 pad 2: /~ALERT4 -> /Line4/~Alert_Ext
- P14 pad 2: /Line4/CLK_S -> Net-(C63-Pad2)
- P14 pad 3: /Line4/MISO_S -> Net-(C62-Pad2)
- P14 pad 4: /Line4/MOSI_S -> Net-(C61-Pad2)
- P14 pad 5: /NCS4 -> Net-(C60-Pad2)
- P4 pad 1: /~FAULT1 -> /Line1/~Fault_Ext
- P4 pad 2: /~ALERT1 -> /Line1/~Alert_Ext
- P5 pad 2: /Line1/CLK_S -> Net-(C21-Pad2)
- P5 pad 3: /Line1/MISO_S -> Net-(C20-Pad2)
- P5 pad 4: /Line1/MOSI_S -> Net-(C19-Pad2)
- P5 pad 5: /NCS1 -> Net-(C18-Pad2)
- P7 pad 1: /~FAULT2 -> /Line2/~Fault_Ext
- P7 pad 2: /~ALERT2 -> /Line2/~Alert_Ext
- P8 pad 2: /Line2/CLK_S -> Net-(C35-Pad2)
- P8 pad 3: /Line2/MISO_S -> Net-(C34-Pad2)
- P8 pad 4: /Line2/MOSI_S -> Net-(C33-Pad2)
- P8 pad 5: /NCS2 -> Net-(C32-Pad2)
- R10 pad 1: /~ALERT4 -> /Line4/~Alert_Ext
- R3 pad 1: /~FAULT1 -> /Line1/~Fault_Ext
- R4 pad 1: /~ALERT1 -> /Line1/~Alert_Ext
- R5 pad 1: /~FAULT2 -> /Line2/~Fault_Ext
- R6 pad 1: /~ALERT2 -> /Line2/~Alert_Ext
- R7 pad 1: /~FAULT3 -> /Line3/~Fault_Ext
- R8 pad 1: /~ALERT3 -> /Line3/~Alert_Ext
- R9 pad 1: /~FAULT4 -> /Line4/~Fault_Ext
- U3 pad 1: /CLK -> /MOSI
- U3 pad 3: /MOSI -> /CLK
- U3 pad 4: /Line1/MOSI_S -> /Line1/CLK_S
- U3 pad 6: /Line1/CLK_S -> /Line1/MOSI_S
- U5 pad 1: /CLK -> /MOSI
- U5 pad 3: /MOSI -> /CLK
- U5 pad 4: /Line2/MOSI_S -> /Line2/CLK_S
- U5 pad 6: /Line2/CLK_S -> /Line2/MOSI_S
- U7 pad 1: /CLK -> /MOSI
- U7 pad 3: /MOSI -> /CLK
- U7 pad 4: /Line3/MOSI_S -> /Line3/CLK_S
- U7 pad 6: /Line3/CLK_S -> /Line3/MOSI_S
- U9 pad 1: /CLK -> /MOSI
- U9 pad 3: /MOSI -> /CLK
- U9 pad 4: /Line4/MOSI_S -> /Line4/CLK_S
- U9 pad 6: /Line4/CLK_S -> /Line4/MOSI_S
Routing:
- net GND: track 6.41 -> 50.7 mm, vias 32 -> 103
- net /NCS2: track 35.5 -> 13.3 mm, vias 0 -> 1
- net /~ALERT1: track 31.6 -> 9.89 mm, vias 2 -> 0
- net /MOSI: track 63.6 -> 42.7 mm, vias 5 -> 1
- net /CLK: track 61.6 -> 41.6 mm, vias 4 -> 0
- net +12V: track 0.00 -> 17.8 mm
- net /MISO: track 69.7 -> 52.5 mm, vias 4 -> 1
- net /~FAULT3: track 9.83 -> 27.0 mm
- net /NCS4: track 41.7 -> 24.6 mm, vias 0 -> 1
- net +5V: track 15.7 -> 32.0 mm
- net /NCS3: track 39.3 -> 23.9 mm, vias 0 -> 1
- net /~FAULT1: track 27.8 -> 12.5 mm, vias 1 -> 0
- net /~ALERT3: track 15.8 -> 30.2 mm, vias 0 -> 2
- net /NCS1: track 40.0 -> 26.5 mm, vias 0 -> 1
- net Net-(C32-Pad2): track 0.00 -> 12.2 mm, vias 0 -> 1
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- added copper zone on B.Cu, net +12V
- added copper zone on B.Cu, net /Line1/~Alert_Ext
- added copper zone on B.Cu, net /Line1/~Fault_Ext
- added copper zone on B.Cu, net /Line2/~Alert_Ext
- added copper zone on B.Cu, net /Line2/~Fault_Ext
- added copper zone on B.Cu, net /Line3/~Alert_Ext
- added copper zone on B.Cu, net /Line3/~Fault_Ext
- added copper zone on B.Cu, net /Line4/~Alert_Ext
- added copper zone on B.Cu, net /Line4/~Fault_Ext
- removed copper zone on In1.Cu, net +12V
Other:
- board size 57.5 x 45 mm -> 57.5 x 49.5 mm
- board text added: "BMS Host Interface Splitter V2.1 TERA TU Graz ©Pöschl Rene, Apr. 2018 Solderpad v0.51"
- board text added: "Host Interface Splitter V2.1"
- board text added: "©2018 Pöschl Solderpad v0.51"
- board text removed: "BMS Host Interface Splitter V2.1 TERA TU Graz ©Pöschl Rene, Apr. 2017 Solderpad v0.51"
- board text removed: "Host Interface Splitter V2"
- board text removed: "©2017 Pöschl Solderpad v0.51"
