File: HW/projects/ibex/BMS_Ibex/HostInterfaceSplitter/HostInterfaceSplitter-V2.1/HostInterfaceSplitter-V2.sch (KiCad schematic (older format))
At the start: 10 parts, among them P1 SPI_IN, P2 12V, P3 Digital_Out, U1 SN74HC21D

Commit message: Sync ibex bms with tera local
Parts:
- removed D2: ~Alert, tera_diodes:LED_0805, symbol LED
- removed D3: ~Fault, tera_diodes:LED_0805, symbol LED
- removed R1, R2: 5k1, tera_rlc:C_0805in, symbol R_Small
- C1: footprint tera_rlc:C_0805in -> tera_rlc:C_0603in
Changed lines of the file:
@@
 $EndSheet
 $Comp
-L +12V #PWR01
+L +12V #PWR8
 U 1 1 57EB9032
 P 4550 1000
-F 0 "#PWR01" H 4550 850 50  0001 C CNN
+F 0 "#PWR8" H 4550 850 50  0001 C CNN
 F 1 "+12V" H 4565 1173 50  0000 C CNN
 F 2 "" H 4550 1000 50  0000 C CNN
@@
 $EndComp
 $Comp
-L +5V #PWR02
+L +5V #PWR10
 U 1 1 57EB911E
 P 4750 900
-F 0 "#PWR02" H 4750 750 50  0001 C CNN
+F 0 "#PWR10" H 4750 750 50  0001 C CNN
 F 1 "+5V" H 4765 1073 50  0000 C CNN
 F 2 "" H 4750 900 50  0000 C CNN
@@
 $EndComp
 $Comp
-L GND #PWR03
+L GND #PWR12
 U 1 1 57EB920A
 P 4800 1950
-F 0 "#PWR03" H 4800 1700 50  0001 C CNN
+F 0 "#PWR12" H 4800 1700 50  0001 C CNN
 F 1 "GND" H 4805 1777 50  0000 C CNN
 F 2 "" H 4800 1950 50  0000 C CNN
@@
 	4800 1900 5000 1900
 $Comp
-L +12V #PWR04
+L +12V #PWR9
 U 1 1 57EBAC18
 P 4550 2550
-F 0 "#PWR04" H 4550 2400 50  0001 C CNN
+F 0 "#PWR9" H 4550 2400 50  0001 C CNN
 F 1 "+12V" H 4565 2723 50  0000 C CNN
 F 2 "" H 4550 2550 50  0000 C CNN
@@
 $EndComp
 $Comp
-L +5V #PWR05
+L +5V #PWR11
 U 1 1 57EBAC1E
 P 4750 2450
-F 0 "#PWR05" H 4750 2300 50  0001 C CNN
+F 0 "#PWR11" H 4750 2300 50  0001 C CNN
 F 1 "+5V" H 4765 2623 50  0000 C CNN
 F 2 "" H 4750 2450 50  0000 C CNN
@@
 $EndComp
 $Comp
-L GND #PWR06
+L GND #PWR13
 U 1 1 57EBAC24
 P 4800 3500
-F 0 "#PWR06" H 4800 3250 50  0001 C CNN
+F 0 "#PWR13" H 4800 3250 50  0001 C CNN
 F 1 "GND" H 4805 3327 50  0000 C CNN
 F 2 "" H 4800 3500 50  0000 C CNN
@@
 	4800 3450 5000 3450
 $Comp
-L +12V #PWR07
+L +12V #PWR14
 U 1 1 57EBE610
 P 7200 950
-F 0 "#PWR07" H 7200 800 50  0001 C CNN
+F 0 "#PWR14" H 7200 800 50  0001 C CNN
 F 1 "+12V" H 7215 1123 50  0000 C CNN
 F 2 "" H 7200 950 50  0000 C CNN
@@
 $EndComp
 $Comp
-L +5V #PWR08
+L +5V #PWR16
 U 1 1 57EBE616
 P 7400 850
-F 0 "#PWR08" H 7400 700 50  0001 C CNN
+F 0 "#PWR16" H 7400 700 50  0001 C CNN
 F 1 "+5V" H 7415 1023 50  0000 C CNN
 F 2 "" H 7400 850 50  0000 C CNN
@@
 $EndComp
 $Comp
-L GND #PWR09
+L GND #PWR18
 U 1 1 57EBE61C
 P 7450 1900
-F 0 "#PWR09" H 7450 1650 50  0001 C CNN
+F 0 "#PWR18" H 7450 1650 50  0001 C CNN
 F 1 "GND" H 7455 1727 50  0000 C CNN
 F 2 "" H 7450 1900 50  0000 C CNN
@@
 	7450 1850 7650 1850
 $Comp
-L +12V #PWR010
+L +12V #PWR15
 U 1 1 57EBE628
 P 7200 2500
-F 0 "#PWR010" H 7200 2350 50  0001 C CNN
+F 0 "#PWR15" H 7200 2350 50  0001 C CNN
 F 1 "+12V" H 7215 2673 50  0000 C CNN
 F 2 "" H 7200 2500 50  0000 C CNN
@@
 $EndComp
 $Comp
-L +5V #PWR011
+L +5V #PWR17
 U 1 1 57EBE62E
 P 7400 2400
-F 0 "#PWR011" H 7400 2250 50  0001 C CNN
+F 0 "#PWR17" H 7400 2250 50  0001 C CNN
 F 1 "+5V" H 7415 2573 50  0000 C CNN
 F 2 "" H 7400 2400 50  0000 C CNN
@@
 $EndComp
 $Comp
-L GND #PWR012
+L GND #PWR19
 U 1 1 57EBE634
 P 7450 3450
-F 0 "#PWR012" H 7450 3200 50  0001 C CNN
+F 0 "#PWR19" H 7450 3200 50  0001 C CNN
 F 1 "GND" H 7455 3277 50  0000 C CNN
 F 2 "" H 7450 3450 50  0000 C CNN
@@
 $EndComp
 $Comp
-L +5V #PWR013
+L +5V #PWR3
 U 1 1 57EC13FF
 P 1850 1100
-F 0 "#PWR013" H 1850 950 50  0001 C CNN
+F 0 "#PWR3" H 1850 950 50  0001 C CNN
 F 1 "+5V" H 1865 1273 50  0000 C CNN
 F 2 "" H 1850 1100 50  0000 C CNN
@@
 	1850 1200 1600 1200
 $Comp
-L GND #PWR014
+L GND #PWR4
 U 1 1 57EC156C
 P 1850 2100
-F 0 "#PWR014" H 1850 1850 50  0001 C CNN
+F 0 "#PWR4" H 1850 1850 50  0001 C CNN
 F 1 "GND" H 1855 1927 50  0000 C CNN
 F 2 "" H 1850 2100 50  0000 C CNN
@@
 $EndComp
 $Comp
-L GND #PWR015
+L GND #PWR6
 U 1 1 57EC87DA
 P 1900 2850
-F 0 "#PWR015" H 1900 2600 50  0001 C CNN
+F 0 "#PWR6" H 1900 2600 50  0001 C CNN
 F 1 "GND" H 1905 2677 50  0000 C CNN
 F 2 "" H 1900 2850 50  0000 C CNN
@@
 	1600 2750 1900 2750
 $Comp
-L +12V #PWR016
+L +12V #PWR5
 U 1 1 57ECA461
 P 1900 2550
-F 0 "#PWR016" H 1900 2400 50  0001 C CNN
+F 0 "#PWR5" H 1900 2400 50  0001 C CNN
 F 1 "+12V" H 1915 2723 50  0000 C CNN
 F 2 "" H 1900 2550 50  0000 C CNN
@@
 F 0 "C1" H 992 4896 50  0000 L CNN
 F 1 "100n" H 992 4805 50  0000 L CNN
-F 2 "tera_rlc:C_0805in" H 992 4759 50  0001 L CNN
+F 2 "tera_rlc:C_0603in" H 992 4759 50  0001 L CNN
 F 3 "" H 900 4850 50  0000 C CNN
 F 4 "52-100n" H 900 4850 60  0001 C CNN "HPN"
@@
 Connection ~ 1050 5050
 $Comp
-L GND #PWR017
+L GND #PWR2
 U 1 1 57EDFA87
 P 1050 5100
-F 0 "#PWR017" H 1050 4850 50  0001 C CNN
+F 0 "#PWR2" H 1050 4850 50  0001 C CNN
 F 1 "GND" H 1055 4927 50  0000 C CNN
 F 2 "" H 1050 5100 50  0000 C CNN
@@
 $EndComp
 $Comp
-L +5V #PWR018
+L +5V #PWR1
 U 1 1 57EE024E
 P 1050 4600
-F 0 "#PWR018" H 1050 4450 50  0001 C CNN
+F 0 "#PWR1" H 1050 4450 50  0001 C CNN
 F 1 "+5V" H 1065 4773 50  0000 C CNN
 F 2 "" H 1050 4600 50  0000 C CNN
@@
 $EndComp
 $Comp
-L R_Small R1
-U 1 1 57EBAFD2
-P 2800 5100
-F 0 "R1" H 2859 5146 50  0000 L CNN
-F 1 "5k1" H 2859 5055 50  0000 L CNN
-F 2 "tera_rlc:C_0805in" H 2800 5100 50  0001 C CNN
-F 3 "" H 2800 5100 50  0000 C CNN
-F 4 "11-5K10" H 2800 5100 60  0001 C CNN "HPN"
-	1    2800 5100
-	1    0    0    -1
-$EndComp
-$Comp
-L R_Small R2
-U 1 1 57EBB42A
-P 3100 5100
-F 0 "R2" H 3159 5146 50  0000 L CNN
-F 1 "5k1" H 3159 5055 50  0000 L CNN
-F 2 "tera_rlc:C_0805in" H 3100 5100 50  0001 C CNN
-F 3 "" H 3100 5100 50  0000 C CNN
-F 4 "11-5K10" H 3100 5100 60  0001 C CNN "HPN"
-	1    3100 5100
-	1    0    0    -1
-$EndComp
-$Comp
-L LED D2
-U 1 1 57EBB52E
-P 2800 5500
-F 0 "D2" V 2900 5700 50  0000 R CNN
-F 1 "~Alert" V 2800 5750 50  0000 R CNN
-F 2 "tera_diodes:LED_0805" H 2800 5500 50  0001 C CNN
-F 3 "" H 2800 5500 50  0000 C CNN
-F 4 "21-0002" V 2800 5500 60  0001 C CNN "HPN"
-	1    2800 5500
-	0    -1   -1   0
-$EndComp
-$Comp
-L LED D3
-U 1 1 57EBB7E1
-P 3100 5500
-F 0 "D3" V 3146 5392 50  0000 R CNN
-F 1 "~Fault" V 3055 5392 50  0000 R CNN
-F 2 "tera_diodes:LED_0805" H 3100 5500 50  0001 C CNN
-F 3 "" H 3100 5500 50  0000 C CNN
-F 4 "21-0002" V 3100 5500 60  0001 C CNN "HPN"
-	1    3100 5500
-	0    -1   -1   0
-$EndComp
-Wire Wire Line
-	2800 5700 2800 5750
-Wire Wire Line
-	2800 5750 3100 5750
-Wire Wire Line
-	3100 5750 3100 5700
-$Comp
-L GND #PWR019
-U 1 1 57EBB9A8
-P 2950 5800
-F 0 "#PWR019" H 2950 5550 50  0001 C CNN
-F 1 "GND" H 2955 5627 50  0000 C CNN
-F 2 "" H 2950 5800 50  0000 C CNN
-F 3 "" H 2950 5800 50  0000 C CNN
-	1    2950 5800
-	1    0    0    -1
-$EndComp
-Wire Wire Line
-	2950 5800 2950 5750
-Connection ~ 2950 5750
-Wire Wire Line
-	3100 5300 3100 5200
-Wire Wire Line
-	3100 5000 3100 4900
-Connection ~ 3100 4900
-Wire Wire Line
-	2800 5300 2800 5200
-Wire Wire Line
-	2800 5000 2800 4800
-Connection ~ 2800 4800
-$Comp
-L PWR_FLAG #FLG020
+L PWR_FLAG #FLG2
 U 1 1 57ED4CB3
 P 1600 2650
-F 0 "#FLG020" H 1600 2745 50  0001 C CNN
+F 0 "#FLG2" H 1600 2745 50  0001 C CNN
 F 1 "PWR_FLAG" H 1600 2874 50  0000 C CNN
 F 2 "" H 1600 2650 50  0000 C CNN
@@
 $EndComp
 $Comp
-L PWR_FLAG #FLG021
+L PWR_FLAG #FLG3
 U 1 1 57ED5D2F
 P 1600 2750
-F 0 "#FLG021" H 1600 2845 50  0001 C CNN
+F 0 "#FLG3" H 1600 2845 50  0001 C CNN
 F 1 "PWR_FLAG" H 1600 2973 50  0000 C CNN
 F 2 "" H 1600 2750 50  0000 C CNN
@@
 $EndComp
 $Comp
-L PWR_FLAG #FLG022
+L PWR_FLAG #FLG1
 U 1 1 57ED856B
 P 1600 1200
-F 0 "#FLG022" H 1600 1295 50  0001 C CNN
+F 0 "#FLG1" H 1600 1295 50  0001 C CNN
 F 1 "PWR_FLAG" H 1600 1424 50  0000 C CNN
 F 2 "" H 1600 1200 50  0000 C CNN
