File: HW/projects/ibex/BMS_Ibex/HostInterfaceSplitter/HostInterfaceSplitter-V2.1/HostLine.sch (KiCad schematic (older format))
At the start: 9 parts, among them P4 Digital_In, P5 SPI_Out, P6 12V_Out, U2 74HCT1G125GW-Q100, U3 NC7WZ16P6X

Commit message: Sync ibex bms with tera local
Parts:
- added C10, C11, C12, C13, C17, C18, C22, C23: 100n, tera_rlc:C_0603in, symbol C
- added C14, C15, C16, C19, C20, C21: 1n, tera_rlc:C_0603in, symbol C
- added D10, D4, D5, D6, D7, D8, D9: 5V, tera_diodes:SD05_tvs_5v, symbol ZENERsmall
- added D11: 15V, tera_diodes:CDSOD323-T15S_tvs_15v, symbol ZENERsmall
- added R11, R12, R13, R14, R15, R16: 1k, tera_rlc:R_0603in, symbol R
- R3, R4: footprint tera_rlc:R_0805in -> tera_rlc:R_0603in
Connections:
- net 12V: now also C23.2, D11.1 (K)
- net 5V: now also C22.2, D9.1 (K)
- net CLK: now also U3.3 (A2); no longer U3.1 (A1)
- net CLK_S: now also U3.4 (Y2), C14.2, R13.2; no longer P5.2 (P2), U3.6 (Y1)
- net GND: now also C10.1, C11.1, C12.1, C13.1, C14.1, C15.1, C16.1, C17.1, C18.1, C19.1, C20.1, C21.1, C22.1, C23.1, D10.2 (A), D11.2 (A), D4.2 (A), D5.2 (A), D6.2 (A), D7.2 (A), D8.2 (A), D9.2 (A)
- net MISO_S: now also C15.2, R14.2; no longer P5.3 (P3)
- net MOSI: now also U3.1 (A1); no longer U3.3 (A2)
- net MOSI_S: now also U3.6 (Y1), C16.2, R15.2; no longer P5.4 (P4), U3.4 (Y2)
- net NCS: now also C17.2, R16.2; no longer P5.5 (P5)
- net ~ALERT: now also C10.2, R11.2; no longer P4.2 (P2), R4.1
- net ~FAULT: now also C11.2, R12.2; no longer P4.1 (P1), R3.1
- new net: C21.2, D10.1 (K), P5.2 (P2), R13.1
- new net: C20.2, D8.1 (K), P5.3 (P3), R14.1
- new net: C19.2, D7.1 (K), P5.4 (P4), R15.1
- new net: C18.2, D6.1 (K), P5.5 (P5), R16.1
- new net ~Alert_Ext: C13.2, D5.1 (K), P4.2 (P2), R11.1, R4.1
- new net ~Fault_Ext: C12.2, D4.1 (K), P4.1 (P1), R12.1, R3.1
Other:
- moved on the sheet: C2, C3, P4, P5, P6, R3, R4, U2, U3
