File: HW/projects/ibex/BMS_Ibex/Interlock/InterlockV2.1-kicad/Interlock.kicad_pcb (KiCad board)
At the start: 2 copper layers, 41 x 24.5 mm, 34 parts, among them K1 ASSR-1218, K2 ASSR-1218, K3 ASSR-1218, P1 12V, P2 crtl, P3 IL1, P4 IL2, U1 TMR_1-1212

Commit message: Sync ibex bms with tera local
Parts:
- C1: value 4,7uF 25V -> 4.7uF 25V
- L1: value 4,7uH 1,2A -> 4.7uH 1.2A
- R8, R9: value 5k6 -> 5k1
Changed lines of the file:
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@@
     (links 50)
     (no_connects 0)
-    (area 49.367857 82.8 108.500001 114.2925)
+    (area 55.424999 87.924999 96.575001 112.575001)
     (thickness 1.6)
     (drawings 25)
@@
       (effects (font (size 0.6 0.6) (thickness 0.1)) (justify mirror))
     )
-    (fp_text value "4,7uH 1,2A" (at -4.953 -0.635 180) (layer B.Fab)
+    (fp_text value "4.7uH 1.2A" (at -4.953 -0.635 180) (layer B.Fab)
       (effects (font (size 0.6 0.6) (thickness 0.1)) (justify mirror))
     )
@@
       (effects (font (size 0.6 0.6) (thickness 0.1)) (justify mirror))
     )
-    (fp_text value 5k6 (at 0 -1.016 270) (layer B.Fab)
+    (fp_text value 5k1 (at 0 -1.016 270) (layer B.Fab)
       (effects (font (size 0.6 0.6) (thickness 0.1)) (justify mirror))
     )
@@
       (effects (font (size 0.6 0.6) (thickness 0.1)) (justify mirror))
     )
-    (fp_text value 5k6 (at 0 -1.016 270) (layer B.Fab)
+    (fp_text value 5k1 (at 0 -1.016 270) (layer B.Fab)
       (effects (font (size 0.6 0.6) (thickness 0.1)) (justify mirror))
     )
@@
       (effects (font (size 0.6 0.6) (thickness 0.1)) (justify mirror))
     )
-    (fp_text value "4,7uF 25V" (at 3.429 0 270) (layer B.Fab)
-      (effects (font (size 0.6 0.6) (thickness 0.1)) (justify mirror))
-    )
+    (fp_text value "4.7uF 25V" (at 3.429 0 270) (layer B.Fab)
+      (effects (font (size 0.6 0.6) (thickness 0.1)) (justify mirror))
+    )
