File: HW/projects/ibex/BMS_Ibex/Interlock/InterlockV2.2-kicad/Interlock.kicad_pcb (KiCad board)
At the start: 2 copper layers, 41 x 24.5 mm, 34 parts, among them K1 ASSR-1218, K2 ASSR-1218, K3 ASSR-1218, P1 12V, P2 crtl, P3 IL1, P4 IL2, U1 TMR_1-1212

Commit message: Sync ibex bms with tera local
Parts:
- JP4: moved to B.Cu
- L1: value 4.7uH 1.2A -> 4.7uH 0.7A
- turned JP4 to 180 degrees
Routing:
- net /IL_Out-: vias 0 -> 1
- net /IL_Out+: vias 2 -> 1
Changed lines of the file:
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@@
   (general
     (links 60)
-    (no_connects 1)
-    (area 49.367857 82.8 108.500001 114.2925)
+    (no_connects 0)
+    (area 55.424999 87.924999 96.575001 112.575001)
     (thickness 1.6)
     (drawings 25)
-    (tracks 113)
+    (tracks 115)
     (zones 0)
     (modules 34)
@@
     (aux_axis_origin 55.5 88)
     (grid_origin 55.5 88)
-    (visible_elements FFFEEF7F)
+    (visible_elements FFFFEF7F)
     (pcbplotparams
       (layerselection 0x010f0_ffffffff)
@@
       (effects (font (size 0.6 0.6) (thickness 0.1)) (justify mirror))
     )
-    (fp_text value "4.7uH 1.2A" (at -4.953 -0.635 180) (layer B.Fab)
+    (fp_text value "4.7uH 0.7A" (at -4.953 -0.635 180) (layer B.Fab)
       (effects (font (size 0.6 0.6) (thickness 0.1)) (justify mirror))
     )
@@
       (net 20 /IL_In-))
   )
-  (module tera_general:SOLDERJUMPER_2 (layer F.Cu)
-    (at 89.282 104.383)
+  (module tera_general:SOLDERJUMPER_2 (layer B.Cu)
+    (at 89.282 104.383 180)
     (descr Solderjumper)
     (tags Solderjumper)
     (attr smd)
-    (fp_text reference JP4 (at 0 1.397) (layer F.Fab)
-      (effects (font (size 0.6 0.6) (thickness 0.1)))
-    )
-    (fp_text value "Last In Line" (at 0 -3.175 90) (layer F.Fab)
-      (effects (font (size 0.5 0.5) (thickness 0.08)))
-    )
-    (fp_text user %R (at -0.254 -1.778) (layer F.SilkS)
-      (effects (font (size 1 1) (thickness 0.15)))
-    )
-    (fp_line (start 0.95 -1.05) (end -0.95 -1.05) (layer F.CrtYd) (width 0.05))
-    (fp_line (start 0.95 1.05) (end 0.95 -1.05) (layer F.CrtYd) (width 0.05))
-    (fp_line (start -0.95 1.05) (end 0.95 1.05) (layer F.CrtYd) (width 0.05))
-    (fp_line (start -0.95 -1.05) (end -0.95 1.05) (layer F.CrtYd) (width 0.05))
-    (pad 1 smd rect (at 0 -0.45) (size 1.4 0.7) (layers F.Cu F.Paste F.Mask)
+    (fp_text reference JP4 (at 0 -1.397 180) (layer B.Fab)
+      (effects (font (size 0.6 0.6) (thickness 0.1)) (justify mirror))
+    )
+    (fp_text value "Last In Line" (at 0 3.175 450) (layer B.Fab)
+      (effects (font (size 0.5 0.5) (thickness 0.08)) (justify mirror))
+    )
+    (fp_text user %R (at -0.254 1.778 180) (layer B.SilkS)
+      (effects (font (size 1 1) (thickness 0.15)) (justify mirror))
+    )
+    (fp_line (start 0.95 1.05) (end -0.95 1.05) (layer B.CrtYd) (width 0.05))
+    (fp_line (start 0.95 -1.05) (end 0.95 1.05) (layer B.CrtYd) (width 0.05))
+    (fp_line (start -0.95 -1.05) (end 0.95 -1.05) (layer B.CrtYd) (width 0.05))
+    (fp_line (start -0.95 1.05) (end -0.95 -1.05) (layer B.CrtYd) (width 0.05))
+    (pad 1 smd rect (at 0 0.45 180) (size 1.4 0.7) (layers B.Cu B.Paste B.Mask)
       (net 23 /IL_Out+))
-    (pad 2 smd rect (at 0 0.45) (size 1.4 0.7) (layers F.Cu F.Paste F.Mask)
+    (pad 2 smd rect (at 0 -0.45 180) (size 1.4 0.7) (layers B.Cu B.Paste B.Mask)
       (net 19 /IL_Out-))
   )
@@
       (effects (font (size 0.6 0.6) (thickness 0.1)) (justify mirror))
     )
-    (fp_text value "220pF 2kV" (at 0 -0.5) (layer B.Fab)
+    (fp_text value "220pF 2kV" (at 0.04 -1.401) (layer B.Fab)
       (effects (font (size 0.6 0.6) (thickness 0.1)) (justify mirror))
     )
@@
     (fp_line (start 1.4 0.835) (end 1.4 -0.835) (layer B.Mask) (width 0.15))
     (fp_line (start -1.4 0.835) (end 1.4 0.835) (layer B.Mask) (width 0.15))
-    (fp_text user %R (at 1.64 -2.001) (layer B.SilkS)
+    (fp_text user %R (at 0 1.899) (layer B.SilkS)
       (effects (font (size 1 1) (thickness 0.15)) (justify mirror))
     )
@@
     (pad 2 smd rect (at 1.7 0) (size 0.6 1.82) (layers B.Cu B.Paste B.Mask)
       (net 18 IL_V-))
-    (pad 1 smd circle (at 2 0.61) (size 0.6 0.6) (layers B.Cu B.Paste B.Mask)
-      (net 1 GND))
+    (pad 2 smd circle (at 2 0.61) (size 0.6 0.6) (layers B.Cu B.Paste B.Mask)
+      (net 18 IL_V-))
     (pad 2 smd rect (at 1.7 0) (size 1.2 1.22) (layers B.Cu B.Paste B.Mask)
       (net 18 IL_V-))
@@
   (segment (start 86.037 103.324002) (end 86.037 101.403) (width 0.5) (layer F.Cu) (net 18))
   (segment (start 83.82 100.203) (end 85.886999 100.203) (width 1) (layer B.Cu) (net 18))
+  (segment (start 89.3 105.9) (end 89.3 104.833) (width 0.25) (layer B.Cu) (net 19))
+  (segment (start 89.282 108.193) (end 89.282 105.918) (width 0.25) (layer F.Cu) (net 19))
+  (segment (start 89.282 105.918) (end 89.3 105.9) (width 0.25) (layer F.Cu) (net 19))
+  (via (at 89.3 105.9) (size 0.75) (drill 0.3) (layers F.Cu B.Cu) (net 19))
   (segment (start 79.502 108.954) (end 80.202 108.954) (width 0.25) (layer F.Cu) (net 19))
   (segment (start 80.202 108.954) (end 81.473 110.225) (width 0.25) (layer F.Cu) (net 19))
   (segment (start 81.473 110.225) (end 87.25 110.225) (width 0.25) (layer F.Cu) (net 19))
-  (segment (start 89.282 108.193) (end 89.282 104.833) (width 0.25) (layer F.Cu) (net 19))
   (segment (start 87.25 110.225) (end 89.282 108.193) (width 0.25) (layer F.Cu) (net 19))
-  (segment (start 89.282 104.833) (end 91.15 104.833) (width 0.25) (layer F.Cu) (net 19))
-  (segment (start 91.15 104.833) (end 92.457 103.526) (width 0.25) (layer F.Cu) (net 19))
-  (segment (start 92.457 103.526) (end 92.457 102.351) (width 0.25) (layer F.Cu) (net 19))
+  (segment (start 89.282 104.833) (end 91.15 104.833) (width 0.25) (layer B.Cu) (net 19))
+  (segment (start 91.15 104.833) (end 92.457 103.526) (width 0.25) (layer B.Cu) (net 19))
+  (segment (start 92.457 103.526) (end 92.457 102.351) (width 0.25) (layer B.Cu) (net 19))
   (segment (start 79.502 108.954) (end 79.702 108.954) (width 0.25) (layer F.Cu) (net 19))
   (segment (start 77.216 109.982) (end 77.724 109.982) (width 0.25) (layer F.Cu) (net 19))
@@
   (segment (start 82.042 99.685) (end 85.091 96.636) (width 0.25) (layer F.Cu) (net 22))
   (via (at 85.091 96.636) (size 0.75) (drill 0.3) (layers F.Cu B.Cu) (net 22))
-  (segment (start 88.012 103.875) (end 89.282 103.875) (width 0.25) (layer F.Cu) (net 23))
+  (segment (start 88.012 103.875) (end 89.282 103.875) (width 0.25) (layer B.Cu) (net 23))
   (segment (start 83.937137 104.257137) (end 87.629863 104.257137) (width 0.25) (layer B.Cu) (net 23))
   (segment (start 87.629863 104.257137) (end 88.012 103.875) (width 0.25) (layer B.Cu) (net 23))
-  (via (at 88.012 103.875) (size 0.75) (drill 0.3) (layers F.Cu B.Cu) (net 23))
-  (segment (start 89.282 103.933) (end 89.282 103.026) (width 0.25) (layer F.Cu) (net 23))
-  (segment (start 89.282 103.026) (end 92.457 99.851) (width 0.25) (layer F.Cu) (net 23))
+  (segment (start 89.282 103.933) (end 89.282 103.026) (width 0.25) (layer B.Cu) (net 23))
+  (segment (start 89.282 103.026) (end 92.457 99.851) (width 0.25) (layer B.Cu) (net 23))
   (segment (start 79.248 104.267) (end 83.937137 104.257137) (width 0.25) (layer F.Cu) (net 23))
   (segment (start 83.947 104.267) (end 83.937137 104.257137) (width 0.25) (layer F.Cu) (net 23))
