File: HW/projects/ibex/BMS_Ibex/Interlock/InterlockV2.2-kicad/Interlock.sch (KiCad schematic (older format))
At the start: 29 parts, among them K1 ASSR-1218, K2 ASSR-1218, K3 ASSR-1218, P1 12V, P2 crtl, P3 IL1, P4 IL2, U1 TMR_1-1212

Commit message: Sync ibex bms with tera local
Parts:
- L1: value 4.7uH 1.2A -> 4.7uH 0.7A
Changed lines of the file:
@@
 P 2150 1750
 F 0 "L1" H 2180 1790 50  0000 L CNN
-F 1 "4.7uH 1.2A" V 2050 1500 50  0000 L CNN
+F 1 "4.7uH 0.7A" V 2050 1500 50  0000 L CNN
 F 2 "tera_rlc:L_muarta_LQH32PN" H 2150 1750 50  0001 C CNN
 F 3 "" H 2150 1750 50  0000 C CNN
