File: HW/projects/ibex/BMS_Ibex/Master/BMS_Master_V6.1_kicad/2xRelaisWithRM.sch (KiCad schematic (older format))
At the start: 12 parts, among them IC4 TLE8102SG, P7 K_CH1, P8 K_CH2, Q1 BSS205N

Commit message: Sync ibex bms with tera local
Parts:
- C10: symbol C -> Device:C
- D4, D5: symbol LED -> Device:LED
- IC4: symbol TLE8102SG -> tera_general:TLE8102SG
- P7, P8: symbol CONN_01X04 -> Connector_Generic:Conn_01x04
- Q1: symbol BSS205N -> tera_general:BSS205N
- R10, R11, R7, R8, R9: symbol R -> Device:R
Changed lines of the file:
@@
-EESchema Schematic File Version 2
-LIBS:power
-LIBS:device
-LIBS:transistors
-LIBS:conn
-LIBS:linear
-LIBS:regul
-LIBS:74xx
-LIBS:cmos4000
-LIBS:adc-dac
-LIBS:memory
-LIBS:xilinx
-LIBS:microcontrollers
-LIBS:dsp
-LIBS:microchip
-LIBS:analog_switches
-LIBS:motorola
-LIBS:texas
-LIBS:intel
-LIBS:audio
-LIBS:interface
-LIBS:digital-audio
-LIBS:philips
-LIBS:display
-LIBS:cypress
-LIBS:siliconi
-LIBS:opto
-LIBS:atmel
-LIBS:contrib
-LIBS:valves
-LIBS:ft232rl
-LIBS:relais
-LIBS:Supply
-LIBS:tera_general
-LIBS:tera_switches
-LIBS:tera_logic
-LIBS:tera_processors
-LIBS:tera_connectors
-LIBS:tera_emc_prodection
+EESchema Schematic File Version 4
 LIBS:BMS_Master_V6_kicad-cache
-EELAYER 25 0
+EELAYER 26 0
 EELAYER END
 $Descr A4 11693 8268
@@
 $EndDescr
 $Comp
-L TLE8102SG IC4
+L tera_general:TLE8102SG IC4
 U 1 1 56F50D05
 P 2900 4500
@@
 AR Path="/56F50775/56F6E70D/56F50D05" Ref="IC?"  Part="1"
 AR Path="/56F50775/56F7A222/56F50D05" Ref="IC5"  Part="1"
-F 0 "IC5" H 2900 5137 60  0000 C CNN
+F 0 "IC4" H 2900 5137 60  0000 C CNN
 F 1 "TLE8102SG" H 2900 5031 60  0000 C CNN
 F 2 "infineon:INF-PG-DSO-12-11-EP_N_EPvias" H 2850 4500 60  0001 C CNN
@@
 $EndComp
 $Comp
-L CONN_01X04 P7
+L Connector_Generic:Conn_01x04 P7
 U 1 1 56F510D7
-P 5050 3750
+P 5000 3750
 AR Path="/56F50775/56F58707/56F510D7" Ref="P7"  Part="1"
 AR Path="/56F50775/56F59A35/56F510D7" Ref="P?"  Part="1"
 AR Path="/56F50775/56F6E70D/56F510D7" Ref="P?"  Part="1"
 AR Path="/56F50775/56F7A222/56F510D7" Ref="P9"  Part="1"
-F 0 "P9" V 5250 3750 50  0000 C CNN
-F 1 "K_CH1" V 5150 3800 50  0000 C CNN
-F 2 "tera_Connectors_JST:JST_XH_B04B-XH-A_04x2.50mm_Straight" H 5050 3750 50  0001 C CNN
-F 3 "" H 5050 3750 50  0000 C CNN
-F 4 "02-0904" H 0   0   50  0001 C CNN "HPN"
-	1    5050 3750
+F 0 "P7" V 5200 3750 50  0000 C CNN
+F 1 "K_CH1" V 5100 3800 50  0000 C CNN
+F 2 "tera_Connectors_JST:JST_XH_B04B-XH-A_04x2.50mm_Straight" H 5000 3750 50  0001 C CNN
+F 3 "" H 5000 3750 50  0000 C CNN
+F 4 "02-0904" H -50 0   50  0001 C CNN "HPN"
+	1    5000 3750
 	0    -1   -1   0
 $EndComp
 $Comp
-L LED D4
+L Device:LED D4
 U 1 1 56F51697
 P 4000 3900
@@
 AR Path="/56F50775/56F6E70D/56F51697" Ref="D?"  Part="1"
 AR Path="/56F50775/56F7A222/56F51697" Ref="D6"  Part="1"
-F 0 "D6" V 4046 3792 50  0000 R CNN
+F 0 "D4" V 4046 3792 50  0000 R CNN
 F 1 "K_CH1" V 3955 3792 50  0000 R CNN
 F 2 "tera_diodes:LED_0805" H 4000 3900 50  0001 C CNN
@@
 $EndComp
 $Comp
-L R R7
+L Device:R R7
 U 1 1 56FBF234
 P 4000 3500
@@
 AR Path="/56F50775/56F6E70D/56FBF234" Ref="R?"  Part="1"
 AR Path="/56F50775/56F7A222/56FBF234" Ref="R12"  Part="1"
-F 0 "R12" H 4070 3546 50  0000 L CNN
+F 0 "R7" H 4070 3546 50  0000 L CNN
 F 1 "12k" H 4070 3455 50  0000 L CNN
 F 2 "tera_rlc:R_0805in" V 3930 3500 50  0001 C CNN
@@
 $EndComp
 $Comp
-L C C10
+L Device:C C10
 U 1 1 56FBF235
 P 3550 4050
@@
 AR Path="/56F50775/56F6E70D/56FBF235" Ref="C?"  Part="1"
 AR Path="/56F50775/56F7A222/56FBF235" Ref="C11"  Part="1"
-F 0 "C11" V 3298 4050 50  0000 C CNN
+AR Path="/56FBF235" Ref="C11"  Part="1"
+F 0 "C10" V 3298 4050 50  0000 C CNN
 F 1 "100n" V 3389 4050 50  0000 C CNN
 F 2 "tera_rlc:C_0603in" H 3588 3900 50  0001 C CNN
@@
 $EndComp
 $Comp
-L LED D5
+L Device:LED D5
 U 1 1 56F52A53
 P 4400 3900
@@
 AR Path="/56F50775/56F6E70D/56F52A53" Ref="D?"  Part="1"
 AR Path="/56F50775/56F7A222/56F52A53" Ref="D7"  Part="1"
-F 0 "D7" V 4446 3792 50  0000 R CNN
+F 0 "D5" V 4446 3792 50  0000 R CNN
 F 1 "K_CH2" V 4355 3792 50  0000 R CNN
 F 2 "tera_diodes:LED_0805" H 4400 3900 50  0001 C CNN
@@
 $EndComp
 $Comp
-L R R8
+L Device:R R8
 U 1 1 56FBF237
 P 4400 3500
@@
 AR Path="/56F50775/56F6E70D/56FBF237" Ref="R?"  Part="1"
 AR Path="/56F50775/56F7A222/56FBF237" Ref="R13"  Part="1"
-F 0 "R13" H 4470 3546 50  0000 L CNN
+F 0 "R8" H 4470 3546 50  0000 L CNN
 F 1 "12k" H 4470 3455 50  0000 L CNN
 F 2 "tera_rlc:R_0805in" V 4330 3500 50  0001 C CNN
@@
 $EndComp
 $Comp
-L CONN_01X04 P8
+L Connector_Generic:Conn_01x04 P8
 U 1 1 56F53CE4
-P 5650 3750
+P 5600 3750
 AR Path="/56F50775/56F58707/56F53CE4" Ref="P8"  Part="1"
 AR Path="/56F50775/56F59A35/56F53CE4" Ref="P?"  Part="1"
 AR Path="/56F50775/56F6E70D/56F53CE4" Ref="P?"  Part="1"
 AR Path="/56F50775/56F7A222/56F53CE4" Ref="P10"  Part="1"
-F 0 "P10" V 5850 3750 50  0000 C CNN
-F 1 "K_CH2" V 5750 3700 50  0000 C CNN
-F 2 "tera_Connectors_JST:JST_XH_B04B-XH-A_04x2.50mm_Straight" H 5650 3750 50  0001 C CNN
-F 3 "" H 5650 3750 50  0000 C CNN
-F 4 "02-0904" H 0   0   50  0001 C CNN "HPN"
-	1    5650 3750
+F 0 "P8" V 5800 3750 50  0000 C CNN
+F 1 "K_CH2" V 5700 3700 50  0000 C CNN
+F 2 "tera_Connectors_JST:JST_XH_B04B-XH-A_04x2.50mm_Straight" H 5600 3750 50  0001 C CNN
+F 3 "" H 5600 3750 50  0000 C CNN
+F 4 "02-0904" H -50 0   50  0001 C CNN "HPN"
+	1    5600 3750
 	0    -1   -1   0
 $EndComp
 $Comp
-L R R10
+L Device:R R10
 U 1 1 56F54F4C
 P 5100 4800
@@
 AR Path="/56F50775/56F6E70D/56F54F4C" Ref="R?"  Part="1"
 AR Path="/56F50775/56F7A222/56F54F4C" Ref="R15"  Part="1"
-F 0 "R15" H 5170 4846 50  0000 L CNN
+F 0 "R10" H 5170 4846 50  0000 L CNN
 F 1 "18k" H 5170 4755 50  0000 L CNN
 F 2 "tera_rlc:R_0805in" V 5030 4800 50  0001 C CNN
@@
 $EndComp
 $Comp
-L R R11
+L Device:R R11
 U 1 1 56F54FD1
 P 5100 5200
@@
 AR Path="/56F50775/56F6E70D/56F54FD1" Ref="R?"  Part="1"
 AR Path="/56F50775/56F7A222/56F54FD1" Ref="R16"  Part="1"
-F 0 "R16" H 5170 5246 50  0000 L CNN
+F 0 "R11" H 5170 5246 50  0000 L CNN
 F 1 "12k" H 5170 5155 50  0000 L CNN
 F 2 "tera_rlc:R_0805in" V 5030 5200 50  0001 C CNN
@@
 $EndComp
 $Comp
-L BSS205N Q1
+L tera_general:BSS205N Q1
 U 1 1 56F5519C
 P 4700 5250
@@
 AR Path="/56F50775/56F6E70D/56F5519C" Ref="Q?"  Part="1"
 AR Path="/56F50775/56F7A222/56F5519C" Ref="Q2"  Part="1"
-F 0 "Q2" H 4773 5346 50  0000 L CNN
+F 0 "Q1" H 4773 5346 50  0000 L CNN
 F 1 "BSS205N" H 4773 5255 50  0000 L CNN
 F 2 "tera_sot:SOT-23" H 4800 5225 50  0001 L CIN
@@
 $EndComp
 $Comp
-L R R9
+L Device:R R9
 U 1 1 56F55984
 P 4700 4800
@@
 AR Path="/56F50775/56F6E70D/56F55984" Ref="R?"  Part="1"
 AR Path="/56F50775/56F7A222/56F55984" Ref="R14"  Part="1"
-F 0 "R14" H 4770 4846 50  0000 L CNN
+F 0 "R9" H 4770 4846 50  0000 L CNN
 F 1 "10k" H 4770 4755 50  0000 L CNN
 F 2 "tera_rlc:R_0603in" V 4630 4800 50  0001 C CNN
@@
 	3300 4700 3400 4700
 Wire Wire Line
-	3400 4700 3400 5400
+	3400 4700 3400 4800
 Wire Wire Line
 	3300 4800 3400 4800
@@
 	3350 4100 3300 4100
 Wire Wire Line
-	3350 3600 3350 4100
+	3350 3600 3350 4050
 Wire Wire Line
 	3400 4050 3350 4050
@@
 	3750 4050 3700 4050
 Wire Wire Line
-	3300 4200 4900 4200
-Wire Wire Line
-	4000 4200 4000 4100
+	3300 4200 4000 4200
+Wire Wire Line
+	4000 4200 4000 4050
 Wire Wire Line
 	4000 3250 4000 3350
 Wire Wire Line
-	4000 3650 4000 3700
-Wire Wire Line
-	4400 4100 4400 4300
+	4000 3650 4000 3750
+Wire Wire Line
+	4400 4050 4400 4300
 Wire Wire Line
 	4400 3250 4400 3350
 Wire Wire Line
-	4400 3650 4400 3700
-Wire Wire Line
-	3300 4300 5500 4300
+	4400 3650 4400 3750
+Wire Wire Line
+	3300 4300 4400 4300
 Wire Wire Line
 	4900 4200 4900 3950
@@
 	5600 4050 5600 3950
 Wire Wire Line
-	5000 4050 5900 4050
+	5000 4050 5600 4050
 Wire Wire Line
 	5000 4050 5000 3950
@@
 	4700 5400 4700 5350
 Wire Wire Line
-	3100 5400 5100 5400
+	3100 5400 3400 5400
 Wire Wire Line
 	5100 5400 5100 5350
 Wire Wire Line
-	5100 4950 5100 5050
+	5100 4950 5100 5000
 Wire Wire Line
 	5100 5000 4950 5000
@@
 	4950 5250 4900 5250
 Wire Wire Line
-	4700 4950 4700 5050
+	4700 4950 4700 5000
 Wire Wire Line
 	4600 5000 4700 5000
 Wire Wire Line
-	2300 4200 2500 4200
+	2300 4200 2400 4200
 Wire Wire Line
 	2400 4200 2400 4100
@@
 	3750 4050 3750 5400
 Wire Wire Line
-	3850 3250 4400 3250
+	3850 3250 4000 3250
 Wire Wire Line
 	4700 4550 4650 4550
@@
 Connection ~ 4000 3250
 Connection ~ 5600 4050
+Wire Wire Line
+	3400 4800 3400 4900
+Wire Wire Line
+	3400 4900 3400 5400
+Wire Wire Line
+	3350 4050 3350 4100
+Wire Wire Line
+	4000 4200 4900 4200
+Wire Wire Line
+	4400 4300 5500 4300
+Wire Wire Line
+	5100 5000 5100 5050
+Wire Wire Line
+	4700 5000 4700 5050
+Wire Wire Line
+	2400 4200 2500 4200
+Wire Wire Line
+	3400 5400 3750 5400
+Wire Wire Line
+	4700 5400 5100 5400
+Wire Wire Line
+	3750 5400 4700 5400
+Wire Wire Line
+	4000 3250 4400 3250
+Wire Wire Line
+	5600 4050 5900 4050
 $EndSCHEMATC
