File: HW/projects/ibex/BMS_Ibex/Master/BMS_Master_V6.1_kicad/BMS_Master_V6_kicad.sch (KiCad schematic (older format))
At the start: 5 parts, among them P1 Interlock, P2 12V_IL, P3 ExtGPIO, U1 STM32f4_board_v3-1

Commit message: Sync ibex bms with tera local
Parts:
- JP1: symbol Jumper_NO_Small -> Device:Jumper_NO_Small
- P1, P3: symbol CONN_01X05 -> Connector_Generic:Conn_01x05
- P2: symbol CONN_01X02 -> Connector_Generic:Conn_01x02
- U1: symbol STM32f4_board_v3-1 -> tera_general:STM32f4_board_v3-1
Changed lines of the file:
@@
-EESchema Schematic File Version 2
-LIBS:power
-LIBS:device
-LIBS:transistors
-LIBS:conn
-LIBS:linear
-LIBS:regul
-LIBS:74xx
-LIBS:cmos4000
-LIBS:adc-dac
-LIBS:memory
-LIBS:xilinx
-LIBS:microcontrollers
-LIBS:dsp
-LIBS:microchip
-LIBS:analog_switches
-LIBS:motorola
-LIBS:texas
-LIBS:intel
-LIBS:audio
-LIBS:interface
-LIBS:digital-audio
-LIBS:philips
-LIBS:display
-LIBS:cypress
-LIBS:siliconi
-LIBS:opto
-LIBS:atmel
-LIBS:contrib
-LIBS:valves
-LIBS:ft232rl
-LIBS:relais
-LIBS:Supply
-LIBS:tera_general
-LIBS:tera_switches
-LIBS:tera_logic
-LIBS:tera_processors
-LIBS:tera_connectors
-LIBS:tera_emc_prodection
+EESchema Schematic File Version 4
 LIBS:BMS_Master_V6_kicad-cache
-EELAYER 25 0
+EELAYER 26 0
 EELAYER END
 $Descr A4 11693 8268
@@
 $EndSheet
 $Comp
-L +12V #PWR01
+L power:+12V #PWR01
 U 1 1 56FEA5A8
 P 1950 1150
@@
 $EndComp
 $Comp
-L +3.3V #PWR02
+L power:+3.3V #PWR02
 U 1 1 56FEB8F4
 P 2250 1350
@@
 $EndComp
 $Comp
-L +5V #PWR03
+L power:+5V #PWR03
 U 1 1 56FEBA50
 P 2100 1250
@@
 $EndComp
 $Comp
-L GND #PWR04
+L power:GND #PWR04
 U 1 1 56FEC261
 P 1900 1650
@@
 $EndComp
 $Comp
-L GND #PWR05
+L power:GND #PWR05
 U 1 1 5709711B
 P 9650 2500
@@
 $EndComp
 $Comp
-L GND #PWR06
+L power:GND #PWR06
 U 1 1 571624A7
 P 9150 5900
@@
 $EndComp
 $Comp
-L GND #PWR07
+L power:GND #PWR07
 U 1 1 57164043
 P 7350 6200
@@
 $EndComp
 $Comp
-L +3.3V #PWR08
+L power:+3.3V #PWR08
 U 1 1 571685D4
 P 7150 4550
@@
 $EndComp
 $Comp
-L +5V #PWR09
+L power:+5V #PWR09
 U 1 1 5716C6FF
 P 8800 4450
@@
 $EndComp
 $Comp
-L +3.3V #PWR010
+L power:+3.3V #PWR010
 U 1 1 5716C857
 P 8650 4550
@@
 $EndComp
 $Comp
-L +5V #PWR011
+L power:+5V #PWR011
 U 1 1 571F6147
 P 5000 4400
@@
 $EndComp
 $Comp
-L GND #PWR012
+L power:GND #PWR012
 U 1 1 571F62C0
 P 5000 5200
@@
 $EndComp
 $Comp
-L CONN_01X05 P1
+L Connector_Generic:Conn_01x05 P1
 U 1 1 572776F2
 P 4100 4600
@@
 $EndComp
 $Comp
-L CONN_01X02 P2
+L Connector_Generic:Conn_01x02 P2
 U 1 1 572776FB
-P 4100 5400
-F 0 "P2" H 4100 5550 50  0000 L CNN
-F 1 "12V_IL" V 4250 5300 50  0000 L CNN
-F 2 "tera_Connectors_JST:JST_XH_B02B-XH-A_02x2.50mm_Straight" H 4100 5400 50  0001 C CNN
-F 3 "" H 4100 5400 50  0000 C CNN
-F 4 "02-0902" H 0   0   50  0001 C CNN "HPN"
-	1    4100 5400
+P 4100 5450
+F 0 "P2" H 4100 5600 50  0000 L CNN
+F 1 "12V_IL" V 4250 5350 50  0000 L CNN
+F 2 "tera_Connectors_JST:JST_XH_B02B-XH-A_02x2.50mm_Straight" H 4100 5450 50  0001 C CNN
+F 3 "" H 4100 5450 50  0000 C CNN
+F 4 "02-0902" H 0   50  50  0001 C CNN "HPN"
+	1    4100 5450
 	1    0    0    1
 $EndComp
 $Comp
-L +12V #PWR013
+L power:+12V #PWR013
 U 1 1 5727BEE4
 P 3700 5300
@@
 $EndComp
 $Comp
-L GND #PWR014
+L power:GND #PWR014
 U 1 1 5727F262
 P 3700 5500
@@
 $EndComp
 $Comp
-L GND #PWR015
+L power:GND #PWR015
 U 1 1 57281F7A
 P 3700 4850
@@
 $EndComp
 $Comp
-L +5V #PWR016
+L power:+5V #PWR016
 U 1 1 57283E2B
 P 3700 4300
@@
 $EndComp
 $Comp
-L +12V #PWR017
+L power:+12V #PWR017
 U 1 1 56FCC5C9
 P 1150 4500
@@
 $EndComp
 $Comp
-L GND #PWR018
+L power:GND #PWR018
 U 1 1 56FCF655
 P 1150 4900
@@
 $EndComp
 $Comp
-L Jumper_NO_Small JP1
+L Device:Jumper_NO_Small JP1
 U 1 1 5701E943
 P 1200 4700
@@
 $EndComp
 $Comp
-L +5V #PWR019
+L power:+5V #PWR019
 U 1 1 57DE1EE6
 P 6950 4500
@@
 $EndComp
 $Comp
-L GND #PWR020
+L power:GND #PWR020
 U 1 1 5813CDE1
 P 2750 7550
@@
 $EndComp
 $Comp
-L +5V #PWR021
+L power:+5V #PWR021
 U 1 1 5814095A
 P 1200 7400
@@
 $EndComp
 $Comp
-L +3.3V #PWR022
+L power:+3.3V #PWR022
 U 1 1 58143753
 P 1150 5750
@@
 $EndComp
 $Comp
-L STM32f4_board_v3-1 U1
+L tera_general:STM32f4_board_v3-1 U1
 U 1 1 581F9E37
 P 4050 1500
@@
 $EndComp
 $Comp
-L STM32f4_board_v3-1 U1
+L tera_general:STM32f4_board_v3-1 U1
 U 2 1 581FA2F9
 P 5600 1900
@@
 $EndComp
 $Comp
-L STM32f4_board_v3-1 U1
+L tera_general:STM32f4_board_v3-1 U1
 U 3 1 581FA586
 P 6950 1900
@@
 $EndComp
 $Comp
-L STM32f4_board_v3-1 U1
+L tera_general:STM32f4_board_v3-1 U1
 U 4 1 581FA726
 P 1950 6500
@@
 $EndComp
 $Comp
-L STM32f4_board_v3-1 U1
+L tera_general:STM32f4_board_v3-1 U1
 U 5 1 581FA8E0
 P 8950 2600
@@
 $EndComp
 $Comp
-L STM32f4_board_v3-1 U1
+L tera_general:STM32f4_board_v3-1 U1
 U 6 1 581FB0E4
 P 8800 2100
@@
 $EndComp
 $Comp
-L STM32f4_board_v3-1 U1
+L tera_general:STM32f4_board_v3-1 U1
 U 7 1 581FB2CA
 P 8900 3250
@@
 $EndComp
 $Comp
-L STM32f4_board_v3-1 U1
+L tera_general:STM32f4_board_v3-1 U1
 U 8 1 581FB4A8
 P 10150 1050
@@
 $EndComp
 $Comp
-L +3.3V #PWR023
+L power:+3.3V #PWR023
 U 1 1 58456FD2
 P 4850 4400
@@
 $EndComp
 $Comp
-L +12P #PWR024
+L power:+12P #PWR024
 U 1 1 584732E5
 P 1800 1050
@@
 $EndComp
 $Comp
-L +12P #PWR025
+L power:+12P #PWR025
 U 1 1 58474964
 P 9100 4250
@@
 $EndComp
 $Comp
-L CONN_01X05 P3
+L Connector_Generic:Conn_01x05 P3
 U 1 1 584A7C04
 P 2300 2500
@@
 $EndComp
 $Comp
-L GND #PWR026
+L power:GND #PWR026
 U 1 1 584A9279
 P 2550 2750
@@
 $EndComp
 $Comp
-L +3.3V #PWR027
+L power:+3.3V #PWR027
 U 1 1 584AB990
 P 2550 2250
@@
 	9300 2100 9800 2100
 Wire Wire Line
-	2750 5800 2750 7550
+	2750 5800 2750 5900
 Wire Wire Line
 	2750 5800 2600 5800
@@
 	2600 7400 2750 7400
 Wire Wire Line
-	1200 7400 1350 7400
-Wire Wire Line
-	1150 5750 1150 7300
+	1200 7400 1300 7400
+Wire Wire Line
+	1150 5750 1150 5800
 Wire Wire Line
 	1150 7300 1350 7300
@@
 NoConn ~ 6000 1900
 NoConn ~ 6000 2000
+Wire Wire Line
+	2750 5900 2750 6000
+Wire Wire Line
+	2750 6000 2750 6100
+Wire Wire Line
+	2750 6100 2750 6200
+Wire Wire Line
+	2750 6200 2750 6300
+Wire Wire Line
+	2750 6300 2750 6400
+Wire Wire Line
+	2750 6400 2750 6500
+Wire Wire Line
+	2750 6500 2750 6600
+Wire Wire Line
+	2750 6600 2750 6700
+Wire Wire Line
+	2750 6700 2750 7100
+Wire Wire Line
+	2750 7100 2750 7300
+Wire Wire Line
+	2750 7400 2750 7500
+Wire Wire Line
+	1150 7100 1150 7300
+Wire Wire Line
+	1150 6700 1150 7100
+Wire Wire Line
+	1150 6600 1150 6700
+Wire Wire Line
+	1150 6500 1150 6600
+Wire Wire Line
+	1150 6400 1150 6500
+Wire Wire Line
+	1150 6300 1150 6400
+Wire Wire Line
+	1150 6200 1150 6300
+Wire Wire Line
+	1150 6100 1150 6200
+Wire Wire Line
+	1150 6000 1150 6100
+Wire Wire Line
+	1150 5900 1150 6000
+Wire Wire Line
+	1150 5800 1150 5900
+Wire Wire Line
+	2750 7500 2750 7550
+Wire Wire Line
+	2750 7300 2750 7400
+Wire Wire Line
+	1300 7400 1350 7400
 $EndSCHEMATC
