File: HW/projects/ibex/BMS_Ibex/Master/BMS_Master_V6.1_kicad/LEM.sch (KiCad schematic (older format))
At the start: 9 parts, among them IC1 LM4132A-1.8, P4 LEM

Commit message: Sync ibex bms with tera local
Parts:
- C1, C2, C3: symbol C_Small -> Device:C_Small
- D1: symbol ZENER -> Device:D_Zener
- IC1: symbol LM4132A-1.8 -> Supply:LM4132A-1.8
- JP2: symbol JUMPER3_NO -> tera_general:JUMPER3_NO
- P4: symbol CONN_01X04 -> Connector_Generic:Conn_01x04
- R1, R2: symbol R_Small -> Device:R_Small
Changed lines of the file:
@@
-EESchema Schematic File Version 2
-LIBS:power
-LIBS:device
-LIBS:transistors
-LIBS:conn
-LIBS:linear
-LIBS:regul
-LIBS:74xx
-LIBS:cmos4000
-LIBS:adc-dac
-LIBS:memory
-LIBS:xilinx
-LIBS:microcontrollers
-LIBS:dsp
-LIBS:microchip
-LIBS:analog_switches
-LIBS:motorola
-LIBS:texas
-LIBS:intel
-LIBS:audio
-LIBS:interface
-LIBS:digital-audio
-LIBS:philips
-LIBS:display
-LIBS:cypress
-LIBS:siliconi
-LIBS:opto
-LIBS:atmel
-LIBS:contrib
-LIBS:valves
-LIBS:ft232rl
-LIBS:relais
-LIBS:Supply
-LIBS:tera_general
-LIBS:tera_switches
-LIBS:tera_logic
-LIBS:tera_processors
-LIBS:tera_connectors
-LIBS:tera_emc_prodection
+EESchema Schematic File Version 4
 LIBS:BMS_Master_V6_kicad-cache
-EELAYER 25 0
+EELAYER 26 0
 EELAYER END
 $Descr A4 11693 8268
@@
 $EndDescr
 $Comp
-L LM4132A-1.8 IC1
+L Supply:LM4132A-1.8 IC1
 U 1 1 571E65BD
 P 2150 3200
@@
 $EndComp
 $Comp
-L C_Small C1
+L Device:C_Small C1
 U 1 1 571E681E
 P 1500 3250
@@
 $EndComp
 $Comp
-L C_Small C2
+L Device:C_Small C2
 U 1 1 571E6954
 P 2550 3250
@@
 $EndComp
 $Comp
-L R_Small R1
+L Device:R_Small R1
 U 1 1 571E6A03
 P 2900 3250
@@
 $EndComp
 $Comp
-L CONN_01X04 P4
+L Connector_Generic:Conn_01x04 P4
 U 1 1 571E6B07
-P 4200 3150
+P 4200 3200
 AR Path="/56F5071E/571E6146/571E6B07" Ref="P4"  Part="1"
 AR Path="/56F5071E/571E9DC1/571E6B07" Ref="P5"  Part="1"
 AR Path="/56F5071E/571E9F88/571E6B07" Ref="P6"  Part="1"
-F 0 "P4" H 4118 2769 50  0000 C CNN
-F 1 "LEM" H 4118 2860 50  0000 C CNN
-F 2 "tera_Connectors_Molex:Molex_PicoBlade_53398-0471_04x1.25mm_Straight" H 4200 3150 50  0001 C CNN
-F 3 "" H 4200 3150 50  0000 C CNN
-F 4 "03-0204" H 0   0   50  0001 C CNN "HPN"
-	1    4200 3150
+F 0 "P4" H 4118 2819 50  0000 C CNN
+F 1 "LEM" H 4118 2910 50  0000 C CNN
+F 2 "tera_Connectors_Molex:Molex_PicoBlade_53398-0471_04x1.25mm_Straight" H 4200 3200 50  0001 C CNN
+F 3 "" H 4200 3200 50  0000 C CNN
+F 4 "03-0204" H 0   50  50  0001 C CNN "HPN"
+	1    4200 3200
 	1    0    0    1
 $EndComp
 $Comp
-L R_Small R2
+L Device:R_Small R2
 U 1 1 571E712E
 P 3750 3600
@@
 $EndComp
 $Comp
-L C_Small C3
+L Device:C_Small C3
 U 1 1 571E73F2
 P 4150 3900
@@
 $EndComp
 $Comp
-L ZENER D1
+L Device:D_Zener D1
 U 1 1 571E7460
 P 3750 4000
@@
 $EndComp
 $Comp
-L JUMPER3_NO JP2
+L tera_general:JUMPER3_NO JP2
 U 1 1 58454F62
 P 3900 2650
@@
 Examples:\nTERA Ibex with HASS 100-s: Supply=5V, Vref generation placed as shown\nTERA Fennek with HO 8-NP/SP33-1000: Supply = 3.3V, No external reference (Internal Vref = 1.65V)
 Wire Wire Line
-	1200 3100 1850 3100
+	1200 3100 1500 3100
 Wire Wire Line
 	1800 3100 1800 3200
@@
 	1800 3200 1850 3200
 Wire Wire Line
-	1200 3400 4000 3400
+	1200 3400 1500 3400
 Wire Wire Line
 	1850 3400 1850 3300
@@
 	1500 3350 1500 3400
 Wire Wire Line
-	2450 3100 4000 3100
+	2450 3100 2550 3100
 Wire Wire Line
 	2550 3100 2550 3150
@@
 	3900 3000 4000 3000
 Wire Wire Line
-	3600 4300 4150 4300
-Wire Wire Line
-	3750 4300 3750 4200
+	3600 4300 3750 4300
+Wire Wire Line
+	3750 4300 3750 4150
 Wire Wire Line
 	4150 4300 4150 4000
@@
 	3750 3200 4000 3200
 Wire Wire Line
-	3750 3700 3750 3800
-Wire Wire Line
-	3750 3750 4550 3750
+	3750 3700 3750 3750
+Wire Wire Line
+	3750 3750 4150 3750
 Wire Wire Line
 	4150 3750 4150 3800
@@
 Connection ~ 3750 3750
 Connection ~ 4150 3750
+Wire Wire Line
+	1800 3100 1850 3100
+Wire Wire Line
+	1500 3100 1800 3100
+Wire Wire Line
+	1500 3400 1850 3400
+Wire Wire Line
+	1850 3400 2550 3400
+Wire Wire Line
+	2550 3100 2900 3100
+Wire Wire Line
+	2550 3400 2900 3400
+Wire Wire Line
+	2900 3100 4000 3100
+Wire Wire Line
+	2900 3400 4000 3400
+Wire Wire Line
+	3750 4300 4150 4300
+Wire Wire Line
+	3750 3750 3750 3850
+Wire Wire Line
+	4150 3750 4550 3750
 $EndSCHEMATC
