File: HW/projects/ibex/BMS_Ibex/Master/BMS_Master_V6.1_kicad/SPI.sch (KiCad schematic (older format))
At the start: 15 parts, among them P15 SPI_Slaves, P16 DI_Slaves, U2 SN74HC138DR, U5 MAX3390EEUD

Commit message: Sync ibex bms with tera local
Parts:
- C14, C25, C26, C27: symbol C -> Device:C
- JP11: symbol JUMPER3_NO -> tera_general:JUMPER3_NO
- P15: symbol CONN_01X09 -> Connector_Generic:Conn_01x09
- P16: symbol CONN_01X02 -> Connector_Generic:Conn_01x02
- R21, R22, R41, R42, R43, R44: symbol R -> Device:R
- U2: symbol SN74HC138DR -> tera_logic:SN74HC138DR
- U5: symbol MAX3390EEUD -> tera_logic:MAX3390EEUD
Changed lines of the file:
@@
-EESchema Schematic File Version 2
-LIBS:power
-LIBS:device
-LIBS:transistors
-LIBS:conn
-LIBS:linear
-LIBS:regul
-LIBS:74xx
-LIBS:cmos4000
-LIBS:adc-dac
-LIBS:memory
-LIBS:xilinx
-LIBS:microcontrollers
-LIBS:dsp
-LIBS:microchip
-LIBS:analog_switches
-LIBS:motorola
-LIBS:texas
-LIBS:intel
-LIBS:audio
-LIBS:interface
-LIBS:digital-audio
-LIBS:philips
-LIBS:display
-LIBS:cypress
-LIBS:siliconi
-LIBS:opto
-LIBS:atmel
-LIBS:contrib
-LIBS:valves
-LIBS:ft232rl
-LIBS:relais
-LIBS:Supply
-LIBS:tera_general
-LIBS:tera_switches
-LIBS:tera_logic
-LIBS:tera_processors
-LIBS:tera_connectors
-LIBS:tera_emc_prodection
+EESchema Schematic File Version 4
 LIBS:BMS_Master_V6_kicad-cache
-EELAYER 25 0
+EELAYER 26 0
 EELAYER END
 $Descr A4 11693 8268
@@
 $EndDescr
 $Comp
-L CONN_01X09 P15
+L Connector_Generic:Conn_01x09 P15
 U 1 1 56FAD51B
 P 7300 1750
@@
 $EndComp
 $Comp
-L C C14
+L Device:C C14
 U 1 1 56FADBA9
 P 3500 3150
+AR Path="/56FADBA9" Ref="C14"  Part="1"
+AR Path="/56F507C6/56FADBA9" Ref="C14"  Part="1"
 F 0 "C14" V 3248 3150 50  0000 C CNN
 F 1 "100n" V 3339 3150 50  0000 C CNN
@@
 $EndComp
 $Comp
-L CONN_01X02 P16
+L Connector_Generic:Conn_01x02 P16
 U 1 1 56FAEA99
-P 7300 2450
-F 0 "P16" H 7378 2488 50  0000 L CNN
-F 1 "DI_Slaves" H 7378 2397 50  0000 L CNN
-F 2 "tera_Connectors_JST:JST_XH_B02B-XH-A_02x2.50mm_Straight" H 7300 2450 50  0001 C CNN
-F 3 "" H 7300 2450 50  0000 C CNN
-F 4 "02-0902" H 0   0   50  0001 C CNN "HPN"
-	1    7300 2450
+P 7300 2500
+F 0 "P16" H 7378 2538 50  0000 L CNN
+F 1 "DI_Slaves" H 7378 2447 50  0000 L CNN
+F 2 "tera_Connectors_JST:JST_XH_B02B-XH-A_02x2.50mm_Straight" H 7300 2500 50  0001 C CNN
+F 3 "" H 7300 2500 50  0000 C CNN
+F 4 "02-0902" H 0   50  50  0001 C CNN "HPN"
+	1    7300 2500
 	1    0    0    1
 $EndComp
 $Comp
-L R R22
+L Device:R R22
 U 1 1 56FAEBAB
 P 6950 2800
@@
 $EndComp
 $Comp
-L R R21
+L Device:R R21
 U 1 1 56FAEC22
 P 6700 2800
@@
 $EndComp
 $Comp
-L MAX3390EEUD U5
+L tera_logic:MAX3390EEUD U5
 U 1 1 57DC6F49
 P 4250 1750
@@
 $EndComp
 $Comp
-L C C25
+L Device:C C25
 U 1 1 57DC929F
 P 3500 1250
+AR Path="/57DC929F" Ref="C25"  Part="1"
+AR Path="/56F507C6/57DC929F" Ref="C25"  Part="1"
 F 0 "C25" V 3248 1250 50  0000 C CNN
 F 1 "100n" V 3339 1250 50  0000 C CNN
@@
 $EndComp
 $Comp
-L C C26
+L Device:C C26
 U 1 1 57DC946D
 P 4900 1300
+AR Path="/57DC946D" Ref="C26"  Part="1"
+AR Path="/56F507C6/57DC946D" Ref="C26"  Part="1"
 F 0 "C26" V 4648 1300 50  0000 C CNN
 F 1 "100n" V 4739 1300 50  0000 C CNN
@@
 $EndComp
 $Comp
-L C C27
+L Device:C C27
 U 1 1 57DCAEE5
 P 5100 1600
+AR Path="/57DCAEE5" Ref="C27"  Part="1"
+AR Path="/56F507C6/57DCAEE5" Ref="C27"  Part="1"
 F 0 "C27" V 4848 1600 50  0000 C CNN
 F 1 "1u" V 4939 1600 50  0000 C CNN
@@
 $EndComp
 $Comp
-L JUMPER3_NO JP11
+L tera_general:JUMPER3_NO JP11
 U 1 1 57E93E3B
 P 3100 1350
@@
 $EndComp
 $Comp
-L R R41
+L Device:R R41
 U 1 1 57E95229
 P 2150 3400
@@
 $EndComp
 $Comp
-L R R42
+L Device:R R42
 U 1 1 57E9534B
 P 2300 3400
@@
 $EndComp
 $Comp
-L R R43
+L Device:R R43
 U 1 1 57E95391
 P 2450 3400
@@
 $EndComp
 $Comp
-L R R44
+L Device:R R44
 U 1 1 57E95413
 P 2600 3400
@@
 $EndComp
 $Comp
-L SN74HC138DR U2
+L tera_logic:SN74HC138DR U2
 U 1 1 57F01901
 P 3200 4000
@@
 	3200 4650 3200 4600
 Wire Wire Line
-	2450 4650 3200 4650
+	2450 4650 2650 4650
 Wire Wire Line
 	2700 4250 2650 4250
 Wire Wire Line
-	2650 4250 2650 4650
+	2650 4250 2650 4350
 Wire Wire Line
 	2700 4350 2650 4350
@@
 	3200 3150 3200 3400
 Wire Wire Line
-	2000 3150 3350 3150
+	2000 3150 2150 3150
 Wire Wire Line
 	3700 3150 3650 3150
 Wire Wire Line
-	6550 3050 6950 3050
+	6550 3050 6700 3050
 Wire Wire Line
 	6950 3050 6950 2950
@@
 	6700 2950 6700 3050
 Wire Wire Line
-	6550 2500 7100 2500
-Wire Wire Line
-	6550 2400 7100 2400
+	6550 2500 6700 2500
+Wire Wire Line
+	6550 2400 6950 2400
 Wire Wire Line
 	4100 4350 3700 4350
@@
 	3850 1850 3850 2100
 Wire Wire Line
-	2900 1050 4150 1050
-Wire Wire Line
-	4350 1050 5400 1050
+	2900 1050 3100 1050
+Wire Wire Line
+	4350 1050 4900 1050
 Wire Wire Line
 	4900 1050 4900 1150
@@
 	4900 2100 4900 1450
 Wire Wire Line
-	3400 2100 5100 2100
+	3400 2100 3500 2100
 Wire Wire Line
 	4250 2050 4250 2100
@@
 	3200 1350 3950 1350
 Wire Wire Line
-	2000 3650 2700 3650
-Wire Wire Line
-	2000 3750 2700 3750
-Wire Wire Line
-	2000 3850 2700 3850
-Wire Wire Line
-	2000 4150 2700 4150
+	2000 3650 2150 3650
+Wire Wire Line
+	2000 3750 2300 3750
+Wire Wire Line
+	2000 3850 2450 3850
+Wire Wire Line
+	2000 4150 2600 4150
 Wire Wire Line
 	2150 3550 2150 3650
@@
 Connection ~ 2600 3150
 NoConn ~ 4550 1850
+Wire Wire Line
+	2650 4650 3200 4650
+Wire Wire Line
+	2650 4350 2650 4650
+Wire Wire Line
+	3200 3150 3350 3150
+Wire Wire Line
+	6700 3050 6950 3050
+Wire Wire Line
+	6700 2500 7100 2500
+Wire Wire Line
+	6950 2400 7100 2400
+Wire Wire Line
+	3500 1050 4150 1050
+Wire Wire Line
+	3500 2100 3850 2100
+Wire Wire Line
+	3850 2100 4250 2100
+Wire Wire Line
+	4900 1050 5100 1050
+Wire Wire Line
+	4250 2100 4900 2100
+Wire Wire Line
+	5100 1050 5400 1050
+Wire Wire Line
+	4900 2100 5100 2100
+Wire Wire Line
+	3100 1050 3500 1050
+Wire Wire Line
+	2150 3650 2700 3650
+Wire Wire Line
+	2300 3750 2700 3750
+Wire Wire Line
+	2450 3850 2700 3850
+Wire Wire Line
+	2600 4150 2700 4150
+Wire Wire Line
+	2150 3150 2300 3150
+Wire Wire Line
+	2300 3150 2450 3150
+Wire Wire Line
+	2450 3150 2600 3150
+Wire Wire Line
+	2600 3150 3200 3150
 $EndSCHEMATC
