File: HW/projects/ibex/BMS_Ibex/Master/BMS_Master_V6.1_kicad/TemperatureMeasurement.sch (KiCad schematic (older format))
At the start: 23 parts, among them IC8 LT1461ACS8-5, P21 TS3, P22 TS1, P23 TS4, P24 TS2

Commit message: Sync ibex bms with tera local
Parts:
- C17, C18, C19, C20, C21, C22: symbol C_Small -> Device:C_Small
- D24, D25, D26, D27: symbol ZENERsmall -> Device:D_Zener_Small
- IC8: symbol LT1461ACS8-5 -> Supply:LT1461ACS8-5
- P21, P22, P23, P24: symbol CONN_01X02 -> Connector_Generic:Conn_01x02
- R33, R34, R35, R36, R37, R38, R39, R40: symbol R_Small -> Device:R_Small
Changed lines of the file:
@@
-EESchema Schematic File Version 2
-LIBS:power
-LIBS:device
-LIBS:transistors
-LIBS:conn
-LIBS:linear
-LIBS:regul
-LIBS:74xx
-LIBS:cmos4000
-LIBS:adc-dac
-LIBS:memory
-LIBS:xilinx
-LIBS:microcontrollers
-LIBS:dsp
-LIBS:microchip
-LIBS:analog_switches
-LIBS:motorola
-LIBS:texas
-LIBS:intel
-LIBS:audio
-LIBS:interface
-LIBS:digital-audio
-LIBS:philips
-LIBS:display
-LIBS:cypress
-LIBS:siliconi
-LIBS:opto
-LIBS:atmel
-LIBS:contrib
-LIBS:valves
-LIBS:ft232rl
-LIBS:relais
-LIBS:Supply
-LIBS:tera_general
-LIBS:tera_switches
-LIBS:tera_logic
-LIBS:tera_processors
-LIBS:tera_connectors
-LIBS:tera_emc_prodection
+EESchema Schematic File Version 4
 LIBS:BMS_Master_V6_kicad-cache
-EELAYER 25 0
+EELAYER 26 0
 EELAYER END
 $Descr A4 11693 8268
@@
 $EndDescr
 $Comp
-L CONN_01X02 P22
+L Connector_Generic:Conn_01x02 P22
 U 1 1 572C6E5A
-P 2650 1600
-F 0 "P22" H 2569 1319 50  0000 C CNN
-F 1 "TS1" H 2569 1410 50  0000 C CNN
-F 2 "tera_Connectors_Molex:Molex_PicoBlade_53398-0271_02x1.25mm_Straight" H 2650 1600 50  0001 C CNN
-F 3 "" H 2650 1600 50  0000 C CNN
-F 4 "03-0202" H 0   0   50  0001 C CNN "HPN"
-	1    2650 1600
+P 2650 1650
+F 0 "P22" H 2569 1369 50  0000 C CNN
+F 1 "TS1" H 2569 1460 50  0000 C CNN
+F 2 "tera_Connectors_Molex:Molex_PicoBlade_53398-0271_02x1.25mm_Straight" H 2650 1650 50  0001 C CNN
+F 3 "" H 2650 1650 50  0000 C CNN
+F 4 "03-0202" H 0   50  50  0001 C CNN "HPN"
+	1    2650 1650
 	-1   0    0    1
 $EndComp
 $Comp
-L R_Small R34
+L Device:R_Small R34
 U 1 1 572C6F84
 P 2950 1800
@@
 $EndComp
 $Comp
-L C_Small C18
+L Device:C_Small C18
 U 1 1 572C6FE8
 P 3250 1800
@@
 $EndComp
 $Comp
-L R_Small R36
+L Device:R_Small R36
 U 1 1 572C707A
 P 3250 2100
@@
 $EndComp
 $Comp
-L ZENERsmall D25
+L Device:D_Zener_Small D25
 U 1 1 572C7151
 P 3500 2100
@@
 $EndComp
 $Comp
-L CONN_01X02 P21
+L Connector_Generic:Conn_01x02 P21
 U 1 1 572C83C4
-P 2600 2700
-F 0 "P21" H 2519 2419 50  0000 C CNN
-F 1 "TS3" H 2519 2510 50  0000 C CNN
-F 2 "tera_Connectors_Molex:Molex_PicoBlade_53398-0271_02x1.25mm_Straight" H 2600 2700 50  0001 C CNN
-F 3 "" H 2600 2700 50  0000 C CNN
-F 4 "03-0202" H 0   0   50  0001 C CNN "HPN"
-	1    2600 2700
+P 2600 2750
+F 0 "P21" H 2519 2469 50  0000 C CNN
+F 1 "TS3" H 2519 2560 50  0000 C CNN
+F 2 "tera_Connectors_Molex:Molex_PicoBlade_53398-0271_02x1.25mm_Straight" H 2600 2750 50  0001 C CNN
+F 3 "" H 2600 2750 50  0000 C CNN
+F 4 "03-0202" H 0   50  50  0001 C CNN "HPN"
+	1    2600 2750
 	-1   0    0    1
 $EndComp
 $Comp
-L R_Small R33
+L Device:R_Small R33
 U 1 1 572C83CA
 P 2900 2900
@@
 $EndComp
 $Comp
-L C_Small C17
+L Device:C_Small C17
 U 1 1 572C83D0
 P 3200 2900
@@
 $EndComp
 $Comp
-L R_Small R35
+L Device:R_Small R35
 U 1 1 572C83D6
 P 3200 3200
@@
 $EndComp
 $Comp
-L ZENERsmall D24
+L Device:D_Zener_Small D24
 U 1 1 572C83DC
 P 3450 3200
@@
 $EndComp
 $Comp
-L CONN_01X02 P24
+L Connector_Generic:Conn_01x02 P24
 U 1 1 572C8835
-P 4500 1600
-F 0 "P24" H 4419 1319 50  0000 C CNN
-F 1 "TS2" H 4419 1410 50  0000 C CNN
-F 2 "tera_Connectors_Molex:Molex_PicoBlade_53398-0271_02x1.25mm_Straight" H 4500 1600 50  0001 C CNN
-F 3 "" H 4500 1600 50  0000 C CNN
-F 4 "03-0202" H 0   0   50  0001 C CNN "HPN"
-	1    4500 1600
+P 4500 1650
+F 0 "P24" H 4419 1369 50  0000 C CNN
+F 1 "TS2" H 4419 1460 50  0000 C CNN
+F 2 "tera_Connectors_Molex:Molex_PicoBlade_53398-0271_02x1.25mm_Straight" H 4500 1650 50  0001 C CNN
+F 3 "" H 4500 1650 50  0000 C CNN
+F 4 "03-0202" H 0   50  50  0001 C CNN "HPN"
+	1    4500 1650
 	-1   0    0    1
 $EndComp
 $Comp
-L R_Small R38
+L Device:R_Small R38
 U 1 1 572C883B
 P 4800 1800
@@
 $EndComp
 $Comp
-L C_Small C20
+L Device:C_Small C20
 U 1 1 572C8841
 P 5100 1800
@@
 $EndComp
 $Comp
-L R_Small R40
+L Device:R_Small R40
 U 1 1 572C8847
 P 5100 2100
@@
 $EndComp
 $Comp
-L ZENERsmall D27
+L Device:D_Zener_Small D27
 U 1 1 572C884D
 P 5350 2100
@@
 $EndComp
 $Comp
-L CONN_01X02 P23
+L Connector_Generic:Conn_01x02 P23
 U 1 1 572C8864
-P 4450 2700
-F 0 "P23" H 4369 2419 50  0000 C CNN
-F 1 "TS4" H 4369 2510 50  0000 C CNN
-F 2 "tera_Connectors_Molex:Molex_PicoBlade_53398-0271_02x1.25mm_Straight" H 4450 2700 50  0001 C CNN
-F 3 "" H 4450 2700 50  0000 C CNN
-F 4 "03-0202" H 0   0   50  0001 C CNN "HPN"
-	1    4450 2700
+P 4450 2750
+F 0 "P23" H 4369 2469 50  0000 C CNN
+F 1 "TS4" H 4369 2560 50  0000 C CNN
+F 2 "tera_Connectors_Molex:Molex_PicoBlade_53398-0271_02x1.25mm_Straight" H 4450 2750 50  0001 C CNN
+F 3 "" H 4450 2750 50  0000 C CNN
+F 4 "03-0202" H 0   50  50  0001 C CNN "HPN"
+	1    4450 2750
 	-1   0    0    1
 $EndComp
 $Comp
-L R_Small R37
+L Device:R_Small R37
 U 1 1 572C886A
 P 4750 2900
@@
 $EndComp
 $Comp
-L C_Small C19
+L Device:C_Small C19
 U 1 1 572C8870
 P 5050 2900
@@
 $EndComp
 $Comp
-L R_Small R39
+L Device:R_Small R39
 U 1 1 572C8876
 P 5050 3200
@@
 $EndComp
 $Comp
-L ZENERsmall D26
+L Device:D_Zener_Small D26
 U 1 1 572C887C
 P 5300 3200
@@
 $EndComp
 $Comp
-L LT1461ACS8-5 IC8
+L Supply:LT1461ACS8-5 IC8
 U 1 1 56FBE7B0
 P 9000 1700
@@
 $EndComp
 $Comp
-L C_Small C21
+L Device:C_Small C21
 U 1 1 56FBEF9A
 P 8250 1750
@@
 $EndComp
 $Comp
-L C_Small C22
+L Device:C_Small C22
 U 1 1 56FBF749
 P 9450 1700
@@
 	3250 1550 3250 1700
 Wire Wire Line
-	3250 1900 3250 2000
-Wire Wire Line
-	2950 1950 3700 1950
+	3250 1900 3250 1950
+Wire Wire Line
+	2950 1950 3250 1950
 Wire Wire Line
 	2950 1950 2950 1900
@@
 	3250 2200 3250 2250
 Wire Wire Line
-	3100 2250 3500 2250
+	3100 2250 3250 2250
 Wire Wire Line
 	3500 2250 3500 2200
@@
 	3200 2650 3200 2800
 Wire Wire Line
-	3200 3000 3200 3100
-Wire Wire Line
-	2900 3050 3650 3050
+	3200 3000 3200 3050
+Wire Wire Line
+	2900 3050 3200 3050
 Wire Wire Line
 	2900 3050 2900 3000
@@
 	3200 3300 3200 3350
 Wire Wire Line
-	3050 3350 3450 3350
+	3050 3350 3200 3350
 Wire Wire Line
 	3450 3350 3450 3300
@@
 	5100 1550 5100 1700
 Wire Wire Line
-	5100 1900 5100 2000
-Wire Wire Line
-	4800 1950 5550 1950
+	5100 1900 5100 1950
+Wire Wire Line
+	4800 1950 5100 1950
 Wire Wire Line
 	4800 1950 4800 1900
@@
 	5100 2200 5100 2250
 Wire Wire Line
-	4950 2250 5350 2250
+	4950 2250 5100 2250
 Wire Wire Line
 	5350 2250 5350 2200
@@
 	5050 2650 5050 2800
 Wire Wire Line
-	5050 3000 5050 3100
-Wire Wire Line
-	4750 3050 5500 3050
+	5050 3000 5050 3050
+Wire Wire Line
+	4750 3050 5050 3050
 Wire Wire Line
 	4750 3050 4750 3000
@@
 	5050 3300 5050 3350
 Wire Wire Line
-	4900 3350 5300 3350
+	4900 3350 5050 3350
 Wire Wire Line
 	5300 3350 5300 3300
@@
 	5050 2650 4650 2650
 Wire Wire Line
-	9300 1600 9750 1600
-Wire Wire Line
-	8150 1600 8700 1600
+	9300 1600 9450 1600
+Wire Wire Line
+	8150 1600 8250 1600
 Wire Wire Line
 	8250 1650 8250 1600
@@
 	8250 1850 8250 1900
 Wire Wire Line
-	8150 1900 9450 1900
+	8150 1900 8250 1900
 Wire Wire Line
 	8700 1900 8700 1800
@@
 Connection ~ 8250 1600
 Connection ~ 8250 1900
+Wire Wire Line
+	3250 2250 3500 2250
+Wire Wire Line
+	3500 1950 3700 1950
+Wire Wire Line
+	3250 1950 3250 2000
+Wire Wire Line
+	3250 1950 3500 1950
+Wire Wire Line
+	3200 3350 3450 3350
+Wire Wire Line
+	3450 3050 3650 3050
+Wire Wire Line
+	3200 3050 3200 3100
+Wire Wire Line
+	3200 3050 3450 3050
+Wire Wire Line
+	5100 2250 5350 2250
+Wire Wire Line
+	5350 1950 5550 1950
+Wire Wire Line
+	5100 1950 5100 2000
+Wire Wire Line
+	5100 1950 5350 1950
+Wire Wire Line
+	5050 3350 5300 3350
+Wire Wire Line
+	5300 3050 5500 3050
+Wire Wire Line
+	5050 3050 5050 3100
+Wire Wire Line
+	5050 3050 5300 3050
+Wire Wire Line
+	8700 1900 9450 1900
+Wire Wire Line
+	9450 1600 9750 1600
+Wire Wire Line
+	8250 1600 8700 1600
+Wire Wire Line
+	8250 1900 8700 1900
 $EndSCHEMATC
