File: HW/projects/ibex/BMS_Ibex/Master/BMS_Master_V6.2_kicad/BMS_Master_V6_kicad.kicad_pcb (KiCad board)
At the start: 4 copper layers, 93.5 x 61 mm, 143 parts, among them IC1 LM4132A-1.8, IC2 LM4132A-1.8, IC3 LM4132A-1.8, IC4 TLE8102SG, IC5 TLE8102SG, IC6 TLE8102SG, IC7 TLE8102SG, IC8 LT1461ACS8-5, P1 Interlock, P10 K_CH2, P11 K_CH1, P12 K_CH2, P13 K_CH1, P14 K_CH2, P15 SPI_Slaves, P16 DI_Slaves, P17 CAN_CON_2pol, P19 12V_CRTL, P2 12V_IL, P20 12V_PWR, P21 TS3, P22 TS1, P23 TS4, P24 TS2, P3 ExtGPIO, P4 LEM, P5 LEM, P6 LEM, P7 K_CH1, P8 K_CH2, P9 K_CH1, Q1 BSS205N, Q2 BSS205N, U1 STM32f4_board_v3-1, U2 SN74HC138DR, U5 MAX3390EEUD

Commit message: Sync ibex bms with tera local
Parts:
- removed D20: 5V, tera_diodes:DO-216AA
- removed D21, D26: 3V3, tera_diodes:DO-216AA
- removed JP11: JUMPER3_NO, tera_general:SOLDERJUMPER_3
- removed P16: DI_Slaves, tera_Connectors_JST:JST_XH_B02B-XH-A_02x2.50mm_Straight
- removed P23: TS4, tera_Connectors_Molex:Molex_PicoBlade_53398-0271_02x1.25mm_Straight
- removed R39: ?R, tera_rlc:R_0603in
- added C15: 100n, tera_rlc:C_0603in, F.Cu at (84.0, 85.0)
- added C23: 100n, tera_rlc:C_0603in, F.Cu at (86.0, 85.0)
- added C24: 100n, tera_rlc:C_0603in, B.Cu at (140.5, 103.2)
- added C28: 100n, tera_rlc:C_0603in, B.Cu at (138.1, 106.5)
- added C29: 4u7, tera_rlc:C_0805in, B.Cu at (102.1, 96.9)
- added C30: 4u7, tera_rlc:C_0805in, B.Cu at (132.8, 92.8)
- added C31: 4u7, tera_rlc:C_0805in, B.Cu at (95.4, 94.7)
- added C32: 100n, tera_rlc:C_0603in, B.Cu at (80.3, 100.8)
- added C33: 100n, tera_rlc:C_0603in, B.Cu at (85.0, 103.5)
- added C34: 100n, tera_rlc:C_0603in, B.Cu at (85.0, 110.0)
- added C35: 100n, tera_rlc:C_0603in, B.Cu at (80.0, 107.2)
- added D12: 3V3, tera_diodes:uClamp3310D_tvs_3v3, B.Cu at (127.3, 69.5)
- added D13: 3V3, tera_diodes:uClamp3310D_tvs_3v3, F.Cu at (127.3, 68.3)
- added D28: 3V3, tera_diodes:uClamp3310D_tvs_3v3, F.Cu at (127.3, 74.7)
- added G1: TSR_0.5-2450, traco_power:TSR_0.5, F.Cu at (135.0, 91.8)
- added G2: TSR_0.5-2433, traco_power:TSR_0.5, F.Cu at (98.0, 92.3)
- added JP5: Jumper_NO_Small, tera_general:SOLDERJUMPER_2_1mm, B.Cu at (133.9, 73.5)
- added JP6: Jumper_NO_Small, tera_general:SOLDERJUMPER_2_1mm, B.Cu at (133.9, 72.0)
- added JP7: Jumper_NO_Small, tera_general:SOLDERJUMPER_2_1mm, B.Cu at (133.9, 70.5)
- added L1: 3u3, tera_rlc:L_0805in, B.Cu at (135.0, 95.0)
- added L3: 3u3, tera_rlc:L_0805in, B.Cu at (99.8, 94.7)
- added P18: Buttons, tera_Connectors_JST:JST_EH_B03B-EH-A_03x2.50mm_Straight, F.Cu at (85.8, 97.8)
- added Q3: BSS205N, tera_atomic_infineon:BSS205N, F.Cu at (81.5, 101.0)
- added Q4: BSS205N, tera_atomic_infineon:BSS205N, F.Cu at (81.5, 96.2)
- added Q5: BSS205N, tera_atomic_infineon:BSS205N, F.Cu at (79.5, 91.5)
- added Q6: BSS205N, tera_atomic_infineon:BSS205N, F.Cu at (112.1, 64.0)
- added R23: 10k, tera_rlc:R_0603in, B.Cu at (138.8, 112.2)
- added R24: 100R, tera_rlc:R_0603in, F.Cu at (127.3, 72.7)
- added R25: 100R, tera_rlc:R_0603in, F.Cu at (127.3, 70.3)
- added R26: 100R, tera_rlc:R_0603in, B.Cu at (127.3, 71.5)
- added R45: 2K2, tera_rlc:R_0603in, F.Cu at (78.5, 95.4)
- added R46: 2K2, tera_rlc:R_0603in, F.Cu at (78.5, 99.0)
- added R47: 2K2, tera_rlc:R_0603in, F.Cu at (78.5, 102.9)
- added R48: 1K, tera_rlc:R_0603in, F.Cu at (86.0, 88.5)
- added R49: 1K, tera_rlc:R_0603in, F.Cu at (84.0, 88.5)
- added U3: HostFilter, local_footprints:HostFilter, F.Cu at (139.6, 81.4)
- C19: value 100n -> 4u7; footprint tera_rlc:C_0603in -> tera_rlc:C_0805in
- D1, D2, D24, D25, D27, D3: footprint tera_diodes:DO-216AA -> tera_diodes:uClamp3310D_tvs_3v3
- P15: value SPI_Slaves -> Debug_USART; footprint tera_Connectors_Molex:Molex_PicoBlade_53398-0971_09x1.25mm_Straight -> tera_Connectors_Molex:Molex_KK-254_AE-6410-03A_1x03_P2.54mm_Vertical
- P20: footprint tera_Connectors_Phoenix:MCV_1.5_2-GF-3.5 -> tera_Connectors_Phoenix:PhoenixContact_MC-GF_02x3.50mm_Angled_ThreadedFlange
- P3: value ExtGPIO -> Ext_LED; footprint tera_Connectors_JST:JST_EH_B05B-EH-A_05x2.50mm_Straight -> tera_Connectors_JST:JST_EH_B04B-EH-A_04x2.50mm_Straight
- R14, R30: moved to B.Cu
- R2, R32, R4, R41, R42, R43, R6: footprint tera_rlc:R_0805in -> tera_rlc:R_0603in
- R21: value 10k -> 1k; footprint tera_rlc:R_0805in -> tera_rlc:R_0603in
- R22: value 10k -> 1K; footprint tera_rlc:R_0805in -> tera_rlc:R_0603in
- R37: value ?R -> 1K
- R44: value 1k -> 10k; footprint tera_rlc:R_0805in -> tera_rlc:R_0603in
- moved R22 67.5 mm to (80.0, 104.0), turned to 270 degrees
- moved P15 65.1 mm to (82.3, 111.7), turned to 90 degrees
- moved C19 34.4 mm to (135.5, 99.0), turned to 270 degrees
- moved REF*** 33.1 mm to (94.7, 63.2)
- moved R21 23.9 mm to (140.4, 106.5), turned to 90 degrees
- moved R37 17.7 mm to (85.0, 106.7), turned to 270 degrees
- moved svg2mod 16.7 mm to (133.8, 74.8)
- moved R32 8.80 mm to (104.4, 94.1)
- moved R14 7.89 mm to (123.2, 67.1), turned to 0 degrees
- moved R40 7.73 mm to (93.0, 102.6)
- moved D27 7.12 mm to (93.0, 102.6), turned to 0 degrees
- moved D25 6.69 mm to (88.3, 102.5), turned to 180 degrees
- moved P22 6.36 mm to (87.8, 108.4)
- moved D23 6.07 mm to (102.7, 102.7)
- moved R2 6.04 mm to (112.5, 92.0), turned to 270 degrees
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Connections:
- C19 pad 1: /TemperatureMeasurement/V_ref -> +12V
- C19 pad 2: /TS4 -> GND
- C3 pad 1: /LEM1 -> Net-(C3-Pad1)
- C6 pad 1: /LEM2 -> Net-(C6-Pad1)
- C9 pad 1: /LEM3 -> Net-(C9-Pad1)
- D1 pad 1: /LEM1 -> Net-(C3-Pad1)
- D2 pad 1: /LEM2 -> Net-(C6-Pad1)
- D3 pad 1: /LEM3 -> Net-(C9-Pad1)
- P1 pad 4: /Interlock_OK -> Net-(C28-Pad2)
- P15 pad 1: GND -> Net-(C35-Pad1)
- P15 pad 2: /SPI_Controller/NCS4 -> Net-(C34-Pad1)
- P15 pad 3: /SPI_Controller/NCS3 -> GND
- P3 pad 1: GND -> Net-(P3-Pad1)
- P3 pad 2: /EXT_GPIO_3 -> Net-(P3-Pad2)
- P3 pad 3: /EXT_GPIO_2 -> Net-(P3-Pad3)
- P3 pad 4: /EXT_GPIO_1 -> +5V
- P4 pad 2: Net-(P4-Pad2) -> Net-(C3-Pad1)
- P5 pad 2: Net-(P5-Pad2) -> Net-(C6-Pad1)
- P6 pad 2: Net-(P6-Pad2) -> Net-(C9-Pad1)
- R2 pad 1: Net-(P4-Pad2) -> /LEM1
- R2 pad 2: /LEM1 -> Net-(C3-Pad1)
- R21 pad 1: /NFAULT -> Net-(C28-Pad2)
- R21 pad 2: GND -> /Interlock_OK
- R22 pad 1: /NALERT -> /RS232/RxD
- R22 pad 2: GND -> Net-(C35-Pad1)
- R37 pad 1: Net-(P23-Pad1) -> /RS232/TxD
- R37 pad 2: /TS4 -> Net-(C34-Pad1)
- R4 pad 1: Net-(P5-Pad2) -> /LEM2
- R4 pad 2: /LEM2 -> Net-(C6-Pad1)
- R44 pad 1: +5V -> Net-(Q6-Pad3)
- R44 pad 2: /SPI_CS -> +5V
- R6 pad 1: Net-(P6-Pad2) -> /LEM3
- R6 pad 2: /LEM3 -> Net-(C9-Pad1)
- U1 pad 10: /Interlock_On1 -> /~TMP_REF_SHDN
- U1 pad 11: /Interlock_On2 -> Net-(U1-Pad11)
- U1 pad 12: Net-(U1-Pad12) -> /BTN_ON
- U1 pad 13: Net-(U1-Pad13) -> /BTN_OFF
- U1 pad 14: /EXT_GPIO_3 -> /EXT_LED_1
- U1 pad 15: /EXT_GPIO_2 -> /EXT_LED_2
- U1 pad 16: /EXT_GPIO_1 -> /EXT_LED_3
- U1 pad 49: /Precharge_Fault -> /NALERT
- U1 pad 55: /TS4 -> /Interlock_OK
- U1 pad 6: Net-(U1-Pad6) -> /RS232/TxD
- U1 pad 7: Net-(U1-Pad7) -> /RS232/RxD
- U1 pad 71: /Interlock_OK -> /Interlock_On2
- U1 pad 72: /~TMP_REF_SHDN -> /Interlock_On1
- U1 pad 76: /NALERT -> /Precharge_Fault
- U2 pad 5: GND -> Net-(Q6-Pad3)
- U2 pad 6: /SPI_CS -> +5V
- U5 pad 2: /MISO -> /SPI_Controller/MISO_3V3
- U5 pad 3: /MOSI -> /SPI_Controller/MOSI_3V3
- U5 pad 4: /SCLK -> /SPI_Controller/SCLK_3V3
- U5 pad 5: GND -> Net-(U5-Pad5)
- U5 pad 8: Net-(JP11-Pad2) -> /SPI_CS
Routing:
- net +3V3: track 68.1 -> 21.8 mm, vias 16 -> 15
- net /RS232/TxD: track 0.00 -> 45.7 mm, vias 0 -> 1
- net /TS4: track 42.5 -> 0.00 mm, vias 3 -> 0
- net /Interlock_On2: track 85.2 -> 44.7 mm, vias 2 -> 1
- net /Interlock_On1: track 87.6 -> 47.5 mm, vias 2 -> 1
- net /RS232/RxD: track 0.00 -> 37.5 mm, vias 0 -> 1
- net /EXT_GPIO_3: track 30.5 -> 0.00 mm
- net /EXT_LED_3: track 0.00 -> 30.5 mm
- net /EXT_GPIO_2: track 27.1 -> 0.00 mm
- net +12V: track 2.36 -> 29.0 mm
- net /EXT_LED_2: track 0.00 -> 25.8 mm
- net /EXT_GPIO_1: track 23.7 -> 0.00 mm
- net /EXT_LED_1: track 0.00 -> 21.3 mm
- net /~TMP_REF_SHDN: track 44.4 -> 65.1 mm
- net /BTN_ON: track 0.00 -> 20.1 mm
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- added copper zone on B.Cu, net +12V
- added copper zone on B.Cu, net Net-(C30-Pad1)
- added copper zone on B.Cu, net Net-(C31-Pad1)
- removed copper zone on B.Cu, net +3V3
Other:
- board text added: "BMS Master V6.2 TERA TU Graz ©Pöschl, Apr. 2018 Solderpad v0.51"
- board text added: "©Pöschl, 2018 Solderpad v0.51"
- board text removed: "BMS Master V6.1"
- board text removed: "BMS Master V6.2 TERA TU Graz ©Pöschl, Jun.2017 Solderpad v0.51"
- board text removed: "©Pöschl, 2017 Solderpad v0.51"
