File: HW/projects/ibex/BMS_Ibex/Master/BMS_Master_V6.2_kicad/BMS_Master_V6_kicad.sch (KiCad schematic (older format))
At the start: 6 parts, among them P1 Interlock, P2 12V_IL, P3 ExtGPIO, U1 STM32f4_board_v3-1

Commit message: Sync ibex bms with tera local
Parts:
- removed P3: ExtGPIO, tera_Connectors_JST:JST_EH_B05B-EH-A_05x2.50mm_Straight, symbol CONN_01X05
- added C24, C28: 100n, tera_rlc:C_0603in, symbol Device:C
- added R21: 1k, tera_rlc:R_0603in, symbol Device:R
- JP1: symbol Jumper_NO_Small -> Device:Jumper_NO_Small
- P1: symbol CONN_01X05 -> Connector_Generic:Conn_01x05
- P2: symbol CONN_01X02 -> Connector_Generic:Conn_01x02
- R23: renamed from R?; footprint tera_rlc:R_0805in -> tera_rlc:R_0603in; symbol R -> Device:R; HPN 11-1K00 -> 11-10K0
- U1: symbol STM32f4_board_v3-1 -> tera_general:STM32f4_board_v3-1
Connections:
- net TS4 is gone; now on net Interlock_OK: U1.55 (PC3)
- net GND: now also C24.1, C28.1
- net Interlock_OK: now also C24.2, R21.2; no longer P1.4 (P4), R23.1, U1.71 (PC4)
- net Interlock_On1: now also U1.72 (PC5); no longer U1.10 (PB6)
- net Interlock_On2: now also U1.71 (PC4); no longer U1.11 (PB7)
- net NALERT: now also U1.49 (PC8); no longer U1.76 (PB10)
- net Precharge_Fault: now also U1.76 (PB10); no longer U1.49 (PC8)
- net ~TMP_REF_SHDN: now also U1.10 (PB6); no longer U1.72 (PC5)
- net BTN_ON: now reaches U1.12 (PB8)
- net BTN_OFF: now reaches U1.13 (PB9)
- net RS232/TxD: now reaches U1.6 (DebugTXD)
- net RS232/RxD: now reaches U1.7 (DebugRXD)
- net EXT_GPIO_1 renamed EXT_LED_3
- net EXT_GPIO_2 renamed EXT_LED_2
- net EXT_GPIO_3 renamed EXT_LED_1
- new net: C28.2, P1.4 (Pin_4), R21.1, R23.1
- no-connect marks 20 -> 17
Other:
- moved on the sheet: R23
