File: HW/projects/ibex/BMS_Ibex/Master/BMS_Master_V6.2_kicad/CAN.sch (KiCad schematic (older format))
At the start: 10 parts, among them P17 CAN_CON_2pol

Commit message: Sync ibex bms with tera local
Parts:
- C15: symbol C -> Device:C
- D12, D13: symbol SUPPRESSOR -> tera_general:SUPPRESSOR
- JP7, JP8: symbol Jumper_NO_Small -> Device:Jumper_NO_Small
- L1: symbol CM_CHOKE -> tera_general:CM_CHOKE
- P17: symbol CAN_CON_2pol -> tera_connectors:CAN_CON_2pol
- R24, R25: symbol R -> Device:R
- S1: symbol SWITCH_DPDT -> tera_switches:SWITCH_DPDT
Changed lines of the file:
@@
-EESchema Schematic File Version 2
-LIBS:power
-LIBS:device
-LIBS:transistors
-LIBS:conn
-LIBS:linear
-LIBS:regul
-LIBS:74xx
-LIBS:cmos4000
-LIBS:adc-dac
-LIBS:memory
-LIBS:xilinx
-LIBS:microcontrollers
-LIBS:dsp
-LIBS:microchip
-LIBS:analog_switches
-LIBS:motorola
-LIBS:texas
-LIBS:intel
-LIBS:audio
-LIBS:interface
-LIBS:digital-audio
-LIBS:philips
-LIBS:display
-LIBS:cypress
-LIBS:siliconi
-LIBS:opto
-LIBS:atmel
-LIBS:contrib
-LIBS:valves
-LIBS:ft232rl
-LIBS:relais
-LIBS:Supply
-LIBS:tera_general
-LIBS:tera_switches
-LIBS:tera_logic
-LIBS:tera_processors
-LIBS:tera_connectors
-LIBS:tera_emc_prodection
+EESchema Schematic File Version 4
 LIBS:BMS_Master_V6_kicad-cache
-EELAYER 25 0
+EELAYER 26 0
 EELAYER END
 $Descr A4 11693 8268
 encoding utf-8
-Sheet 14 14
+Sheet 14 16
 Title "BMS Master"
 Date "2017-01-06"
@@
 $EndDescr
 $Comp
-L SUPPRESSOR D13
+L tera_general:SUPPRESSOR D13
 U 1 1 56F60DD7
 P 7300 3250
@@
 $EndComp
 $Comp
-L Jumper_NO_Small JP7
+L Device:Jumper_NO_Small JP7
 U 1 1 56F60DD8
 P 5450 2250
@@
 $EndComp
 $Comp
-L Jumper_NO_Small JP8
+L Device:Jumper_NO_Small JP8
 U 1 1 56F60DD9
 P 5450 3250
@@
 $EndComp
 $Comp
-L SUPPRESSOR D12
+L tera_general:SUPPRESSOR D12
 U 1 1 56F60DDA
 P 4650 3300
@@
 $EndComp
 $Comp
-L R R24
+L Device:R R24
 U 1 1 56F60DDB
 P 6350 3850
@@
 $EndComp
 $Comp
-L R R25
+L Device:R R25
 U 1 1 56F60DDC
 P 6550 3850
@@
 $EndComp
 $Comp
-L C C15
+L Device:C C15
 U 1 1 56F60DDD
 P 6450 4150
@@
 AR Path="/56F507DC/56F5B634/56F60DDD" Ref="C16"  Part="1"
 AR Path="/58175C82/56F60DDD" Ref="C16"  Part="1"
+AR Path="/56F60DDD" Ref="C16"  Part="1"
 F 0 "C16" H 6475 4250 50  0000 L CNN
 F 1 "47nF" H 6475 4050 50  0000 L CNN
@@
 $EndComp
 $Comp
-L CM_CHOKE L1
+L tera_general:CM_CHOKE L1
 U 1 1 56F60DE1
 P 5450 2750
@@
 $EndComp
 $Comp
-L CAN_CON_2pol P17
+L tera_connectors:CAN_CON_2pol P17
 U 1 1 581338CD
 P 8750 2700
@@
 $EndComp
 $Comp
-L SWITCH_DPDT S1
+L tera_switches:SWITCH_DPDT S1
 U 1 1 5816ED00
 P 6500 3150
