File: HW/projects/ibex/BMS_Ibex/Master/BMS_Master_V6.2_kicad/SPI.sch (KiCad schematic (older format))
At the start: 17 parts, among them P15 SPI_Slaves, P16 DI_Slaves, U2 SN74HC138DR, U5 MAX3390EEUD

Commit message: Sync ibex bms with tera local
Parts:
- removed P15: SPI_Slaves, tera_Connectors_Molex:Molex_PicoBlade_53398-0971_09x1.25mm_Straight, symbol CONN_01X09
- removed P16: DI_Slaves, tera_Connectors_JST:JST_XH_B02B-XH-A_02x2.50mm_Straight, symbol CONN_01X02
- removed R21, R22: 10k, tera_rlc:R_0805in, symbol R
- added D12, D13, D28: 3V3, tera_diodes:uClamp3310D_tvs_3v3, symbol Device:D_Zener_Small
- added JP5, JP6, JP7: Jumper_NO_Small, tera_general:SOLDERJUMPER_2_1mm, symbol Device:Jumper_NO_Small
- added Q6: BSS205N, tera_atomic_infineon:BSS205N, symbol tera_general:BSS205N
- added U3: HostFilter, local_footprints:HostFilter, symbol local_symbols:HostFilter
- C14, C25, C26, C27: symbol C -> Device:C
- R24, R25, R26: renamed from R?; value 1k -> 100R; footprint tera_rlc:R_0805in -> tera_rlc:R_0603in; symbol R -> Device:R; HPN 11-1K00 -> 11-100R
- R41, R42, R43: footprint tera_rlc:R_0805in -> tera_rlc:R_0603in; symbol R -> Device:R
- R44: value 1k -> 10k; footprint tera_rlc:R_0805in -> tera_rlc:R_0603in; symbol R -> Device:R; HPN 11-1K00 -> 11-10K0
- U2: symbol SN74HC138DR -> tera_logic:SN74HC138DR
- U5: symbol MAX3390EEUD -> tera_logic:MAX3390EEUD
Connections:
- net +5V: now also R44.2, U2.6 (E3), U3.4 (+5V); no longer R44.1
- net GND: now also D12.2 (A), D13.2 (A), D28.2 (A), Q6.2 (S), U3.1 (GND), U3.15 (GND), U3.16 (GND), U3.6 (GND), U3.7 (GND); no longer R24.2, R25.2, R26.2, U2.5 (E2), U5.5 (IN4)
- net MISO: now also R24.2, D28.1 (K); no longer U5.2 (OUT1)
- net MISO_5V: now also JP5.2, U3.9 (MISO); no longer R26.1
- net MOSI: now also R25.2, D13.1 (K); no longer R24.1, U5.3 (IN2)
- net MOSI_5V: now also JP6.2, U3.11 (MOSI)
- net NALERT: now also U3.5 (~Alert)
- net NCS1: now also U3.8 (NCS1)
- net NCS2: now also U3.10 (NCS2)
- net NCS3: now also U3.12 (NCS3)
- net NCS4: now also U3.14 (NCS4)
- net NFAULT: now also U3.3 (~Fault)
- net SCLK: now also R26.2, D12.1 (K); no longer R25.1, U5.4 (IN3)
- net SCLK_5V: now also JP7.2, U3.13 (SCLK)
- net SPI_CS: now also U5.8 (EN1), Q6.1 (G); no longer R44.2, U2.6 (E3)
- new net: Q6.3 (D), R44.1, U2.5 (E2)
- new net +12V: U3.2 (+12V)
- new net MISO_3V3: JP5.1, R24.1, U5.2 (OUT1)
- new net MOSI_3V3: JP6.1, R25.1, U5.3 (IN2)
- new net SCLK_3V3: JP7.1, R26.1, U5.4 (IN3)
- no-connect marks 1 -> 2
Other:
- note removed: "5V SPI should be better in an noisy environment!"
- note removed: "EN input should not exceed 3.3+0.4V\nIf 5V pullups are used, permanently disable thristade mode!"
- note removed: "Resistors for broken\nwire detection."
- moved on the sheet: C26, C27, R24, R25, R26, R44
