File: HW/projects/ibex/BMS_Ibex/Master/BMS_Master_V6.2_kicad/TemperatureMeasurement.sch (KiCad schematic (older format))
At the start: 23 parts, among them IC8 LT1461ACS8-5, P21 TS3, P22 TS1, P23 TS4, P24 TS2

Commit message: Sync ibex bms with tera local
Parts:
- removed C19: 100n, tera_rlc:C_0603in, symbol C_Small
- removed D26: 3V3, tera_diodes:DO-216AA, symbol ZENERsmall
- removed P23: TS4, tera_Connectors_Molex:Molex_PicoBlade_53398-0271_02x1.25mm_Straight, symbol CONN_01X02
- removed R37, R39: ?R, tera_rlc:R_0603in, symbol R_Small
- C17, C18, C20, C21, C22: symbol C_Small -> Device:C_Small
- D24, D25, D27: footprint tera_diodes:DO-216AA -> tera_diodes:uClamp3310D_tvs_3v3; symbol ZENERsmall -> Device:D_Zener_Small
- IC8: symbol LT1461ACS8-5 -> Supply:LT1461ACS8-5
- P21, P22, P24: symbol CONN_01X02 -> Connector_Generic:Conn_01x02
- R33, R34, R35, R36, R38, R40: symbol R_Small -> Device:R_Small
