File: HW/projects/ibex/BMS_Ibex/Master/BMS_Master_V6.2_kicad/supply.sch (KiCad schematic (older format))
At the start: 16 parts, among them P19 12V_CRTL, P20 12V_PWR

Commit message: Sync ibex bms with tera local
Parts:
- removed D20: 5V, tera_diodes:DO-216AA, symbol ZENER
- removed D21: 3V3, tera_diodes:DO-216AA, symbol ZENER
- added C19, C29, C30, C31: 4u7, tera_rlc:C_0805in, symbol Device:C_Small
- added G1: TSR_0.5-2450, traco_power:TSR_0.5, symbol Supply:TSR_0.5-2450
- added G2: TSR_0.5-2433, traco_power:TSR_0.5, symbol Supply:TSR_0.5-2433
- added L1, L3: 3u3, tera_rlc:L_0805in, symbol Device:L_Small
- D16, D17: symbol ZENER -> Device:D_Zener
- D18, D19, D22, D23: symbol LED -> BMS_Master_V6_kicad-rescue:LED-RESCUE-BMS_Master_V6_kicad
- P19: symbol CONN_01X02 -> Connector_Generic:Conn_01x02
- P20: footprint tera_Connectors_Phoenix:MCV_1.5_2-GF-3.5 -> tera_Connectors_Phoenix:PhoenixContact_MC-GF_02x3.50mm_Angled_ThreadedFlange; symbol CONN_01X02 -> Connector_Generic:Conn_01x02
- PS1, PS2: symbol DCDC_Stepdown_v6 -> tera_general:DCDC_Stepdown_v6
- R29, R30, R31: symbol R -> Device:R
- R32: footprint tera_rlc:R_0805in -> tera_rlc:R_0603in; symbol R -> Device:R
Connections:
- net +12V_CRTL: now also C19.1, C29.1, L1.2, L3.2
- net +3V3: now also G2.3 (Vout)
- net +5V: now also G1.3 (Vout)
- net GND: now also C19.2, C29.2, C30.2, C31.2, G1.2 (GND), G2.2 (GND)
- new net: C31.1, G2.1 (Vin), L3.1
- new net: C30.1, G1.1 (Vin), L1.1
Other:
- note added: "Example inductor: \nCPI0805E3R3R-10"
- note added: "Replacement for TERA DC/DC\n\nInput filter should not be necessary for our application."
- moved on the sheet: D16, D17
