File: HW/projects/ibex/BMS_Ibex/Messboard/bms_board_V5.1/bms_board.kicad_pcb (KiCad board)
At the start: 4 copper layers, 39 x 42 mm, 66 parts, among them CON1 TS1, CON2 TS2, CON3 Host_Interface, IC1 TI-bq76pl536, Q1 BSS205N, Q2 BSS205N, X1 DaisyChain_North, X10 DaisyChain_South, X3 Balancer_Interface, X7 Prog_Voltage

Commit message: Sync ibex bms with tera local
Parts:
- added JP2: Jumper_NO_Small, tera_general:SOLDERJUMPER_2_1mm, F.Cu at (66.4, 135.5)
- added JP3: Jumper_NO_Small, tera_general:SOLDERJUMPER_2_1mm, F.Cu at (80.8, 112.4)
- moved R5 4.01 mm to (81.2, 118.4)
- moved JP1 0.53 mm to (81.2, 115.9)
Connections:
- X1 pad 9: +BATT -> Net-(JP3-Pad2)
- X10 pad 9: GND -> Net-(JP2-Pad2)
Routing:
- net /+5V_LDOA: track 26.5 -> 22.1 mm
- net Net-(JP2-Pad2): track 0.00 -> 2.86 mm
- net Net-(JP3-Pad2): track 0.00 -> 2.72 mm
- net GND: track 22.4 -> 20.6 mm, vias 20 -> 22
- net Net-(JP1-Pad3): track 1.93 -> 2.54 mm
- net +BATT: vias 3 -> 4
