File: HW/projects/ibex/BMS_Ibex/Messboard/bms_board_V5.1/bms_board.sch (KiCad schematic (older format))
At the start: 62 parts, among them CON1 TS1, CON2 TS2, CON3 Host_Interface, IC1 TI-bq76pl536, Q1 BSS205N, Q2 BSS205N, X1 DaisyChain_North, X10 DaisyChain_South, X3 Balancer_Interface, X7 Prog_Voltage

Commit message: Sync ibex bms with tera local
Parts:
- added JP2, JP3: Jumper_NO_Small, tera_general:SOLDERJUMPER_2_1mm, symbol Jumper_NO_Small
Connections:
- net +BATT: now also JP3.1; no longer X1.9 (P9)
- net GND: now also JP2.1; no longer X10.9 (P9)
- new net: JP2.2, X10.9 (P9)
- new net: JP3.2, X1.9 (P9)
Changed lines of the file:
@@
 $EndDescr
 $Comp
-L GND #PWR01
+L GND #PWR7
 U 1 1 56EB298C
 P 2050 2150
-F 0 "#PWR01" H 2050 1900 50  0001 C CNN
+F 0 "#PWR7" H 2050 1900 50  0001 C CNN
 F 1 "GND" H 2058 1977 50  0000 C CNN
 F 2 "" H 2050 2150 50  0000 C CNN
@@
 $EndComp
 $Comp
-L GND #PWR02
+L GND #PWR5
 U 1 1 56EB2BB3
 P 1550 2000
-F 0 "#PWR02" H 1550 1750 50  0001 C CNN
+F 0 "#PWR5" H 1550 1750 50  0001 C CNN
 F 1 "GND" H 1558 1827 50  0000 C CNN
 F 2 "" H 1550 2000 50  0000 C CNN
@@
 $EndComp
 $Comp
-L GND #PWR03
+L GND #PWR11
 U 1 1 56EB2C48
 P 3100 1050
-F 0 "#PWR03" H 3100 800 50  0001 C CNN
+F 0 "#PWR11" H 3100 800 50  0001 C CNN
 F 1 "GND" H 3108 877 50  0000 C CNN
 F 2 "" H 3100 1050 50  0000 C CNN
@@
 $EndComp
 $Comp
-L +5V #PWR04
+L +5V #PWR8
 U 1 1 56EB2CF0
 P 2650 950
-F 0 "#PWR04" H 2650 800 50  0001 C CNN
+F 0 "#PWR8" H 2650 800 50  0001 C CNN
 F 1 "+5V" H 2668 1123 50  0000 C CNN
 F 2 "" H 2650 950 50  0000 C CNN
@@
 $EndComp
 $Comp
-L GND #PWR05
+L GND #PWR13
 U 1 1 56EB3A5D
 P 3900 1600
-F 0 "#PWR05" H 3900 1350 50  0001 C CNN
+F 0 "#PWR13" H 3900 1350 50  0001 C CNN
 F 1 "GND" H 3908 1427 50  0000 C CNN
 F 2 "" H 3900 1600 50  0000 C CNN
@@
 $EndComp
 $Comp
-L GND #PWR06
+L GND #PWR9
 U 1 1 56EB3C80
 P 2800 2150
-F 0 "#PWR06" H 2800 1900 50  0001 C CNN
+F 0 "#PWR9" H 2800 1900 50  0001 C CNN
 F 1 "GND" H 2808 1977 50  0000 C CNN
 F 2 "" H 2800 2150 50  0000 C CNN
@@
 $EndComp
 $Comp
-L GND #PWR07
+L GND #PWR12
 U 1 1 56EB3FF8
 P 3400 2450
-F 0 "#PWR07" H 3400 2200 50  0001 C CNN
+F 0 "#PWR12" H 3400 2200 50  0001 C CNN
 F 1 "GND" H 3408 2277 50  0000 C CNN
 F 2 "" H 3400 2450 50  0000 C CNN
@@
 $EndComp
 $Comp
-L GND #PWR08
+L GND #PWR26
 U 1 1 56EB49C1
 P 9450 4650
-F 0 "#PWR08" H 9450 4400 50  0001 C CNN
+F 0 "#PWR26" H 9450 4400 50  0001 C CNN
 F 1 "GND" H 9458 4477 50  0000 C CNN
 F 2 "" H 9450 4650 50  0000 C CNN
@@
 $EndComp
 $Comp
-L +BATT #PWR09
+L +BATT #PWR2
 U 1 1 56EB4B90
 P 1400 1000
-F 0 "#PWR09" H 1400 850 50  0001 C CNN
+F 0 "#PWR2" H 1400 850 50  0001 C CNN
 F 1 "+BATT" H 1418 1173 50  0000 C CNN
 F 2 "" H 1400 1000 50  0000 C CNN
@@
 $EndComp
 $Comp
-L GND #PWR010
+L GND #PWR10
 U 1 1 56EB6272
 P 2850 6450
-F 0 "#PWR010" H 2850 6200 50  0001 C CNN
+F 0 "#PWR10" H 2850 6200 50  0001 C CNN
 F 1 "GND" H 2850 6300 50  0000 C CNN
 F 2 "" H 2850 6450 50  0000 C CNN
@@
 $EndComp
 $Comp
-L +5V #PWR011
+L +5V #PWR24
 U 1 1 56EBEE2E
 P 8900 5200
-F 0 "#PWR011" H 8900 5050 50  0001 C CNN
+F 0 "#PWR24" H 8900 5050 50  0001 C CNN
 F 1 "+5V" H 8918 5373 50  0000 C CNN
 F 2 "" H 8900 5200 50  0000 C CNN
@@
 $EndComp
 $Comp
-L +5V #PWR012
+L +5V #PWR25
 U 1 1 56EBA63A
 P 8900 5850
-F 0 "#PWR012" H 8900 5700 50  0001 C CNN
+F 0 "#PWR25" H 8900 5700 50  0001 C CNN
 F 1 "+5V" H 8918 6023 50  0000 C CNN
 F 2 "" H 8900 5850 50  0000 C CNN
@@
 $EndComp
 $Comp
-L GND #PWR013
+L GND #PWR21
 U 1 1 56EC4D70
-P 7500 1550
-F 0 "#PWR013" H 7500 1300 50  0001 C CNN
-F 1 "GND" H 7508 1377 50  0000 C CNN
-F 2 "" H 7500 1550 50  0000 C CNN
-F 3 "" H 7500 1550 50  0000 C CNN
-	1    7500 1550
-	1    0    0    -1
-$EndComp
-$Comp
-L GND #PWR014
+P 7650 1550
+F 0 "#PWR21" H 7650 1300 50  0001 C CNN
+F 1 "GND" H 7658 1377 50  0000 C CNN
+F 2 "" H 7650 1550 50  0000 C CNN
+F 3 "" H 7650 1550 50  0000 C CNN
+	1    7650 1550
+	1    0    0    -1
+$EndComp
+$Comp
+L GND #PWR19
 U 1 1 56EC5583
 P 6950 2700
-F 0 "#PWR014" H 6950 2450 50  0001 C CNN
+F 0 "#PWR19" H 6950 2450 50  0001 C CNN
 F 1 "GND" H 6958 2527 50  0000 C CNN
 F 2 "" H 6950 2700 50  0000 C CNN
@@
 $EndComp
 $Comp
-L GND #PWR015
+L GND #PWR17
 U 1 1 56EC7B84
 P 6100 2900
-F 0 "#PWR015" H 6100 2650 50  0001 C CNN
+F 0 "#PWR17" H 6100 2650 50  0001 C CNN
 F 1 "GND" H 6108 2727 50  0000 C CNN
 F 2 "" H 6100 2900 50  0000 C CNN
@@
 $EndComp
 $Comp
-L GND #PWR016
+L GND #PWR18
 U 1 1 56EC7C31
 P 6300 1850
-F 0 "#PWR016" H 6300 1600 50  0001 C CNN
+F 0 "#PWR18" H 6300 1600 50  0001 C CNN
 F 1 "GND" H 6308 1677 50  0000 C CNN
 F 2 "" H 6300 1850 50  0000 C CNN
@@
 $EndComp
 $Comp
-L +5V #PWR017
+L +5V #PWR16
 U 1 1 56EC8A39
 P 6050 900
-F 0 "#PWR017" H 6050 750 50  0001 C CNN
+F 0 "#PWR16" H 6050 750 50  0001 C CNN
 F 1 "+5V" H 6068 1073 50  0000 C CNN
 F 2 "" H 6050 900 50  0000 C CNN
@@
 $EndComp
 $Comp
-L +5V #PWR018
+L +5V #PWR15
 U 1 1 56EC9488
 P 5900 1750
-F 0 "#PWR018" H 5900 1600 50  0001 C CNN
+F 0 "#PWR15" H 5900 1600 50  0001 C CNN
 F 1 "+5V" H 5918 1923 50  0000 C CNN
 F 2 "" H 5900 1750 50  0000 C CNN
@@
 $EndComp
 $Comp
-L GND #PWR019
+L GND #PWR27
 U 1 1 56ECF501
 P 9550 1850
-F 0 "#PWR019" H 9550 1600 50  0001 C CNN
+F 0 "#PWR27" H 9550 1600 50  0001 C CNN
 F 1 "GND" H 9558 1677 50  0000 C CNN
 F 2 "" H 9550 1850 50  0000 C CNN
@@
 $EndComp
 $Comp
-L GND #PWR020
+L GND #PWR28
 U 1 1 56ECF5C0
 P 9550 2800
-F 0 "#PWR020" H 9550 2550 50  0001 C CNN
+F 0 "#PWR28" H 9550 2550 50  0001 C CNN
 F 1 "GND" H 9558 2627 50  0000 C CNN
 F 2 "" H 9550 2800 50  0000 C CNN
@@
 R17 till R20 only\nfor first device in\ndaisy chain
 $Comp
-L GND #PWR021
+L GND #PWR23
 U 1 1 56ED0C25
 P 8850 2450
-F 0 "#PWR021" H 8850 2200 50  0001 C CNN
+F 0 "#PWR23" H 8850 2200 50  0001 C CNN
 F 1 "GND" H 8858 2277 50  0000 C CNN
 F 2 "" H 8850 2450 50  0000 C CNN
 F 3 "" H 8850 2450 50  0000 C CNN
 	1    8850 2450
-	1    0    0    -1
-$EndComp
-$Comp
-L +BATT #PWR022
-U 1 1 56ED1A84
-P 8450 1250
-F 0 "#PWR022" H 8450 1100 50  0001 C CNN
-F 1 "+BATT" H 8468 1423 50  0000 C CNN
-F 2 "" H 8450 1250 50  0000 C CNN
-F 3 "" H 8450 1250 50  0000 C CNN
-	1    8450 1250
 	1    0    0    -1
 $EndComp
@@
 $EndComp
 $Comp
-L +BATT #PWR023
+L +BATT #PWR1
 U 1 1 56ED3686
 P 600 5800
-F 0 "#PWR023" H 600 5650 50  0001 C CNN
+F 0 "#PWR1" H 600 5650 50  0001 C CNN
 F 1 "+BATT" V 500 5950 50  0000 C CNN
 F 2 "" H 600 5800 50  0000 C CNN
@@
 $EndComp
 $Comp
-L GND #PWR024
+L GND #PWR14
 U 1 1 56ED69AF
 P 4800 6050
-F 0 "#PWR024" H 4800 5800 50  0001 C CNN
+F 0 "#PWR14" H 4800 5800 50  0001 C CNN
 F 1 "GND" H 4808 5877 50  0000 C CNN
 F 2 "" H 4800 6050 50  0000 C CNN
@@
 $EndComp
 $Comp
-L GND #PWR025
+L GND #PWR20
 U 1 1 56ED9E5D
 P 7000 6250
-F 0 "#PWR025" H 7000 6000 50  0001 C CNN
+F 0 "#PWR20" H 7000 6000 50  0001 C CNN
 F 1 "GND" H 7008 6077 50  0000 C CNN
 F 2 "" H 7000 6250 50  0000 C CNN
@@
 $EndComp
 $Comp
-L GND #PWR026
+L GND #PWR6
 U 1 1 56ECCB5F
 P 1800 4950
-F 0 "#PWR026" H 1800 4700 50  0001 C CNN
+F 0 "#PWR6" H 1800 4700 50  0001 C CNN
 F 1 "GND" H 1800 4800 50  0000 C CNN
 F 2 "" H 1800 4950 50  0000 C CNN
@@
 $EndComp
 $Comp
-L +BATT #PWR027
+L +BATT #PWR30
 U 1 1 56EDD9A3
 P 9950 1750
-F 0 "#PWR027" H 9950 1600 50  0001 C CNN
+F 0 "#PWR30" H 9950 1600 50  0001 C CNN
 F 1 "+BATT" H 9950 1900 50  0000 C CNN
 F 2 "" H 9950 1750 50  0000 C CNN
@@
 $EndComp
 $Comp
-L +BATT #PWR028
+L +BATT #PWR29
 U 1 1 56EDE180
 P 9950 800
-F 0 "#PWR028" H 9950 650 50  0001 C CNN
+F 0 "#PWR29" H 9950 650 50  0001 C CNN
 F 1 "+BATT" H 9950 950 50  0000 C CNN
 F 2 "" H 9950 800 50  0000 C CNN
@@
 $EndComp
 $Comp
-L GND #PWR029
+L GND #PWR4
 U 1 1 56EEA720
 P 1450 6450
-F 0 "#PWR029" H 1450 6200 50  0001 C CNN
+F 0 "#PWR4" H 1450 6200 50  0001 C CNN
 F 1 "GND" H 1450 6300 50  0000 C CNN
 F 2 "" H 1450 6450 50  0000 C CNN
@@
 $EndComp
 $Comp
-L GND #PWR030
+L GND #PWR3
 U 1 1 56EF8AA3
 P 1400 1400
-F 0 "#PWR030" H 1400 1150 50  0001 C CNN
+F 0 "#PWR3" H 1400 1150 50  0001 C CNN
 F 1 "GND" H 1408 1227 50  0000 C CNN
 F 2 "" H 1400 1400 50  0000 C CNN
@@
 	7050 2400 7050 2050
 Wire Wire Line
-	7350 1550 7350 1500
-Wire Wire Line
-	7350 1500 7500 1500
-Wire Wire Line
-	7500 1500 7500 1550
+	7350 1400 7350 1550
 Wire Wire Line
 	6950 2450 6950 2050
@@
 Wire Wire Line
 	8850 2450 8850 2050
-Wire Wire Line
-	8450 1550 8450 1250
 Wire Wire Line
 	600  5800 1200 5800
@@
 +5V_Host
 $Comp
-L PWR_FLAG #FLG031
+L PWR_FLAG #FLG1
 U 1 1 59362D21
 P 850 5900
-F 0 "#FLG031" H 850 5995 50  0001 C CNN
+F 0 "#FLG1" H 850 5995 50  0001 C CNN
 F 1 "PWR_FLAG" H 850 6123 50  0000 C CNN
 F 2 "" H 850 5900 50  0000 C CNN
@@
 Connection ~ 850  5800
 $Comp
-L PWR_FLAG #FLG032
+L PWR_FLAG #FLG2
 U 1 1 59362FF9
 P 1700 6400
-F 0 "#FLG032" H 1700 6495 50  0001 C CNN
+F 0 "#FLG2" H 1700 6495 50  0001 C CNN
 F 1 "PWR_FLAG" H 1700 6607 30  0000 C CNN
 F 2 "" H 1700 6400 50  0000 C CNN
@@
 Connection ~ 1700 6350
 NoConn ~ 9550 4750
+$Comp
+L +BATT #PWR22
+U 1 1 56ED1A84
+P 8450 1250
+F 0 "#PWR22" H 8450 1100 50  0001 C CNN
+F 1 "+BATT" H 8468 1423 50  0000 C CNN
+F 2 "" H 8450 1250 50  0000 C CNN
+F 3 "" H 8450 1250 50  0000 C CNN
+	1    8450 1250
+	1    0    0    -1
+$EndComp
+$Comp
+L Jumper_NO_Small JP3
+U 1 1 5AB98B02
+P 8450 1400
+F 0 "JP3" H 8400 1350 50  0000 L CNN
+F 1 "Jumper_NO_Small" H 8460 1340 50  0001 C CNN
+F 2 "tera_general:SOLDERJUMPER_2_1mm" H 8450 1400 50  0001 C CNN
+F 3 "" H 8450 1400 50  0000 C CNN
+	1    8450 1400
+	0    1    1    0
+$EndComp
+$Comp
+L Jumper_NO_Small JP2
+U 1 1 5AB98F61
+P 7500 1400
+F 0 "JP2" H 7450 1350 50  0000 L CNN
+F 1 "Jumper_NO_Small" H 7510 1340 50  0001 C CNN
+F 2 "tera_general:SOLDERJUMPER_2_1mm" H 7500 1400 50  0001 C CNN
+F 3 "" H 7500 1400 50  0000 C CNN
+	1    7500 1400
+	-1   0    0    1
+$EndComp
+Wire Wire Line
+	7400 1400 7350 1400
+Wire Wire Line
+	7650 1550 7650 1400
+Wire Wire Line
+	7650 1400 7600 1400
+Wire Wire Line
+	8450 1250 8450 1300
+Wire Wire Line
+	8450 1500 8450 1550
 $EndSCHEMATC
